File: DI8/DI8.kicad_sch (KiCad schematic)
At the start: 32 parts, among them J1 Conn_01x10, J2 Conn_01x04, J3 Conn_01x04, SW1 SW_SPDT, SW2 SW_SPDT, SW3 SW_SPDT, U1 PCF8574, U2 PC817, U3 PC817, U4 PC817, U5 PC817, U6 PC817, U7 PC817, U8 PC817, U9 PC817

Commit message: sync
Parts:
- removed J1: Conn_01x10, symbol Connector_Generic:Conn_01x10
- removed SW1, SW2, SW3: SW_SPDT, Button_Switch_THT:SW_Slide_SPDT_Straight_CK_OS102011MS2Q, symbol Switch:SW_SPDT
- removed U1: PCF8574, symbol Interface_Expansion:PCF8574
- added J1, J4: Conn_01x08, TerminalBlock_Phoenix:TerminalBlock_Phoenix_MKDS-1,5-8-5.08_1x08_P5.08mm_Horizontal, symbol Connector_Generic:Conn_01x08
- added J5, J6: Conn_01x10, Connector_PinHeader_2.54mm:PinHeader_1x10_P2.54mm_Vertical, symbol Connector_Generic:Conn_01x10
- added J7: Conn_01x02, TerminalBlock_Phoenix:TerminalBlock_Phoenix_MKDS-1,5-2-5.08_1x02_P5.08mm_Horizontal, symbol Connector_Generic:Conn_01x02
- added JP1, JP2, JP3: Jumper_3_Bridged12, Connector_PinHeader_2.54mm:PinHeader_1x03_P2.54mm_Vertical, symbol Jumper:Jumper_3_Bridged12
- added R17, R18, R19, R20, R21, R22, R23, R24: 1.1k, Resistor_THT:R_Axial_DIN0207_L6.3mm_D2.5mm_P10.16mm_Horizontal, symbol Device:R
- added R25, R26, R27, R28, R29, R30, R31, R32: 10k, Resistor_THT:R_Axial_DIN0207_L6.3mm_D2.5mm_P10.16mm_Horizontal, symbol Device:R
- added U10, U11, U12, U13, U14, U15, U16, U9: PC817, Package_DIP:DIP-4_W7.62mm, symbol Isolator:PC817
- added U17: PCF8575DBR, Package_SO:SSOP-24_5.3x8.2mm_P0.65mm, symbol Interface_Expansion:PCF8575DBR
- R1: renamed from R9; footprint (none) -> Resistor_THT:R_Axial_DIN0207_L6.3mm_D2.5mm_P10.16mm_Horizontal
- R10: renamed from R2; footprint (none) -> Resistor_THT:R_Axial_DIN0207_L6.3mm_D2.5mm_P10.16mm_Horizontal
- R11: renamed from R3; footprint (none) -> Resistor_THT:R_Axial_DIN0207_L6.3mm_D2.5mm_P10.16mm_Horizontal
- R12: renamed from R4; footprint (none) -> Resistor_THT:R_Axial_DIN0207_L6.3mm_D2.5mm_P10.16mm_Horizontal
- R13: renamed from R5; footprint (none) -> Resistor_THT:R_Axial_DIN0207_L6.3mm_D2.5mm_P10.16mm_Horizontal
- R14: renamed from R6; footprint (none) -> Resistor_THT:R_Axial_DIN0207_L6.3mm_D2.5mm_P10.16mm_Horizontal
- R15: renamed from R7; footprint (none) -> Resistor_THT:R_Axial_DIN0207_L6.3mm_D2.5mm_P10.16mm_Horizontal
- R16: renamed from R8; footprint (none) -> Resistor_THT:R_Axial_DIN0207_L6.3mm_D2.5mm_P10.16mm_Horizontal
- R2: renamed from R10; footprint (none) -> Resistor_THT:R_Axial_DIN0207_L6.3mm_D2.5mm_P10.16mm_Horizontal
- R3: renamed from R11; footprint (none) -> Resistor_THT:R_Axial_DIN0207_L6.3mm_D2.5mm_P10.16mm_Horizontal
- R4: renamed from R12; footprint (none) -> Resistor_THT:R_Axial_DIN0207_L6.3mm_D2.5mm_P10.16mm_Horizontal
- R5: renamed from R13; footprint (none) -> Resistor_THT:R_Axial_DIN0207_L6.3mm_D2.5mm_P10.16mm_Horizontal
- R6: renamed from R14; footprint (none) -> Resistor_THT:R_Axial_DIN0207_L6.3mm_D2.5mm_P10.16mm_Horizontal
- R7: renamed from R15; footprint (none) -> Resistor_THT:R_Axial_DIN0207_L6.3mm_D2.5mm_P10.16mm_Horizontal
- R8: renamed from R16; footprint (none) -> Resistor_THT:R_Axial_DIN0207_L6.3mm_D2.5mm_P10.16mm_Horizontal
- R9: renamed from R1; footprint (none) -> Resistor_THT:R_Axial_DIN0207_L6.3mm_D2.5mm_P10.16mm_Horizontal
- renumbered U2 to U1, U3 to U2, U4 to U3, U5 to U4, U6 to U5, U7 to U6, U8 to U7, U9 to U8
Connections:
- net +5V: now also JP1.3 (B), JP2.3 (B), JP3.3 (B), R25.1, R26.1, R27.1, R28.1, R29.1, R30.1, R31.1, R32.1, U17.24 (VCC)
- net A1: now also JP1.2 (C), U17.21 (A0)
- net A2: now also JP2.2 (C), U17.2 (A1)
- net A3: now also JP3.2 (C), U17.3 (A2)
- net GND: now also JP1.1 (A), JP2.1 (A), JP3.1 (A), U10.3, U11.3, U12.3, U13.3, U14.3, U15.3, U16.3, U17.12 (GND), U9.3
- net SCL: now also U17.22 (SCL)
- net SDA: now also U17.23 (SDA)
- net M: now reaches U1.2, U2.2, U3.2, U4.2, U5.2, U6.2, U7.2, U8.2
- net M: now also J7.2 (Pin_2), U10.2, U11.2, U12.2, U13.2, U14.2, U15.2, U16.2, U9.2
- net P7: now reaches R16.2, U8.4
- net P7: now also J5.8 (Pin_8), U17.11 (P7)
- net at R3.1: now also J1.3 (Pin_3)
- net at R5.1: now also J1.5 (Pin_5)
- net P5: now reaches R14.2, U6.4
- net P5: now also J5.6 (Pin_6), U17.9 (P5)
- net P3: now reaches R12.2, U4.4
- net P3: now also J5.4 (Pin_4), U17.7 (P3)
- net P0: now reaches R9.2, U1.4
- net P0: now also J5.1 (Pin_1), U17.4 (P0)
- net P6: now reaches R15.2, U7.4
- net P6: now also J5.7 (Pin_7), U17.10 (P6)
- net P2: now reaches R11.2, U3.4
- net P2: now also J5.3 (Pin_3), U17.6 (P2)
- net at R7.1: now also J1.7 (Pin_7)
- net at R1.1: now also J1.1 (Pin_1)
- net P4: now reaches R13.2, U5.4
- net P4: now also J5.5 (Pin_5), U17.8 (P4)
- net at R8.1: now also J1.8 (Pin_8)
- net at R2.1: now also J1.2 (Pin_2)
- net at R4.1: now also J1.4 (Pin_4)
- net at R6.1: now also J1.6 (Pin_6)
- net P1: now reaches R10.2, U2.4
- net P1: now also J5.2 (Pin_2), U17.5 (P1)
- new net: R20.2, U12.1
- new net: R18.2, U10.1
- new net: J4.2 (Pin_2), R18.1
- new net: R19.2, U11.1
- new net: R21.2, U13.1
- new net: J4.1 (Pin_1), R17.1
- new net: R17.2, U9.1
- new net: R22.2, U14.1
- new net: R24.2, U16.1
- new net: J4.3 (Pin_3), R19.1
- new net: J4.4 (Pin_4), R20.1
- new net: J4.5 (Pin_5), R21.1
- new net: J4.6 (Pin_6), R22.1
- new net: J4.7 (Pin_7), R23.1
- new net: J4.8 (Pin_8), R24.1
- new net: R23.2, U15.1
- new net P10: J6.1 (Pin_1), R25.2, U17.13 (P10), U9.4
- new net P11: J6.2 (Pin_2), R26.2, U10.4, U17.14 (P11)
- new net P12: J6.3 (Pin_3), R27.2, U11.4, U17.15 (P12)
- new net P13: J6.4 (Pin_4), R28.2, U12.4, U17.16 (P13)
- new net P14: J6.5 (Pin_5), R29.2, U13.4, U17.17 (P14)
- new net P15: J6.6 (Pin_6), R30.2, U14.4, U17.18 (P15)
- new net P16: J6.7 (Pin_7), R31.2, U15.4, U17.19 (P16)
- new net P17: J6.8 (Pin_8), R32.2, U16.4, U17.20 (P17)
- no-connect marks 1 -> 0
Other:
- note added: "Подключение шлейфа"
- moved on the sheet: F1, J2, J3, R1, R10, R11, R12, R13, R14, R15, R16, R2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
