File: PM-OC8/current/PM-OC8.kicad_sch (KiCad schematic)
At the start: 26 parts, among them J1 Conn_01x10_Pin, J2 Conn_01x10_Pin, U1 PC817, U2 PC817, U3 PC817, U4 PC817, U5 PC817, U6 PC817, U7 PC817, U8 PC817

Commit message: add files
Other:
- moved on the sheet: J2
