File: PM-OC8/current/PM-OC8.kicad_pcb (KiCad board)
At the start: 2 copper layers, 25.4 x 53.3 mm, 26 parts, among them J1 Conn_01x10_Pin, J2 Conn_01x10_Pin, U1 PC817, U2 PC817, U3 PC817, U4 PC817, U5 PC817, U6 PC817, U7 PC817, U8 PC817

Commit message: add files
Parts:
- moved J2 1.66 mm to (121.9, 102.9)
- moved J1 0.88 mm to (106.7, 102.9)
Routing:
- net Net-(D5-K): track 23.4 -> 17.0 mm
- net Net-(D3-K): track 24.3 -> 17.9 mm
- net +5V: track 113.2 -> 110.8 mm
- net Net-(D2-K): track 19.7 -> 17.8 mm
- net Net-(D8-K): track 27.2 -> 25.4 mm
- net Net-(J2-Pin_9): track 25.6 -> 23.9 mm
- net Net-(J2-Pin_7): track 17.4 -> 15.8 mm
- net Net-(J2-Pin_6): track 25.6 -> 27.2 mm
- net Net-(J2-Pin_5): track 15.4 -> 13.8 mm
- net Net-(J2-Pin_4): track 28.6 -> 30.3 mm
- net Net-(J2-Pin_2): track 36.2 -> 37.9 mm
- net GND: track 71.4 -> 73.0 mm
- net Net-(J2-Pin_8): track 31.9 -> 33.6 mm
- net Net-(D6-K): track 18.7 -> 17.1 mm
- net Net-(J2-Pin_3): track 22.7 -> 21.3 mm
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Other:
- board text added: "PM-OC8"
- board text added: "v0.0.1"
- board text removed: "PM-OC8-0.0.1"

Commit message: sync
Changed lines of the file:
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@@
 			(pdf_front_fp_property_popups yes)
 			(pdf_back_fp_property_popups yes)
-			(dxfpolygonmode yes)
+			(dxfpolygonmode no)
 			(dxfimperialunits yes)
 			(dxfusepcbnewfont yes)
@@
 			(sketchpadsonfab no)
 			(subtractmaskfromsilk no)
-			(outputformat 1)
+			(outputformat 4)
 			(mirror no)
 			(drillshape 0)
@@
 		)
 		(stroke
-			(width 0.2)
+			(width 0.127)
 			(type solid)
 		)
