File: DI16/DI16.kicad_pcb (KiCad board)
At the start: 2 copper layers, 120 x 80 mm, 60 parts, among them J1 Conn_01x08, J2 Conn_01x04, J3 Conn_01x04, J4 Conn_01x08, J5 Conn_01x10, J6 Conn_01x10, J7 Conn_01x02, U1 PC817, U10 PC817, U11 PC817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

Commit message: power source
Parts:
- R1, R17, R18, R19, R2, R20, R21, R22, R23, R24, R3, R4, R5, R6, R7, R8: value 1.1k -> 1.1к; footprint Resistor_THT:R_Axial_DIN0207_L6.3mm_D2.5mm_P10.16mm_Horizontal -> Resistor_THT:R_Axial_DIN0309_L9.0mm_D3.2mm_P5.08mm_Vertical
- R10, R11, R12, R13, R14, R15, R16, R25, R26, R27, R28, R29, R30, R31, R32, R9: value 10k -> 10к; footprint Resistor_THT:R_Axial_DIN0207_L6.3mm_D2.5mm_P10.16mm_Horizontal -> Resistor_THT:R_Axial_DIN0207_L6.3mm_D2.5mm_P5.08mm_Vertical
- U17: value PCF8575DBR -> PCF8575TS
- moved R22 5.09 mm to (191.4, 80.5)
- moved R11 5.08 mm to (158.4, 103.4)
- moved R5 5.08 mm to (143.2, 88.1)
- moved R7 5.08 mm to (143.2, 72.9)
- moved R23 5.08 mm to (191.4, 72.9)
- moved R24 5.08 mm to (191.4, 65.2)
- moved R6 5.08 mm to (143.2, 80.5)
- moved R8 5.08 mm to (143.2, 65.2)
- moved R10 5.08 mm to (158.4, 100.8)
- moved R12 5.08 mm to (158.4, 105.9)
- moved R13 5.08 mm to (158.4, 108.4)
- moved R14 5.08 mm to (158.4, 111.0)
- moved R15 5.08 mm to (158.4, 113.5)
- moved R16 5.08 mm to (158.4, 116.0)
- moved R25 5.08 mm to (186.4, 98.3)
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
Commit message: PM-GE16
Parts:
- removed J4: Conn_01x08, TerminalBlock_Phoenix:TerminalBlock_Phoenix_MKDS-1,5-8-5.08_1x08_P5.08mm_Horizontal
- removed J7: Conn_01x02, TerminalBlock_Phoenix:TerminalBlock_Phoenix_MKDS-1,5-2-5.08_1x02_P5.08mm_Horizontal
- added J10: Conn_01x03_Socket, TerminalBlock_Phoenix:TerminalBlock_Phoenix_MKDS-1,5-3-5.08_1x03_P5.08mm_Horizontal, F.Cu at (120.3, 55.1)
- added J9: Terminal_01x08_Socket, TerminalBlock_Phoenix:TerminalBlock_Phoenix_MKDS-1,5-8-5.08_1x08_P5.08mm_Horizontal, F.Cu at (206.7, 55.1)
- F1: footprint Fuse:Fuseholder_Cylinder-5x20mm_Schurter_0031_8201_Horizontal_Open -> Fuse:Fuseholder_Cylinder-5x20mm_Stelvio-Kontek_PTF78_Horizontal_Open
- J1: value Conn_01x08 -> Terminal_01x08_Socket
- J2, J3: value Conn_01x04 -> PinHeader_01x04_angle
- moved F1 20.1 mm to (112.7, 116.0), turned to 0 degrees
- moved J1 2.54 mm to (163.5, 55.1)
Other:
- outline, holes or cut-outs redrawn
