File: DI16/DI16.kicad_sch (KiCad schematic)
At the start: 60 parts, among them J1 Conn_01x08, J2 Conn_01x04, J3 Conn_01x04, J4 Conn_01x08, J5 Conn_01x10, J6 Conn_01x10, J7 Conn_01x02, U1 PC817, U10 PC817, U11 PC817, U12 PC817, U13 PC817, U14 PC817, U15 PC817, U16 PC817, U17 PCF8575DBR, U2 PC817, U3 PC817, U4 PC817, U5 PC817, U6 PC817, U7 PC817, U8 PC817, U9 PC817

Commit message: power source
Parts:
- removed R1, R17, R18, R19, R2, R20, R21, R22, R23, R24, R3, R4, R5, R6, R7, R8: 1.1k, Resistor_THT:R_Axial_DIN0207_L6.3mm_D2.5mm_P10.16mm_Horizontal, symbol Device:R
- removed R10, R11, R12, R13, R14, R15, R16, R25, R26, R27, R28, R29, R30, R31, R32, R9: 10k, Resistor_THT:R_Axial_DIN0207_L6.3mm_D2.5mm_P10.16mm_Horizontal, symbol Device:R
- removed U1, U10, U11, U12, U13, U14, U15, U16, U2, U3, U4, U5, U6, U7, U8, U9: PC817, Package_DIP:DIP-4_W7.62mm, symbol Isolator:PC817
- removed U17: PCF8575DBR, Package_SO:SSOP-24_5.3x8.2mm_P0.65mm, symbol Interface_Expansion:PCF8575DBR
- added R1, R17, R18, R19, R2, R20, R21, R22, R23, R24, R3, R4, R5, R6, R7, R8: 1.1к, Resistor_THT:R_Axial_DIN0309_L9.0mm_D3.2mm_P5.08mm_Vertical, symbol PlcModules:R_1.1k_0.5wt
- added R10, R11, R12, R13, R14, R15, R16, R25, R26, R27, R28, R29, R30, R31, R32, R9: 10к, Resistor_THT:R_Axial_DIN0207_L6.3mm_D2.5mm_P5.08mm_Vertical, symbol PlcModules:R_10k_0.25wt
- added U1, U10, U11, U12, U13, U14, U15, U16, U2, U3, U4, U5, U6, U7, U8, U9: PC817, Package_DIP:DIP-4_W7.62mm, symbol PlcModules:PC817
- added U17: PCF8575TS, Package_SO:SSOP-24_5.3x8.2mm_P0.65mm, symbol PlcModules:PCF8575TS
Connections:
- net +5V: now also R10.1, R11.1, R12.1, R13.1, R14.1, R15.1, R16.1, R25.1, R26.1, R27.1, R28.1, R29.1, R30.1, R31.1, R32.1, R9.1, U17.24 (VCC)
- net A1: now also U17.21 (A0)
- net A2: now also U17.2 (A1)
- net A3: now also U17.3 (A2)
- net GND: now also U1.3, U10.3, U11.3, U12.3, U13.3, U14.3, U15.3, U16.3, U17.12 (GND), U2.3, U3.3, U4.3, U5.3, U6.3, U7.3, U8.3, U9.3
- net M: now also U1.2, U10.2, U11.2, U12.2, U13.2, U14.2, U15.2, U16.2, U2.2, U3.2, U4.2, U5.2, U6.2, U7.2, U8.2, U9.2
- net P0: now also R9.2, U1.4, U17.4 (P0)
- net P1: now also R10.2, U17.5 (P1), U2.4
- net P10: now also R25.2, U17.13 (P10), U9.4
- net P11: now also R26.2, U10.4, U17.14 (P11)
- net P12: now also R27.2, U11.4, U17.15 (P12)
- net P13: now also R28.2, U12.4, U17.16 (P13)
- net P14: now also R29.2, U13.4, U17.17 (P14)
- net P15: now also R30.2, U14.4, U17.18 (P15)
- net P16: now also R31.2, U15.4, U17.19 (P16)
- net P17: now also R32.2, U16.4, U17.20 (P17)
- net P2: now also R11.2, U17.6 (P2), U3.4
- net P3: now also R12.2, U17.7 (P3), U4.4
- net P4: now also R13.2, U17.8 (P4), U5.4
- net P5: now also R14.2, U17.9 (P5), U6.4
- net P6: now also R15.2, U17.10 (P6), U7.4
- net P7: now also R16.2, U17.11 (P7), U8.4
- net SCL: now also U17.22 (SCL)
- net SDA: now also U17.23 (SDA)
- net at J1.3 (Pin_3): now also R3.1
- net at J1.5 (Pin_5): now also R5.1
- net at J4.2 (Pin_2): now also R18.1
- net at J1.7 (Pin_7): now also R7.1
- net at J4.1 (Pin_1): now also R17.1
- net at J1.1 (Pin_1): now also R1.1
- net at J1.8 (Pin_8): now also R8.1
- net at J1.2 (Pin_2): now also R2.1
- net at J1.4 (Pin_4): now also R4.1
- net at J1.6 (Pin_6): now also R6.1
- net at J4.3 (Pin_3): now also R19.1
- net at J4.4 (Pin_4): now also R20.1
- net at J4.5 (Pin_5): now also R21.1
- net at J4.6 (Pin_6): now also R22.1
- net at J4.7 (Pin_7): now also R23.1
- net at J4.8 (Pin_8): now also R24.1
- new net: R6.2, U6.1
- new net: R1.2, U1.1
- new net: R8.2, U8.1
- new net: R3.2, U3.1
- new net: R20.2, U12.1
- new net: R19.2, U11.1
- new net: R4.2, U4.1
- new net: R18.2, U10.1
- new net: R24.2, U16.1
- new net: R17.2, U9.1
- new net: R21.2, U13.1
- new net: R7.2, U7.1
- new net: R23.2, U15.1
- new net: R5.2, U5.1
- new net: R22.2, U14.1
- new net: R2.2, U2.1

Commit message: PM-GE16
Parts:
- removed F1: Fuse, Fuse:Fuseholder_Cylinder-5x20mm_Schurter_0031_8201_Horizontal_Open, symbol Device:Fuse
- removed J1, J4: Conn_01x08, TerminalBlock_Phoenix:TerminalBlock_Phoenix_MKDS-1,5-8-5.08_1x08_P5.08mm_Horizontal, symbol Connector_Generic:Conn_01x08
- removed J2, J3: Conn_01x04, Connector_PinHeader_2.54mm:PinHeader_1x04_P2.54mm_Horizontal, symbol Connector_Generic:Conn_01x04
- removed J7: Conn_01x02, TerminalBlock_Phoenix:TerminalBlock_Phoenix_MKDS-1,5-2-5.08_1x02_P5.08mm_Horizontal, symbol Connector_Generic:Conn_01x02
- added F1: Fuse, Fuse:Fuseholder_Cylinder-5x20mm_Stelvio-Kontek_PTF78_Horizontal_Open, symbol PlcModules:Fuse
- added J1, J9: Terminal_01x08_Socket, TerminalBlock_Phoenix:TerminalBlock_Phoenix_MKDS-1,5-8-5.08_1x08_P5.08mm_Horizontal, symbol PlcModules:Terminal_01x08_Socket
- added J10: Conn_01x03_Socket, TerminalBlock_Phoenix:TerminalBlock_Phoenix_MKDS-1,5-3-5.08_1x03_P5.08mm_Horizontal, symbol PlcModules:Terminal_01x03_Socket
- added J2, J3: PinHeader_01x04_angle, Connector_PinHeader_2.54mm:PinHeader_1x04_P2.54mm_Horizontal, symbol PlcModules:PinHeader_01x04_angle
- added J4, J8: Conn_01x08_Pin, symbol PlcModules:Terminal_01x08_Pin
- added J7: Conn_01x03_Pin, symbol PlcModules:Terminal_01x03_Pin
Connections:
- net +5V: now also F1.1
- net GND: now also J2.3 (Pin_3), J3.3 (Pin_3)
- net M: now also J10.2 (Pin_2)
- net SCL: now also J2.1 (Pin_1), J3.1 (Pin_1)
- net SDA: now also J2.4 (Pin_4), J3.4 (Pin_4)
- net at R8.1: now also J1.8 (Pin_8)
- net at R4.1: now also J1.4 (Pin_4)
- net at R20.1: now also J9.4 (Pin_4)
- net at R6.1: now also J1.6 (Pin_6)
- net at R3.1: now also J1.3 (Pin_3)
- net at R1.1: now also J1.1 (Pin_1)
- net at R21.1: now also J9.5 (Pin_5)
- net at R5.1: now also J1.5 (Pin_5)
- net at R2.1: now also J1.2 (Pin_2)
- net at R7.1: now also J1.7 (Pin_7)
- net at R17.1: now also J9.1 (Pin_1)
- net at R18.1: now also J9.2 (Pin_2)
- net at R19.1: now also J9.3 (Pin_3)
- net at R22.1: now also J9.6 (Pin_6)
- net at R23.1: now also J9.7 (Pin_7)
- net at R24.1: now also J9.8 (Pin_8)
- new net: F1.2, J2.2 (Pin_2), J3.2 (Pin_2)
Other:
- company: (none) -> UST
- title: (none) -> Модуль DI16

Commit message: sync
Parts:
- added U18: NA555_PD, Package_DIP:DIP-8_W7.62mm_LongPads, symbol temp:NA555_PD
Connections:
- no-connect marks 0 -> 1
Changed lines of the file:
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@@
 		(color 0 0 0 0)
 	)
+	(no_connect
+		(at 26.67 35.56)
+	)
 	(wire
 		(pts
@@
 					(unit 1)
 				)
+			)
+		)
+	)
+	(symbol
+		(lib_id "temp:NA555_PD")
+		(at 269.24 213.36 0)
+		(unit 1)
+		(exclude_from_sim no)
+		(in_bom yes)
+		(on_board yes)
+		(dnp no)
+		(fields_autoplaced yes)
+		(property "Reference" "U18"
+			(at 271.4341 213.36 0)
+			(effects
+				(font
+					(size 1.27 1.27)
+				)
+				(justify left)
+			)
+		)
+		(property "Value" "NA555_PD"
+			(at 271.4341 215.9 0)
+			(effects
+				(font
+					(size 1.27 1.27)
+				)
+				(justify left)
+			)
+		)
+		(property "Footprint" "Package_DIP:DIP-8_W7.62mm_LongPads"
+			(at 269.24 213.36 0)
+			(effects
+				(font
+					(size 1.27 1.27)
+				)
+				(hide yes)
+			)
+		)
+		(property "Datasheet" ""
+			(at 269.24 213.36 0)
+			(effects
+				(font
+					(size 1.27 1.27)
+				)
+				(hide yes)
+			)
+		)
+		(property "Description" ""
+			(at 269.24 213.36 0)
+			(effects
+				(font
+					(size 1.27 1.27)
+				)
+				(hide yes)
+			)
+		)
+		(pin "6"
+		)
+		(pin "2"
+		)
+		(pin "5"
+		)
+		(pin "7"
+		)
+		(pin "4"
+		)
+		(pin "8"
+		)
+		(pin "1"
+		)
+		(pin "3"
+		)
+		(instances
+			(project "DI16"
+				(path "/9da2aeb3-ff67-4afa-a5d0-11128825e2f7"
+					(reference "U18")
+					(unit 1)
+				)
