File: PM-GE16/PM-GE16.kicad_pcb (KiCad board)
At the start: 2 copper layers, 30.5 x 30.5 mm, 6 parts, among them J1 Conn_02x08_Top_Bottom, J2 Conn_01x04_Pin, J3 Conn_01x03, J4 Conn_01x03, J5 Conn_01x03, U2 PCA9555PW

Commit message: sync
Parts:
- removed J2: Conn_01x04_Pin, Connector_PinHeader_2.54mm:PinHeader_1x04_P2.54mm_Vertical_SMD_Pin1Left
- J1: value Conn_02x08_Top_Bottom -> Conn_02x10_Odd_Even; footprint Connector_PinHeader_2.54mm:PinHeader_2x08_P2.54mm_Vertical_SMD -> Connector_PinHeader_2.54mm:PinHeader_2x10_P2.54mm_Vertical_SMD
- moved J3 15.3 mm to (82.5, 52.0), turned to 0 degrees
- moved J5 15.3 mm to (97.8, 52.0), turned to 0 degrees
- moved J1 6.36 mm to (91.5, 62.2)
- moved U2 1.90 mm to (91.4, 69.8), turned to 180 degrees
- moved J4 1.34 mm to (90.2, 52.0), turned to 0 degrees
Connections:
- net Net-(J1-Pin_1) renamed /00
- net Net-(J1-Pin_16) renamed /17
- J1 pad 10: Net-(J1-Pin_10) -> /14
- J1 pad 11: Net-(J1-Pin_11) -> /05
- J1 pad 12: Net-(J1-Pin_12) -> /15
- J1 pad 13: Net-(J1-Pin_13) -> /06
- J1 pad 14: Net-(J1-Pin_14) -> /16
- J1 pad 15: Net-(J1-Pin_15) -> /07
- J1 pad 2: Net-(J1-Pin_2) -> /10
- J1 pad 3: Net-(J1-Pin_3) -> /01
- J1 pad 4: Net-(J1-Pin_4) -> /11
- J1 pad 5: Net-(J1-Pin_5) -> /02
- J1 pad 6: Net-(J1-Pin_6) -> /12
- J1 pad 7: Net-(J1-Pin_7) -> /03
- J1 pad 8: Net-(J1-Pin_8) -> /13
- J1 pad 9: Net-(J1-Pin_9) -> /04
- U2 pad 10: Net-(J1-Pin_7) -> /06
- U2 pad 11: Net-(J1-Pin_8) -> /07
- U2 pad 13: Net-(J1-Pin_9) -> /10
- U2 pad 14: Net-(J1-Pin_10) -> /11
- U2 pad 15: Net-(J1-Pin_11) -> /12
- U2 pad 16: Net-(J1-Pin_12) -> /13
- U2 pad 17: Net-(J1-Pin_13) -> /14
- U2 pad 18: Net-(J1-Pin_14) -> /15
- U2 pad 19: Net-(J1-Pin_15) -> /16
- U2 pad 5: Net-(J1-Pin_2) -> /01
- U2 pad 6: Net-(J1-Pin_3) -> /02
- U2 pad 7: Net-(J1-Pin_4) -> /03
- U2 pad 8: Net-(J1-Pin_5) -> /04
- U2 pad 9: Net-(J1-Pin_6) -> /05
Routing:
- net VDD: track 3.66 -> 51.4 mm
- net GND: track 6.43 -> 46.0 mm, vias 4 -> 1
- net Net-(J1-Pin_2): track 22.8 -> 0.00 mm, vias 1 -> 0
- net /01: track 0.00 -> 22.3 mm, vias 0 -> 1
- net /10: track 0.00 -> 18.5 mm, vias 0 -> 1
- net /02: track 0.00 -> 18.3 mm, vias 0 -> 1
- net /11: track 0.00 -> 16.8 mm, vias 0 -> 1
- net Net-(J1-Pin_4): track 15.6 -> 0.00 mm, vias 1 -> 0
- net /12: track 0.00 -> 15.2 mm, vias 0 -> 1
- net Net-(J1-Pin_14): track 13.9 -> 0.00 mm, vias 1 -> 0
- net /04: track 0.00 -> 13.4 mm, vias 0 -> 1
- net /03: track 0.00 -> 13.4 mm, vias 0 -> 1
- net Net-(J1-Pin_6): track 13.4 -> 0.00 mm, vias 1 -> 0
- net /13: track 0.00 -> 13.2 mm, vias 0 -> 1
- net Net-(J1-Pin_3): track 12.8 -> 0.00 mm, vias 1 -> 0
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- added copper zone on B.Cu, net (none)
- added copper zone on F.Cu, net (none)
- removed copper zone on B.Cu, net GND
- removed copper zone on F.Cu, net VDD
Other:
- board text added: "PM-GE16"
- board text removed: "PM-GE16-0.0.1"
