File: PM-GE16/PM-GE16.kicad_sch (KiCad schematic)
At the start: 6 parts, among them J1 Conn_02x08_Top_Bottom, J2 Conn_01x04_Pin, J3 Conn_01x03, J4 Conn_01x03, J5 Conn_01x03, U2 PCA9555PW

Commit message: sync
Parts:
- removed J1: Conn_02x08_Top_Bottom, Connector_PinHeader_2.54mm:PinHeader_2x08_P2.54mm_Vertical_SMD, symbol Connector_Generic:Conn_02x08_Top_Bottom
- removed J2: Conn_01x04_Pin, Connector_PinHeader_2.54mm:PinHeader_1x04_P2.54mm_Vertical_SMD_Pin1Left, symbol Connector:Conn_01x04_Pin
- added J1: Conn_02x10_Odd_Even, Connector_PinHeader_2.54mm:PinHeader_2x10_P2.54mm_Vertical_SMD, symbol Connector_Generic:Conn_02x10_Odd_Even
- U2: NextPCB_price (none) -> 0.75761; NextPCB_url (none) -> https://www.hqonline.com/product-detail/enzhipu-nxp--pca955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
Connections:
- net GND: now also J1.19 (Pin_19)
- net SCL: now also J1.20 (Pin_20)
- net SDA: now also J1.18 (Pin_18)
- net VDD: now also J1.17 (Pin_17)
- net 06: now reaches U2.10 (IO0_6)
- net 06: now also J1.13 (Pin_13)
- net 07: now reaches U2.11 (IO0_7)
- net 07: now also J1.15 (Pin_15)
- net 10: now reaches U2.13 (IO1_0)
- net 10: now also J1.2 (Pin_2)
- net 11: now reaches U2.14 (IO1_1)
- net 11: now also J1.4 (Pin_4)
- net 12: now reaches U2.15 (IO1_2)
- net 12: now also J1.6 (Pin_6)
- net 13: now reaches U2.16 (IO1_3)
- net 13: now also J1.8 (Pin_8)
- net 14: now reaches U2.17 (IO1_4)
- net 14: now also J1.10 (Pin_10)
- net 15: now reaches U2.18 (IO1_5)
- net 15: now also J1.12 (Pin_12)
- net 16: now reaches U2.19 (IO1_6)
- net 16: now also J1.14 (Pin_14)
- net 17: now reaches U2.20 (IO1_7)
- net 17: now also J1.16 (Pin_16)
- net 00: now reaches U2.4 (IO0_0)
- net 00: now also J1.1 (Pin_1)
- net 01: now reaches U2.5 (IO0_1)
- net 01: now also J1.3 (Pin_3)
- net 02: now reaches U2.6 (IO0_2)
- net 02: now also J1.5 (Pin_5)
- net 03: now reaches U2.7 (IO0_3)
- net 03: now also J1.7 (Pin_7)
- net 04: now reaches U2.8 (IO0_4)
- net 04: now also J1.9 (Pin_9)
- net 05: now reaches U2.9 (IO0_5)
- net 05: now also J1.11 (Pin_11)
