File: PM-Base-RQ8/PM-Base-RQ8.kicad_pcb (KiCad board)
At the start: 2 copper layers, 99.1 x 99.1 mm, 22 parts, among them J1 Conn_01x02_Socket, J10 Conn_02x08_Odd_Even, J11 Conn_02x08_Odd_Even, J12 Conn_02x08_Odd_Even, J13 Conn_02x08_Odd_Even, J14 Conn_01x04_Socket, J15 Conn_01x04_Socket, J16 Conn_01x04_Socket, J19 Conn_01x10_Socket, J2 Conn_01x02_Socket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

Commit message: Update PM-Base-RQ8.kicad_pcb
Routing:
- net Net-(J11-Pin_8): track 54.3 -> 44.7 mm
- net Net-(J13-Pin_6): track 57.1 -> 50.8 mm, vias 0 -> 2
- net Net-(J13-Pin_8): track 52.2 -> 45.9 mm
- net Net-(J12-Pin_10): track 59.6 -> 55.9 mm, vias 0 -> 2
- net Net-(J11-Pin_4): track 44.1 -> 41.3 mm
- net Net-(J11-Pin_2): track 47.3 -> 44.6 mm
- net Net-(J12-Pin_16): track 56.7 -> 59.3 mm, vias 0 -> 2
- net Net-(J12-Pin_14): track 56.7 -> 59.2 mm, vias 0 -> 2
- net Net-(J13-Pin_4): track 48.9 -> 46.7 mm, vias 0 -> 2
- net GND: track 16.2 -> 18.0 mm, vias 7 -> 6
- net /SCL: track 70.5 -> 71.7 mm, vias 0 -> 2
- net Net-(J10-Pin_10): track 30.9 -> 29.8 mm
- net Net-(J11-Pin_6): track 45.6 -> 44.6 mm
- net Net-(J10-Pin_5): track 32.8 -> 31.9 mm
- net /SDA: track 70.5 -> 71.4 mm, vias 0 -> 2
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Other:
- copper layers 2 -> 4
