File: PM-RQ8-base/PM-RQ8-base.kicad_pcb (KiCad board)
At the start: 4 copper layers, 99.1 x 99.1 mm, 31 parts, among them J10 2EDGR-5.08-02P, J11 2EDGR-5.08-02P, J12 2EDGR-5.08-02P, J13 2EDGR-5.08-02P, J14 2EDGR-5.08-02P, J15 2EDGR-5.08-02P, J16 2EDGR-5.08-02P, J17 Conn_02x10_Odd_Even, J18 S4B-PH-SM4-TB, J19 S4B-PH-SM4-TB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

Commit message: PM-DI16-base
Parts:
- removed J17: Conn_02x10_Odd_Even, Connector_PinSocket_2.54mm:PinSocket_2x10_P2.54mm_Vertical_SMD
- added J25: Conn_02x08_socket, Connector_PinSocket_2.54mm:PinSocket_2x08_P2.54mm_Vertical_SMD, F.Cu at (99.1, 100.3)
- J19: moved to B.Cu
- moved Logo1 15.2 mm to (144.8, 144.8)
- moved J19 15.0 mm to (160.0, 141.0), turned to 0 degrees
- moved Logo2 14.0 mm to (133.3, 144.8)
- moved U3 5.08 mm to (160.1, 132.1)
- moved J18 0.66 mm to (160.0, 141.0)
- renumbered REF** to Logo1, REF** to Logo2
Routing:
- net /K8: track 117.8 -> 0.00 mm, vias 2 -> 0
- net /K7: track 110.9 -> 0.00 mm, vias 1 -> 0
- net /K6: track 94.6 -> 0.00 mm
- net /K5: track 84.4 -> 0.00 mm
- net /SDA: track 82.6 -> 0.00 mm
- net /K4: track 75.7 -> 0.00 mm
- net /SCL: track 71.5 -> 0.00 mm, vias 2 -> 0
- net /K3: track 69.6 -> 0.00 mm
- net /K2: track 67.4 -> 0.00 mm, vias 1 -> 0
- net /K1: track 67.3 -> 0.00 mm, vias 1 -> 0
- net Net-(U1-I6): track 35.9 -> 0.00 mm
- net Net-(J18-Pad1): track 31.1 -> 0.00 mm
- net Net-(U1-I1): track 30.1 -> 0.00 mm, vias 2 -> 0
- net Net-(U1-I7): track 27.5 -> 0.00 mm
- net Net-(U1-I2): track 27.3 -> 0.00 mm, vias 2 -> 0
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
Commit message: v0.0.1 send to nextpcb
Parts:
- removed Logo1: KiCad-Logo2_5mm_SilkScreen, Symbol:KiCad-Logo2_5mm_SilkScreen
- removed Logo2: OSHW-Logo_5.7x6mm_SilkScreen, Symbol:OSHW-Logo_5.7x6mm_SilkScreen
- H1, H2, H3, H4: value MountingHole_3.2mm_M3 -> MountingHole
- moved H1 116.6 mm to (99.1, 54.6)
- moved H2 116.6 mm to (171.4, 54.6)
- moved H3 116.6 mm to (171.4, 146.1)
- moved H4 116.6 mm to (99.1, 146.1)
- moved K8 8.89 mm to (119.6, 143.1)
- moved K7 7.62 mm to (119.6, 131.7)
- moved K6 6.35 mm to (119.6, 120.3)
- moved K5 5.08 mm to (119.6, 108.8)
- moved J10 3.81 mm to (86.4, 72.4)
- moved J11 3.81 mm to (86.4, 82.5)
- moved J13 3.81 mm to (86.4, 102.9)
- moved J14 3.81 mm to (86.4, 113.0)
- moved J15 3.81 mm to (86.4, 123.2)
- moved J16 3.81 mm to (86.4, 133.3)
- moved K4 3.81 mm to (119.6, 97.4)
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Connections:
- J19 pad 1: Net-(J18-Pad1) -> GND
- J19 pad 2: /SDA -> /SCL
- J19 pad 3: /SCL -> /SDA
- J19 pad 4: GND -> Net-(J18-Pad1)
- K1 pad 2: Net-(J9-Pin_1) -> Net-(J9-Pin_2)
- K1 pad 3: Net-(J9-Pin_2) -> Net-(J9-Pin_1)
- K2 pad 2: Net-(J10-Pin_1) -> Net-(J10-Pin_2)
- K2 pad 3: Net-(J10-Pin_2) -> Net-(J10-Pin_1)
- K3 pad 2: Net-(J11-Pin_1) -> Net-(J11-Pin_2)
- K3 pad 3: Net-(J11-Pin_2) -> Net-(J11-Pin_1)
- K4 pad 2: Net-(J12-Pin_1) -> Net-(J12-Pin_2)
- K4 pad 3: Net-(J12-Pin_2) -> Net-(J12-Pin_1)
- K5 pad 2: Net-(J13-Pin_1) -> Net-(J13-Pin_2)
- K5 pad 3: Net-(J13-Pin_2) -> Net-(J13-Pin_1)
- K6 pad 2: Net-(J14-Pin_1) -> Net-(J14-Pin_2)
- K6 pad 3: Net-(J14-Pin_2) -> Net-(J14-Pin_1)
- K7 pad 2: Net-(J15-Pin_1) -> Net-(J15-Pin_2)
- K7 pad 3: Net-(J15-Pin_2) -> Net-(J15-Pin_1)
- K8 pad 2: Net-(J16-Pin_1) -> Net-(J16-Pin_2)
- K8 pad 3: Net-(J16-Pin_2) -> Net-(J16-Pin_1)
Routing:
- net /K8: track 0.00 -> 126.4 mm, vias 0 -> 2
- net /K7: track 0.00 -> 113.8 mm, vias 0 -> 2
- net /K6: track 0.00 -> 105.0 mm, vias 0 -> 2
- net /K5: track 0.00 -> 89.3 mm, vias 0 -> 1
- net /K4: track 0.00 -> 79.0 mm
- net /K3: track 0.00 -> 70.7 mm
- net /K1: track 0.00 -> 68.6 mm
- net /K2: track 0.00 -> 68.4 mm
- net /SCL: track 0.00 -> 61.3 mm, vias 0 -> 2
- net /SDA: track 0.00 -> 58.4 mm, vias 0 -> 2
- net Net-(U1-I7): track 0.00 -> 36.2 mm
- net Net-(U1-I4): track 0.00 -> 29.4 mm
- net Net-(U1-I3): track 0.00 -> 29.0 mm
- net Net-(U1-I1): track 0.00 -> 27.5 mm
- net Net-(U1-I2): track 0.00 -> 27.5 mm, vias 0 -> 2
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Other:
- board text added: "+5V"
- board text added: "SCL"
- board text added: "SDA"

Commit message: work on v0.0.2
Parts:
- added logo_kicad: KiCad-Logo2_8mm_SilkScreen, Symbol:KiCad-Logo2_8mm_SilkScreen, B.Cu at (154.9, 58.4)
- added logo_oshw: OSHW-Symbol_13.4x12mm_SilkScreen, Symbol:OSHW-Symbol_13.4x12mm_SilkScreen, B.Cu at (154.9, 73.7)
- J19: moved to F.Cu
- moved J19 12.7 mm to (147.3, 141.0), turned to 180 degrees
- moved H1 12.7 mm to (111.8, 54.6)
- moved H4 12.7 mm to (111.8, 146.1)
- moved J25 7.62 mm to (91.4, 100.3)
- moved J10 5.08 mm to (81.3, 72.4)
- moved J11 5.08 mm to (81.3, 82.5)
- moved J12 5.08 mm to (81.3, 92.7)
- moved J13 5.08 mm to (81.3, 102.9)
- moved J14 5.08 mm to (81.3, 113.0)
- moved J15 5.08 mm to (81.3, 123.2)
- moved J16 5.08 mm to (81.3, 133.3)
- moved J9 5.08 mm to (81.3, 62.2)
- moved K1 2.54 mm to (117.0, 63.1)
- moved K2 2.54 mm to (117.0, 74.5)
- moved K3 2.54 mm to (117.0, 86.0)
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Connections:
- J19 pad 1: GND -> Net-(J18-Pad1)
- J19 pad 2: /SCL -> /SDA
- J19 pad 3: /SDA -> /SCL
- J19 pad 4: Net-(J18-Pad1) -> GND
- J25 pad 16: GND -> unconnected-(J25-Pin_16-Pad16)
- J25 pad 2: unconnected-(J25-Pin_2-Pad2) -> VDD
- K1 pad 4: GND -> VDD
- K2 pad 4: GND -> VDD
- K3 pad 4: GND -> VDD
- K4 pad 4: GND -> VDD
- K5 pad 4: GND -> VDD
- K6 pad 4: GND -> VDD
- K7 pad 4: GND -> VDD
- K8 pad 4: GND -> VDD
Routing:
- net /K8: track 126.4 -> 147.8 mm, vias 2 -> 0
- net Net-(U1-I3): track 29.0 -> 44.9 mm
- net /K7: track 113.8 -> 126.0 mm, vias 2 -> 0
- net Net-(U1-I5): track 26.5 -> 38.3 mm, vias 2 -> 0
- net /SDA: track 58.4 -> 69.6 mm
- net /SCL: track 61.3 -> 71.5 mm
- net Net-(U1-I7): track 36.2 -> 27.8 mm
- net /K3: track 70.7 -> 78.3 mm
- net /K2: track 68.4 -> 76.0 mm
- net /K1: track 68.6 -> 75.9 mm
- net /K4: track 79.0 -> 85.1 mm
- net /K5: track 89.3 -> 94.0 mm, vias 1 -> 0
- net /K6: track 105.0 -> 108.2 mm, vias 2 -> 0
- net Net-(U1-I4): track 29.4 -> 26.7 mm, vias 0 -> 2
- net Net-(J9-Pin_2): track 43.7 -> 46.2 mm
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Other:
- copper layers 4 -> 2
- board text added: "PM-RQ8-base v0.0.2"
- board text removed: "PM-RQ8-base v0.0.1"

Commit message: v0.0.2
Parts:
- removed J10, J11, J12, J13, J14, J15, J16, J9: 2EDGR-5.08-02P, NextPCB:Degson_2EDGR-5.08-02P
- added J17: 2EDGR-5.08-18P, NextPCB:Degson_2EDGR-5.08-18P, F.Cu at (81.3, 57.1)
Routing:
- net Net-(J17-Pin_13): track 43.5 -> 46.2 mm
- net Net-(J17-Pin_1): track 46.2 -> 43.5 mm
- net Net-(J17-Pin_15): track 44.1 -> 46.8 mm
- net Net-(J17-Pin_3): track 45.7 -> 43.6 mm
- net Net-(J17-Pin_11): track 43.6 -> 45.7 mm
- net Net-(J17-Pin_9): track 44.1 -> 45.2 mm
- net Net-(J17-Pin_5): track 45.2 -> 44.1 mm

Commit message: PM-CPU-RP
Parts:
- moved J18 1.27 mm to (160.0, 141.0)
- moved J19 1.27 mm to (146.1, 141.0)
Routing:
- net Net-(J17-Pin_2): track 37.1 -> 60.4 mm
- net Net-(U1-I3): track 44.9 -> 28.3 mm
- net Net-(U1-I4): track 26.7 -> 43.2 mm, vias 2 -> 0
- net /K8: track 147.8 -> 142.4 mm, vias 0 -> 1
- net /A0: track 21.3 -> 24.6 mm
- net Net-(J17-Pin_1): track 43.5 -> 45.2 mm
- net Net-(U1-I2): track 29.1 -> 27.8 mm
- net /SDA: track 69.6 -> 70.7 mm
- net Net-(U1-I1): track 28.7 -> 27.5 mm
- net GND: track 13.4 -> 14.4 mm
- net /SCL: track 71.5 -> 70.8 mm
- net /K7: track 126.0 -> 126.8 mm, vias 0 -> 1

Commit message: send to nextpcb
Routing:
- net Net-(U1-I3): track 28.3 -> 29.7 mm
- net Net-(U1-I2): track 27.8 -> 29.2 mm
- net Net-(U1-I1): track 27.5 -> 28.8 mm
Changed lines of the file:
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@@
-	)
-	(segment
-		(start 158.395 95.6674)
-		(end 154.94 92.2124)
-		(width 0.2)
-		(layer "F.Cu")
-		(net 13)
 	)
 	(segment
@@
 	)
 	(segment
-		(start 154.94 92.2124)
+		(start 158.395 95.6674)
+		(end 153.416 90.6884)
+		(width 0.2)
+		(layer "F.Cu")
+		(net 13)
+	)
+	(segment
+		(start 153.416 90.6884)
+		(end 153.416 72.289)
+		(width 0.2)
+		(layer "F.Cu")
+		(net 13)
+	)
+	(segment
+		(start 153.416 72.289)
 		(end 154.94 70.765)
 		(width 0.2)
@@
 	)
 	(segment
-		(start 155.9319 74.3614)
+		(start 154.216 76.0773)
 		(end 157.48 72.8133)
 		(width 0.2)
@@
 	)
 	(segment
-		(start 155.9319 91.9521)
-		(end 155.9319 74.3614)
+		(start 154.216 90.357028)
+		(end 154.216 76.0773)
+		(width 0.2)
+		(layer "F.Cu")
+		(net 18)
+	)
+	(segment
+		(start 159.695 95.836028)
+		(end 154.216 90.357028)
+		(width 0.2)
+		(layer "F.Cu")
+		(net 18)
+	)
+	(segment
+		(start 159.695 96.8425)
+		(end 159.695 95.836028)
 		(width 0.2)
 		(layer "F.Cu")
@@
 	)
 	(segment
-		(start 159.695 95.7152)
-		(end 155.9319 91.9521)
-		(width 0.2)
-		(layer "F.Cu")
-		(net 18)
-	)
-	(segment
-		(start 159.695 96.8425)
-		(end 159.695 95.7152)
-		(width 0.2)
-		(layer "F.Cu")
-		(net 18)
-	)
-	(segment
 		(start 163.83 70.765)
 		(end 163.83 78.0592)
@@
 	)
 	(segment
-		(start 159.045 95.6333)
-		(end 155.5032 92.0915)
+		(start 153.816 90.522714)
+		(end 153.816 74.7628)
+		(width 0.2)
+		(layer "F.Cu")
+		(net 22)
+	)
+	(segment
+		(start 153.816 74.7628)
+		(end 156.21 72.3688)
 		(width 0.2)
 		(layer "F.Cu")
@@
 	)
 	(segment
-		(start 155.5032 73.0756)
-		(end 156.21 72.3688)
+		(start 159.045 95.751714)
+		(end 153.816 90.522714)
 		(width 0.2)
 		(layer "F.Cu")
@@
 	)
 	(segment
-		(start 155.5032 92.0915)
-		(end 155.5032 73.0756)
-		(width 0.2)
-		(layer "F.Cu")
-		(net 22)
-	)
-	(segment
 		(start 159.045 96.8425)
-		(end 159.045 95.6333)
-		(width 0.2)
-		(layer "F.Cu")
+		(end 159.045 95.751714)
+		(width 0.2)
+		(layer "F.Cu")

Commit message: add docs
Other:
- board text removed: "0,0000 mm / 0,0000 mm"
- board text removed: "0,3000 mm"
- board text removed: "1,6000 mm"
- board text removed: "2"
- board text removed: "99,0600 mm x 99,0600 mm"
- board text removed: "None"
- board text removed: "Габариты платы:"
- board text removed: "Количество слоёв меди:"
- board text removed: "Контроль импеданса:"
- board text removed: "Краевой соединитель:"
- board text removed: "Метал. торцы:"
- board text removed: "Мин. дорожка/зазор:"
- board text removed: "Мин. сверло:"
- board text removed: "Нет"
- board text removed: "Периферийные полу-отверстия:"
- board text removed: "Покрытие меди:"
- board text removed: "Толщина платы:"
- board text removed: "ХАРАКТЕРИСТИКИ ПЛАТЫ"
