File: PM-DI16-front-DC24/PM-DI16-front-DC24.kicad_pcb (KiCad board)
At the start: 2 copper layers, 30.5 x 99.1 mm, 52 parts, among them J1 Conn_02x08_Odd_Even, J2 Conn_02x08_Odd_Even

Commit message: v0.0.1 send to nextpcb
Parts:
- moved R10 2.54 mm to (132.1, 104.1)
- moved R9 2.54 mm to (142.2, 104.1)
- moved J2 2.54 mm to (134.1, 124.5)
- moved R11 2.54 mm to (142.2, 109.2)
- moved R12 2.54 mm to (132.1, 109.2)
- moved R13 2.54 mm to (142.2, 139.7)
- moved R14 2.54 mm to (132.1, 139.7)
- moved R15 2.54 mm to (142.2, 144.8)
- moved R16 2.54 mm to (132.1, 144.8)
- renumbered REF** to logo_kicad, REF** to logo_oshw
Routing:
- net Net-(D20-A): track 54.6 -> 46.1 mm
- net Net-(D18-A): track 23.0 -> 31.4 mm
- net /OUT13: track 22.6 -> 15.2 mm
- net Net-(D14-K): track 37.4 -> 31.2 mm
- net Net-(D13-K): track 26.1 -> 20.2 mm
- net Net-(D11-K): track 20.5 -> 14.8 mm
- net /IN06: track 17.2 -> 22.9 mm
- net Net-(D22-A): track 45.1 -> 40.0 mm
- net Net-(D23-A): track 17.9 -> 21.2 mm
- net /OUT07: track 15.0 -> 18.1 mm
- net /OUT10: track 20.1 -> 23.0 mm, vias 2 -> 1
- net /OUT00: track 14.8 -> 17.7 mm
- net /OUT14: track 11.0 -> 13.6 mm
- net /OUT12: track 15.1 -> 17.6 mm
- net Net-(D17-A): track 12.0 -> 13.4 mm
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
Commit message: v0.0.2
Parts:
- removed J2: Conn_02x08_Odd_Even, NextPCB:Conn_02x08_pin_angle
- removed logo_kicad: KiCad-Logo2_5mm_SilkScreen, Symbol:KiCad-Logo2_5mm_SilkScreen
- removed logo_oshw: OSHW-Logo_5.7x6mm_SilkScreen, Symbol:OSHW-Logo_5.7x6mm_SilkScreen
- added Logo_kicad: KiCad-Logo2_5mm_SilkScreen, Symbol:KiCad-Logo2_5mm_SilkScreen, B.Cu at (152.4, 104.1)
- added REF**: OSHW-Symbol_6.7x6mm_SilkScreen, Symbol:OSHW-Symbol_6.7x6mm_SilkScreen, B.Cu at (152.4, 91.4)
- J1: value Conn_02x08_Odd_Even -> Conn_02x16_pin; footprint NextPCB:Conn_02x08_pin_angle -> NextPCB:Conn_02x16_pin
- moved R12 36.7 mm to (141.0, 144.8)
- moved R5 36.7 mm to (151.1, 55.9)
- moved R6 34.9 mm to (151.1, 62.2)
- moved R10 29.3 mm to (141.0, 132.1)
- moved R7 29.3 mm to (151.1, 68.6)
- moved R11 29.2 mm to (141.0, 138.4)
- moved R8 28.8 mm to (151.1, 74.9)
- moved J1 25.5 mm to (142.2, 100.3), turned to 180 degrees
- moved R9 21.6 mm to (141.0, 125.7)
- moved R14 20.5 mm to (151.1, 132.1)
- moved D10 20.3 mm to (132.1, 63.5)
- moved D11 20.3 mm to (132.1, 68.6)
- moved D12 20.3 mm to (132.1, 73.7)
- moved D13 20.3 mm to (132.1, 78.7)
- moved D14 20.3 mm to (132.1, 83.8)
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Connections:
- J1 pad 10: /OUT03 -> /IN04
- J1 pad 11: /IN02 -> /OUT05
- J1 pad 12: /OUT02 -> /IN05
- J1 pad 13: /IN01 -> /OUT06
- J1 pad 14: /OUT01 -> /IN06
- J1 pad 15: /IN00 -> /OUT07
- J1 pad 16: /OUT00 -> /IN07
Routing:
- net /IN12: track 13.8 -> 73.9 mm
- net /IN01: track 18.8 -> 69.3 mm
- net /IN04: track 16.7 -> 66.9 mm
- net /IN17: track 16.4 -> 59.1 mm
- net /IN10: track 14.4 -> 54.6 mm
- net /IN05: track 16.4 -> 56.2 mm
- net Net-(D15-K): track 15.5 -> 52.6 mm
- net Net-(D13-K): track 20.2 -> 52.4 mm
- net /IN06: track 22.9 -> 53.2 mm
- net Net-(D12-K): track 42.4 -> 12.9 mm
- net /IN07: track 16.4 -> 45.4 mm
- net /IN13: track 19.0 -> 47.4 mm
- net Net-(D19-A): track 10.9 -> 37.4 mm, vias 1 -> 2
- net /OUT02: track 11.0 -> 36.3 mm
- net /IN16: track 17.2 -> 42.1 mm
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- added copper zone on B.Cu, net (none)
- added copper zone on F.Cu, net (none)
Other:
- board text added: "PM-DI16-front-DC24 v0.0.2"
- board text removed: "PM-DI16-front-DC24 v0.0.1"

Commit message: InvenTree
Parts:
- D1, D17, D18, D19, D2, D20, D21, D22, D23, D24, D3, D4, D5, D6, D7, D8: value KPTD-3216ZGC -> KPT-3216CGCK; footprint NextPCB:LED_KPTD-3216ZGC -> NextPCB:Kingbright_KPT-3216CGCK
- J1: value Conn_02x16_pin -> PinHeader P2.54 02x16 SMD Straight
- R1, R10, R11, R12, R13, R14, R15, R16, R2, R3, R4, R5, R6, R7, R8, R9: value 1.1k 1W -> 2.2k
- moved D13 0.64 mm to (132.1, 79.4)
