File: PM-AI-IU4/PM-AI-IU4.kicad_pcb (KiCad board)
At the start: 2 copper layers, 99.1 x 99.1 mm, 8 parts, among them J1 PinHeader P2.54 01x08 THT Ang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, U1 64900001039

Commit message: PM-AU-IU4
Parts:
- added C1: 100nF 1206, Capacitor_SMD:C_1206_3216Metric_Pad1.33x1.80mm_HandSolder, F.Cu at (82.3, 94.0)
- added J11: 2EDGR-5.08-02P, NextPCB:Degson_2EDGR-5.08-02P, F.Cu at (30.5, 106.7)
- added J2: PinHeader P2.54 02x04 SMD Straight, Connector_PinHeader_2.54mm:PinHeader_2x04_P2.54mm_Vertical_SMD, F.Cu at (61.0, 102.2)
- added J4: 2EDGR-5.08-02P, NextPCB:Degson_2EDGR-5.08-02P, F.Cu at (30.5, 61.0)
- added J7: 2EDGR-5.08-02P, NextPCB:Degson_2EDGR-5.08-02P, F.Cu at (30.5, 76.2)
- added J9: 2EDGR-5.08-02P, NextPCB:Degson_2EDGR-5.08-02P, F.Cu at (30.5, 91.4)
- added U2: ADS1115, Package_SO:TSSOP-10_3x3mm_P0.5mm, F.Cu at (81.3, 101.6)
- moved U1 29.6 mm to (99.1, 96.5), turned to 180 degrees
Other:
- board text added: "+5V"
- board text added: "0x48"
- board text added: "0x49"
- board text added: "0x4A"
- board text added: "0x4B"
- board text added: "CLK"
- board text added: "CS"
- board text added: "GND"
- board text added: "MISO"
- board text added: "MOSI"
- board text added: "PM-AI-IU4 v0.0.1"
- board text added: "SCL"
- board text added: "SDA"
- board text added: "Адрес"
- board text removed: "PM-AI-IU v0.0.1"
