File: PM-AI8-IU-front-10V/PM-AI8-IU-front-10V.kicad_pcb (KiCad board)
At the start: 2 copper layers, 30.5 x 99.1 mm, 17 parts, among them J1 PinHeader P2.54 02x16 SMD Str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

Commit message: PM-AI-xxx docs
Other:
- board text added: "-"
Changed lines of the file:
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@@
+		)
+	)
+	(gr_text "-"
+		(at 54.502857 144.3815 0)
+		(layer "F.SilkS")
+		(effects
+			(font
+				(size 1.5 1.5)
+				(thickness 0.2)
+			)
+			(justify bottom)
 		)
 	)
@@
 		)
 	)
+	(gr_text "-"
+		(at 54.502857 139.3015 0)
+		(layer "F.SilkS")
+		(effects
+			(font
+				(size 1.5 1.5)
+				(thickness 0.2)
+			)
+			(justify bottom)
+		)
+	)
