File: PM-AI8-IU-front-5V/PM-AI8-IU-front-5V.kicad_sch (KiCad schematic)
At the start: 1 part, among them J1 PinHeader P2.54 02x16 SMD Str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

Commit message: PM-AI-xxx docs
Connections:
- net IN1: now reaches J1.1 (Pin_1), J1.2 (Pin_2)
- net IN5: now reaches J1.10 (Pin_10), J1.9 (Pin_9)
- net IN6: now reaches J1.11 (Pin_11), J1.12 (Pin_12)
- net IN7: now reaches J1.13 (Pin_13), J1.14 (Pin_14)
- net IN8: now reaches J1.15 (Pin_15), J1.16 (Pin_16)
- net +5V: now reaches J1.29 (Pin_29)
- net +5V: now also J1.30 (Pin_30)
- net IN2: now reaches J1.3 (Pin_3), J1.4 (Pin_4)
- net GND: now reaches J1.31 (Pin_31)
- net GND: now also J1.32 (Pin_32)
- net IN3: now reaches J1.5 (Pin_5), J1.6 (Pin_6)
- net IN4: now reaches J1.7 (Pin_7), J1.8 (Pin_8)
- no-connect marks 16 -> 12
