File: PM-AI1-W/PM-AI1-W.kicad_sch (KiCad schematic)
At the start: 52 parts, among them J1 2EDGR-5.08-18P, J3 Conn_01x04_Pin, J6 PinHeader_01x12_P2.54_THT_str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, J7 PinHeader_01x12_P2.54_THT_str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, Q1 BSH112, Q2 BSH201, Q4 BSH112, Q7 BSH201, SW1 DSIC05LS-P, U1 AD7195BCPZ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

Commit message: PM-AI1-W
Parts:
- removed J1: 2EDGR-5.08-18P, NextPCB:Degson_2EDGR-5.08-18P, symbol kicad_inventree_lib:Degson_2EDGR-5.08-18P
- added D2: B5819W, Diode_SMD:D_SOD-123, symbol kicad_inventree_lib:B5819W
- added J4: 2EDGR-5.08-08P, kicad_inventree_lib:Degson_2EDGR-5.08-08P, symbol kicad_inventree_lib:Degson_2EDGR-5.08-08P
Connections:
- net +5V: now also D2.2 (A); no longer J6.9 (Pin_9)
- net AD_REFIN(+): now also J4.2 (Pin_2)
- net AD_REFIN(-): now also J4.5 (Pin_5)
- net AGND: now also J4.7 (Pin_7), J4.8 (Pin_8)
- net EXC+: now also J4.1 (Pin_1)
- net EXC-: now also J4.4 (Pin_4)
- net SIG+: now also J4.3 (Pin_3)
- net SIG-: now also J4.6 (Pin_6)
- new net: D2.1 (K), J6.9 (Pin_9)

Commit message: PM-CPU-ESP
Parts:
- added J1: 2EDGK-5.08-08P, symbol kicad_inventree_lib:Degson_2EDGK-5.08-08P
Connections:
- no-connect marks 10 -> 18
Changed lines of the file:
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@@
 	)
 	(no_connect
+		(at 38.1 35.56)
+	)
+	(no_connect
 		(at 254 233.68)
 	)
@@
 	)
 	(no_connect
+		(at 38.1 30.48)
+	)
+	(no_connect
 		(at 254 228.6)
 	)
@@
 	)
 	(no_connect
+		(at 38.1 40.64)
+	)
+	(no_connect
+		(at 38.1 33.02)
+	)
+	(no_connect
+		(at 38.1 38.1)
+	)
+	(no_connect
 		(at 254 236.22)
 	)
 	(no_connect
+		(at 38.1 25.4)
+	)
+	(no_connect
+		(at 38.1 43.18)
+	)
+	(no_connect
 		(at 195.58 129.54)
 	)
@@
 	)
 	(no_connect
+		(at 38.1 27.94)
+	)
+	(no_connect
 		(at 254 231.14)
 	)
@@
 	)
 	(symbol
+		(lib_id "kicad_inventree_lib:Degson_2EDGK-5.08-08P")
+		(at 40.64 25.4 0)
+		(mirror y)
+		(unit 1)
+		(exclude_from_sim no)
+		(in_bom yes)
+		(on_board no)
+		(dnp no)
+		(property "Reference" "J1"
+			(at 40.64 20.32 0)
+			(effects
+				(font
+					(size 1.27 1.27)
+				)
+				(justify right)
+			)
+		)
+		(property "Value" "2EDGK-5.08-08P"
+			(at 26.416 22.86 0)
+			(effects
+				(font
+					(size 1.27 1.27)
+				)
+				(justify right)
+			)
+		)
+		(property "Footprint" ""
+			(at 38.1 25.4 0)
+			(effects
+				(font
+					(size 1.27 1.27)
+				)
+				(hide yes)
+			)
+		)
+		(property "Datasheet" "http://inventree.network/part/97/"
+			(at 38.1 25.4 0)
+			(effects
+				(font
+					(size 1.27 1.27)
+				)
+				(hide yes)
+			)
+		)
+		(property "Description" "Generic connector, single row, 01x02, script generated"
+			(at 38.1 25.4 0)
+			(effects
+				(font
+					(size 1.27 1.27)
+				)
+				(hide yes)
+			)
+		)
+		(property "part_ipn" "2EDGK-5.08-08P"
+			(at 40.64 25.4 0)
+			(effects
+				(font
+					(size 1.27 1.27)
+				)
+				(hide yes)
+			)
+		)
+		(pin "1"
+		)
+		(pin "2"
+		)
+		(pin "3"
+		)
+		(pin "4"
+		)
+		(pin "7"
+		)
+		(pin "5"
+		)
+		(pin "8"
+		)
+		(pin "6"
+		)
+		(instances
+			(project ""
+				(path "/3e910c54-7792-4c2e-8497-3f8a0979c787"
+					(reference "J1")
+					(unit 1)
+				)
+			)
+		)
+	)
+	(symbol
 		(lib_id "power:GND")
 		(at 172.72 83.82 0)
@@
 		(on_board yes)
 		(dnp no)
-		(fields_autoplaced yes)
 		(property "Reference" "J4"
 			(at 46.355 20.32 0)
@@
 		)
 		(property "Value" "2EDGR-5.08-08P"
-			(at 46.355 22.86 0)
+			(at 54.102 22.86 0)
 			(effects
 				(font
