File: PM-CPU-ESP/PM-CPU-ESP.kicad_sch (KiCad schematic)
At the start: 6 parts, among them J1 Conn_01x12_Pin, J2 Conn_01x12_Pin

Commit message: sync
Parts:
- added J3: Conn_02x08_Odd_Even, Connector_PinSocket_2.54mm:PinSocket_2x08_P2.54mm_Vertical_SMD, symbol Connector_Generic:Conn_02x08_Odd_Even
- added PS1: IRM-15-5, NextPCB:Meanwell-IRM-15-5_CONV_IRM-15-5, symbol NextPCB:Meanwell-IRM-15-5

Commit message: PM-CPU-ESP-front
Parts:
- removed J3: Conn_02x08_Odd_Even, Connector_PinSocket_2.54mm:PinSocket_2x08_P2.54mm_Vertical_SMD, symbol Connector_Generic:Conn_02x08_Odd_Even
- added IC1: USR-ES1, NextPCB:USRES1, symbol NextPCB:USR-ES1
- added J10, J11, J4, J9: 2EDGR-5.08-02P, NextPCB:Degson_2EDGR-5.08-02P, symbol NextPCB:Degson_2EDGR-5.08-02P
- added J3: Conn_02x08_socket, Connector_PinSocket_2.54mm:PinSocket_2x08_P2.54mm_Vertical_SMD, symbol NextPCB:Conn_02x08_socket
- added J5, J7: PHR-4, symbol NextPCB:JST_PHR-4
- added J6, J8: S4B-PH-SM4-TB, NextPCB:JST_S4B-PH-SM4-TB_JST_S4B-PH-SM4-TB, symbol NextPCB:JST_S4B-PH-SM4-TB
- added R1, R2: 3k3, Resistor_SMD:R_1206_3216Metric_Pad1.30x1.75mm_HandSolder, symbol NextPCB:R_3k3_0.25W
- added U1, U2: 64900001039, NextPCB:Fuseholder, symbol NextPCB:Fuseholder
- added U3: DS3231M, Package_SO:SOIC-16W_7.5x10.3mm_P1.27mm, symbol Timer_RTC:DS3231M
Connections:
- net +3.3V: now also IC1.B2 (3V3_1), IC1.B3 (3V3_2), J10.1 (Pin_1), R1.1, R2.1
- net +5V: now also J6.1, J8.1, J9.1 (Pin_1), U2.1, U3.2 (VCC)
- net GND: now also PS1.-V, J10.2 (Pin_2), J11.1 (Pin_1), J6.2, J6.4, J8.2, J8.4, J9.2 (Pin_2), R1.2, U3.10 (GND), U3.11 (GND), U3.12 (GND), U3.13 (GND), U3.16 (SCL), U3.5 (GND), U3.6 (GND), U3.7 (GND), U3.8 (GND), U3.9 (GND)
- net at PS1.+V: now also U2.2
- net at PS1.AC/L: now also U1.1
- net at PS1.AC/N: now also J4.2 (Pin_2)
- new net: J4.1 (Pin_1), U1.2
- new net SCL: J11.2 (Pin_2), J6.3, J8.3, R2.2, U3.15 (SDA)
- no-connect marks 9 -> 17
Other:
- note added: "CHIP_EN"
- note added: "GPIO10"
- note added: "GPIO18"
- note added: "GPIO19"
- note added: "GPIO8"
- note added: "GPIO9"
- note added: "U0RXD"
- note added: "U0TXD"
- note added: "VDD33"
- note added: "Подключение внутренней шины"
- moved on the sheet: J1, J2, PS1

Commit message: PM-CPU-ESP
Parts:
- added D1: B5819W, Diode_SMD:D_SOD-123, symbol NextPCB:B5819W
- added J12: ~, NextPCB:XKB_U224-08XN-1WR61, symbol NextPCB:XKB_U224-08XN-1WR61
- added U4: ESP32-C3, symbol NextPCB:Weact_Esp32-C3
- IC1: NextPCB_price (none) -> 4; NextPCB_url (none) -> https://aliexpress.ru/item/1005004860988013.html?spm=a2g2w.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
Connections:
- net +3.3V: now also J3.3 (Pin_3)
- net +5V: now also J3.1 (Pin_1), D1.2 (A), J12.1 (5V), J12.5 (5V); no longer J1.9 (Pin_9)
- net GND: now also IC1.A1 (GND_1), IC1.A2 (GND_2), IC1.B1 (GND_3), J3.15 (Pin_15), J12.4 (GND), J12.8 (GND); no longer J11.1 (Pin_1), J6.2, J8.2, R1.2, U3.16 (SCL)
- net N: now reaches J3.16 (Pin_16)
- net N: now also J4.2 (Pin_2), PS1.AC/N
- net L: now reaches J3.2 (Pin_2)
- net L: now also PS1.AC/L, U1.1
- new net: D1.1 (K), J1.9 (Pin_9)
- new net SDA: J11.1 (Pin_1), J6.2, J8.2, R1.2, U3.16 (SCL)
- no-connect marks 17 -> 42
Other:
- note added: "ESP32"
- note added: "USB (только питание внешних устройств)"
- note added: "W5500 - модуль Ethernet для ESP32"
- note added: "Часы реального времени"
- note removed: "CHIP_EN"
- note removed: "GND"
- note removed: "GPIO0"
- note removed: "GPIO1"
- note removed: "GPIO10"
- note removed: "GPIO18"
- note removed: "GPIO19"
- note removed: "GPIO2"
- note removed: "GPIO3"
- note removed: "GPIO4"
- note removed: "GPIO5"
- note removed: "GPIO6"
- note removed: "GPIO7"
- note removed: "GPIO8"
- note removed: "GPIO9"
- note removed: "U0RXD"
- note removed: "U0TXD"
- note removed: "VB"
- note removed: "VDD33"
- note removed: "VDD5V"
- moved on the sheet: H1, H2, H3, H4, IC1, J1, J2, J3, J5, J6, J7, J8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

Commit message: calculation
Parts:
- removed J1, J2: Conn_01x12_Pin, Connector_PinHeader_2.54mm:PinHeader_1x12_P2.54mm_Vertical, symbol Connector:Conn_01x12_Pin
- removed PS1: IRM-15-5, NextPCB:Meanwell-IRM-15-5_CONV_IRM-15-5, symbol NextPCB:Meanwell-IRM-15-5
- removed U3: DS3231M, Package_SO:SOIC-16W_7.5x10.3mm_P1.27mm, symbol Timer_RTC:DS3231M
- added J13, J2: Conn_01x12_pin, Connector_PinHeader_2.54mm:PinHeader_1x12_P2.54mm_Vertical, symbol NextPCB:Conn_01x12_pin
- added PS1: IRM-20-5, NextPCB:Meanwell-IRM-20-5, symbol NextPCB:Meanwell-IRM-20-5
- added U3: DS3231, Package_SO:SOIC-16W_7.5x10.3mm_P1.27mm, symbol NextPCB:DS3231
Connections:
- net +3.3V: now also J13.10 (Pin_10), J13.9 (Pin_9)
- net +5V: now also U3.2 (VCC)
- net GND: now also J13.11 (Pin_11), J13.12 (Pin_12), J2.11 (Pin_11), J2.12 (Pin_12), PS1.-V, U3.10 (GND), U3.11 (GND), U3.12 (GND), U3.13 (GND), U3.5 (GND), U3.6 (GND), U3.7 (GND), U3.8 (GND), U3.9 (GND)
- net L: now also PS1.AC/L
- net N: now also PS1.AC/N
- net SCL: now also J2.8 (Pin_8), U3.15 (SDA)
- net SDA: now also J2.7 (Pin_7), U3.16 (SCL)
- net at U2.2: now also PS1.+V
- net at D1.1 (K): now also J2.9 (Pin_9)
- no-connect marks 42 -> 40
Other:
- moved on the sheet: D1

Commit message: docs
Other:
- added sheet external_connection (external_connection.kicad_sch)
Changed lines of the file:
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@@
+		)
+	)
+	(sheet
+		(at 327.66 139.7)
+		(size 38.1 25.4)
+		(fields_autoplaced yes)
+		(stroke
+			(width 0.1524)
+			(type solid)
+		)
+		(fill
+			(color 0 0 0 0.0000)
+		)
+		(property "Sheetname" "external_connection"
+			(at 327.66 138.9884 0)
+			(effects
+				(font
+					(size 1.27 1.27)
+				)
+				(justify left bottom)
+			)
+		)
+		(property "Sheetfile" "external_connection.kicad_sch"
+			(at 327.66 165.6846 0)
+			(effects
+				(font
+					(size 1.27 1.27)
+				)
+				(justify left top)
+			)
+		)
+		(instances
+			(project "PM-CPU-ESP"
+				(path "/b2288a30-52a2-458e-b2e2-58b3f8400513"
+					(page "2")
+				)
+			)
 		)
 	)

Commit message: PM_Bus
Parts:
- removed D1: B5819W, Diode_SMD:D_SOD-123, symbol NextPCB:B5819W
- removed IC1: USR-ES1, NextPCB:USRES1, symbol NextPCB:USR-ES1
- removed J12: ~, NextPCB:XKB_U224-08XN-1WR61, symbol NextPCB:XKB_U224-08XN-1WR61
- removed PS1: IRM-20-5, NextPCB:Meanwell-IRM-20-5, symbol NextPCB:Meanwell-IRM-20-5
- removed R1, R2: 3k3, Resistor_SMD:R_1206_3216Metric_Pad1.30x1.75mm_HandSolder, symbol NextPCB:R_3k3_0.25W
- added D2: B5819W, Diode_SMD:D_SOD-123, symbol kicad_inventree_lib:B5819W
- added IC2: USR-ES1, NextPCB:USRES1, symbol kicad_inventree_lib:USR-ES1
- added J1: ~, NextPCB:XKB_U224-08XN-1WR61, symbol kicad_inventree_lib:XKB_U224-08XN-1WR61
- added PS2: IRM-20-5, NextPCB:Meanwell-IRM-20-5, symbol kicad_inventree_lib:Meanwell-IRM-20-5
- added R1, R2: 3k3, Resistor_SMD:R_1206_3216Metric_Pad1.30x1.75mm_HandSolder, symbol kicad_inventree_lib:R_3k3_1206_1%
Connections:
- net +3.3V: now also IC2.B2 (3V3_1), IC2.B3 (3V3_2), R1.1, R2.1
- net +5V: now also D2.2 (A), J1.1 (5V), J1.5 (5V)
- net GND: now also IC2.A1 (GND_1), IC2.A2 (GND_2), IC2.B1 (GND_3), J1.4 (GND), J1.8 (GND), PS2.-V
- net L: now also PS2.AC/L
- net N: now also PS2.AC/N
- net SCL: now also R2.2
- net SDA: now also R1.2
- net at J2.9 (Pin_9): now also D2.1 (K)
- net at U2.2: now also PS2.+V

Commit message: InvenTree
Parts:
- removed J13, J2: Conn_01x12_pin, Connector_PinHeader_2.54mm:PinHeader_1x12_P2.54mm_Vertical, symbol NextPCB:Conn_01x12_pin
- removed J3: Conn_02x08_socket, Connector_PinSocket_2.54mm:PinSocket_2x08_P2.54mm_Vertical_SMD, symbol NextPCB:Conn_02x08_socket
- removed J5, J7: PHR-4, symbol NextPCB:JST_PHR-4
- removed J6, J8: S4B-PH-SM4-TB, NextPCB:JST_S4B-PH-SM4-TB_JST_S4B-PH-SM4-TB, symbol NextPCB:JST_S4B-PH-SM4-TB
- removed U1, U2: 64900001039, NextPCB:Fuseholder, symbol NextPCB:Fuseholder
- added J12: PinHeader P2.54 01x08 THT Angle, Connector_PinHeader_2.54mm:PinHeader_1x08_P2.54mm_Horizontal, symbol kicad_inventree_lib:PinHeader P2.54 01x08 THT Angle
- added J2, J3: PinHeader P2.54 01x12 THT Straight, Connector_PinHeader_2.54mm:PinHeader_1x12_P2.54mm_Vertical, symbol kicad_inventree_lib:PinHeader P2.54 01x12 THT Straight
- added J5: FemaleHeader P2.54 02x08 SMD Straight, Connector_PinSocket_2.54mm:PinSocket_2x08_P2.54mm_Vertical_SMD, symbol kicad_inventree_lib:FemaleHeader P2.54 02x08 SMD Straight
- added U5, U6: 64900001039, NextPCB:Fuseholder, symbol kicad_inventree_lib:Fuseholder
Connections:
- net +3.3V: now also J3.10 (Pin_10), J3.9 (Pin_9), J5.3 (Pin_3)
- net +5V: now also J5.1 (Pin_1), U6.2
- net GND: now also J12.2 (Pin_2), J2.11 (Pin_11), J2.12 (Pin_12), J3.11 (Pin_11), J3.12 (Pin_12), J5.15 (Pin_15)
- net L: now also J5.2 (Pin_2), U5.2
- net N: now also J5.16 (Pin_16)
- net SCL: now also J12.4 (Pin_4), J2.8 (Pin_8)
- net SDA: now also J12.3 (Pin_3), J2.7 (Pin_7)
- net at D2.1 (K): now also J2.9 (Pin_9)
- net at PS2.+V: now also U6.1
- net at J4.1 (Pin_1): now also U5.1
- new net VDD: J12.1 (Pin_1)
- no-connect marks 40 -> 36

Commit message: PM-CPU-ESP
Parts:
- removed J10, J11, J4, J9: 2EDGR-5.08-02P, NextPCB:Degson_2EDGR-5.08-02P, symbol NextPCB:Degson_2EDGR-5.08-02P
- removed J12: PinHeader P2.54 01x08 THT Angle, Connector_PinHeader_2.54mm:PinHeader_1x08_P2.54mm_Horizontal, symbol kicad_inventree_lib:PinHeader P2.54 01x08 THT Angle
- removed J5: FemaleHeader P2.54 02x08 SMD Straight, Connector_PinSocket_2.54mm:PinSocket_2x08_P2.54mm_Vertical_SMD, symbol kicad_inventree_lib:FemaleHeader P2.54 02x08 SMD Straight
- removed PS2: IRM-20-5, NextPCB:Meanwell-IRM-20-5, symbol kicad_inventree_lib:Meanwell-IRM-20-5
- removed U6: 64900001039, NextPCB:Fuseholder, symbol kicad_inventree_lib:Fuseholder
- added C1, C2: 22uF, kicad_inventree_lib:C_2220_5750Metric_Pad1.97x5.40mm_HandSolder, symbol kicad_inventree_lib:C_22uF_50V_2220
- added J10, J11, J4, J9: 2EDGK-5.08-02P, symbol kicad_inventree_lib:Degson_2EDGK-5.08-02P
- added J12: ~, kicad_inventree_lib:PM-front-02x08, symbol kicad_inventree_lib:PM-front-02x08
- added J6: K7805-2000R3, kicad_inventree_lib:K7805-2000R3, symbol kicad_inventree_lib:K7805-2000R3
- added J7: Conn_01x04_Pin, Connector_PinHeader_2.54mm:PinHeader_1x04_P2.54mm_Horizontal, symbol kicad_inventree_lib:PinHeader P2.54 01x04 THT Angle
- added J8: 2EDGR-5.08-08P, kicad_inventree_lib:Degson_2EDGR-5.08-08P, symbol kicad_inventree_lib:Degson_2EDGR-5.08-08P
- added R3, R4, R5, R6: 100, Resistor_SMD:R_1206_3216Metric_Pad1.30x1.75mm_HandSolder, symbol kicad_inventree_lib:R_100_1206_1%
Connections:
- net +3.3V: now also J12.6, J8.5 (Pin_5)
- net +5V: now also C2.1, J12.4, J6.3 (+VO), J7.1 (Pin_1), J8.3 (Pin_3)
- net GND: now also C1.2, C2.2, J12.16, J6.2 (GND), J7.2 (Pin_2), J8.2 (Pin_2), J8.4 (Pin_4), J8.6 (Pin_6)
- net SCL: now also J2.2 (Pin_2), J7.4 (Pin_4), J8.8 (Pin_8); no longer J2.8 (Pin_8)
- net SDA: now also J2.1 (Pin_1), J7.3 (Pin_3), J8.7 (Pin_7); no longer J2.7 (Pin_7)
- net at J2.3 (Pin_3): now also R4.2
- net MISO: now reaches J2.4 (Pin_4)
- net MISO: now also R3.2
- net at J2.5 (Pin_5): now also R5.2
- net at J2.6 (Pin_6): now also R6.2
- net 24V_IN: now reaches U5.1
- net 24V_IN: now also J8.1 (Pin_1)
- net MOSI: now reaches IC2.A3 (MOSI)
- net MOSI: now also R4.1
- net CLK: now reaches IC2.A4 (SCLK)
- net CLK: now also R5.1
- net CS: now reaches IC2.A5 (CS)
- net CS: now also R6.1
- net RST: now reaches IC2.B5 (RST)
- net RST: now also J2.7 (Pin_7)
- net at IC2.B6 (MISO): now also R3.1
- net L renamed +24V
- net +24V: now also C1.1, J12.2, J6.1 (VIN)
- no-connect marks 36 -> 38
Other:
- note added: "Подключение фронтальной платы"
- note added: "Подтяжка I2C"
- note added: "Регулятор напряжения"
- moved on the sheet: D2, IC2, J1, J2, J3, R1, R2, U3, U4, U5
