File: PM-AI8-I/PM-AI8-I.kicad_pcb (KiCad board)
At the start: 2 copper layers, 99.1 x 99.1 mm, 2 parts, among them J1 2EDGR-5.08-18P, U1 AD4111BCPZ

Commit message: PM-DI16-DC24sink
Parts:
- added C1: 4.7 nF, Capacitor_SMD:C_1206_3216Metric_Pad1.33x1.80mm_HandSolder, F.Cu at (76.2, 114.3)
- added D1: SMAJ33CA, Diode_SMD:D_SMA, F.Cu at (58.4, 113.0)
- added R1: 180R, Resistor_SMD:R_1206_3216Metric_Pad1.30x1.75mm_HandSolder, F.Cu at (57.4, 119.4)
- moved U1 7.66 mm to (101.3, 86.6)
Connections:
- J1 pad 10: unconnected-(J1-Pin_10-Pad10) -> FGND
- J1 pad 12: unconnected-(J1-Pin_12-Pad12) -> FGND
- J1 pad 14: unconnected-(J1-Pin_14-Pad14) -> FGND
- J1 pad 16: unconnected-(J1-Pin_16-Pad16) -> FGND
- J1 pad 2: unconnected-(J1-Pin_2-Pad2) -> FGND
- J1 pad 4: unconnected-(J1-Pin_4-Pad4) -> FGND
- J1 pad 6: unconnected-(J1-Pin_6-Pad6) -> FGND
- J1 pad 8: unconnected-(J1-Pin_8-Pad8) -> FGND
- U1 pad 11: unconnected-(U1A-VBIAS--Pad11) -> FGND
- U1 pad 30: unconnected-(U1A-IIN3--Pad30) -> FGND
- U1 pad 31: unconnected-(U1A-IIN2--Pad31) -> FGND
- U1 pad 32: unconnected-(U1A-IIN1--Pad32) -> FGND
- U1 pad 33: unconnected-(U1A-IIN0--Pad33) -> FGND
- U1 pad 41: unconnected-(U1A-EPAD-Pad41) -> AVSS
- U1 pad 8: unconnected-(U1B-AVSS-Pad8) -> AVSS

Commit message: PM-AI8-I
Parts:
- added C10: 100nF, Capacitor_SMD:C_1206_3216Metric_Pad1.33x1.80mm_HandSolder, F.Cu at (91.4, 83.8)
- added C11: 100nF, Capacitor_SMD:C_1206_3216Metric_Pad1.33x1.80mm_HandSolder, F.Cu at (91.4, 91.4)
- added C12: 1uF, Capacitor_SMD:C_1206_3216Metric_Pad1.33x1.80mm_HandSolder, F.Cu at (86.4, 91.4)
- added C2: 4.7 nF, Capacitor_SMD:C_1206_3216Metric_Pad1.33x1.80mm_HandSolder, F.Cu at (68.7, 54.5)
- added C3: 4.7 nF, Capacitor_SMD:C_1206_3216Metric_Pad1.33x1.80mm_HandSolder, F.Cu at (68.7, 57.8)
- added C4: 4.7 nF, Capacitor_SMD:C_1206_3216Metric_Pad1.33x1.80mm_HandSolder, F.Cu at (68.7, 61.2)
- added C5: 4.7 nF, Capacitor_SMD:C_1206_3216Metric_Pad1.33x1.80mm_HandSolder, F.Cu at (68.7, 64.5)
- added C6: 4.7 nF, Capacitor_SMD:C_1206_3216Metric_Pad1.33x1.80mm_HandSolder, F.Cu at (68.7, 67.9)
- added C7: 4.7 nF, Capacitor_SMD:C_1206_3216Metric_Pad1.33x1.80mm_HandSolder, F.Cu at (68.7, 71.2)
- added C8: 4.7 nF, Capacitor_SMD:C_1206_3216Metric_Pad1.33x1.80mm_HandSolder, F.Cu at (68.7, 74.6)
- added C9: 4.7 nF, Capacitor_SMD:C_1206_3216Metric_Pad1.33x1.80mm_HandSolder, F.Cu at (87.4, 62.7)
- added D2: SMAJ33CA, Diode_SMD:D_SMA, F.Cu at (61.6, 55.1)
- added D3: SMAJ33CA, Diode_SMD:D_SMA, F.Cu at (61.6, 59.6)
- added D4: SMAJ33CA, Diode_SMD:D_SMA, F.Cu at (61.6, 64.2)
- added D5: SMAJ33CA, Diode_SMD:D_SMA, F.Cu at (61.6, 68.7)
- added D6: SMAJ33CA, Diode_SMD:D_SMA, F.Cu at (61.6, 73.3)
- added D7: SMAJ33CA, Diode_SMD:D_SMA, F.Cu at (61.6, 77.8)
- added D8: SMAJ33CA, Diode_SMD:D_SMA, F.Cu at (61.6, 82.4)
- added D9: SMAJ33CA, Diode_SMD:D_SMA, F.Cu at (61.6, 86.9)
- added R2: 180R, Resistor_SMD:R_1206_3216Metric_Pad1.30x1.75mm_HandSolder, F.Cu at (74.7, 54.4)
- added R3: 180R, Resistor_SMD:R_1206_3216Metric_Pad1.30x1.75mm_HandSolder, F.Cu at (74.7, 57.7)
- added R4: 180R, Resistor_SMD:R_1206_3216Metric_Pad1.30x1.75mm_HandSolder, F.Cu at (74.7, 61.0)
- added R5: 180R, Resistor_SMD:R_1206_3216Metric_Pad1.30x1.75mm_HandSolder, F.Cu at (74.7, 64.3)
- added R6: 180R, Resistor_SMD:R_1206_3216Metric_Pad1.30x1.75mm_HandSolder, F.Cu at (74.7, 67.6)
- added R7: 180R, Resistor_SMD:R_1206_3216Metric_Pad1.30x1.75mm_HandSolder, F.Cu at (74.7, 70.9)
- added R8: 180R, Resistor_SMD:R_1206_3216Metric_Pad1.30x1.75mm_HandSolder, F.Cu at (74.7, 74.2)
- added R9: 180R, Resistor_SMD:R_1206_3216Metric_Pad1.30x1.75mm_HandSolder, F.Cu at (87.3, 66.0)
- moved R1 61.6 mm to (48.3, 58.4)
- moved C1 57.1 mm to (55.9, 61.0), turned to -90 degrees
- moved D1 50.6 mm to (48.3, 63.5), turned to 180 degrees
Connections:
- C1 pad 1: /voltage_input/VCOM -> /AD_VIN0
- D1 pad 2: FGND -> /voltage_input/IN01
- J1 pad 1: unconnected-(J1-Pin_1-Pad1) -> /voltage_input/IN01
- J1 pad 11: unconnected-(J1-Pin_11-Pad11) -> /voltage_input/IN06
- J1 pad 13: unconnected-(J1-Pin_13-Pad13) -> /voltage_input/IN07
- J1 pad 15: unconnected-(J1-Pin_15-Pad15) -> /voltage_input/IN08
- J1 pad 3: unconnected-(J1-Pin_3-Pad3) -> /voltage_input/IN02
- J1 pad 5: unconnected-(J1-Pin_5-Pad5) -> /voltage_input/IN03
- J1 pad 7: unconnected-(J1-Pin_7-Pad7) -> /voltage_input/IN04
- J1 pad 9: unconnected-(J1-Pin_9-Pad9) -> /voltage_input/IN05
- R1 pad 1: FGND -> /voltage_input/IN01
- R1 pad 2: /voltage_input/VCOM -> /AD_VIN0
- U1 pad 1: unconnected-(U1-VINCOM-Pad1) -> /AD_VINCOM
- U1 pad 2: unconnected-(U1-VIN0-Pad2) -> /AD_VIN0
- U1 pad 26: unconnected-(U1-VIN4-Pad26) -> /AD_VIN4
- U1 pad 27: unconnected-(U1-VIN5-Pad27) -> /AD_VIN5
- U1 pad 28: unconnected-(U1-VIN6-Pad28) -> /AD_VIN6
- U1 pad 29: unconnected-(U1-VIN7-Pad29) -> /AD_VIN7
- U1 pad 3: unconnected-(U1-VIN1-Pad3) -> /AD_VIN1
- U1 pad 4: unconnected-(U1-VION2-Pad4) -> /AD_VIN2
- U1 pad 41: AVSS -> FGND
- U1 pad 5: unconnected-(U1-VIN3-Pad5) -> /AD_VIN3
- U1 pad 6: unconnected-(U1-REFOUT-Pad6) -> Net-(U1-REFOUT)
- U1 pad 7: unconnected-(U1-REGCAPA-Pad7) -> Net-(U1-REGCAPA)
- U1 pad 8: AVSS -> FGND
