File: PM-AI8-I/voltage_input.kicad_sch (KiCad schematic)
At the start: 6 parts

Commit message: PM-AI8-I
Parts:
- added C2, C3, C4, C5, C6, C7, C8: 4.7 nF, Capacitor_SMD:C_1206_3216Metric_Pad1.33x1.80mm_HandSolder, symbol kicad_inventree_lib:C_4.7nF_50V_1206
- added D2, D3, D4, D5, D6, D7, D8: SMAJ33CA, Diode_SMD:D_SMA, symbol Diode:SMAJ33CA
- added R2, R3, R4, R5, R6, R7, R8: 180R, Resistor_SMD:R_1206_3216Metric_Pad1.30x1.75mm_HandSolder, symbol kicad_inventree_lib:R_180R_1206_1%
- renumbered C24 to C1, C1 to C9, D9 to D1, D1 to D9, R17 to R1, R1 to R9
Connections:
- net -: now also C2.2, C4.2, C5.2, C6.2, C7.2, C8.2, D2.1 (A1), D4.1 (A1), D5.1 (A1), D6.1 (A1), D7.1 (A1), D8.1 (A1)
- net IN02: now also D2.2 (A2), R2.1
- net IN03: now also D3.2 (A2), R3.1
- net IN04: now also D4.2 (A2), R4.1
- net IN05: now also D5.2 (A2), R5.1
- net IN06: now also D6.2 (A2), R6.1
- net IN07: now also D7.2 (A2), R7.1
- net IN08: now also D8.2 (A2), R8.1
- new net: C3.2, D3.1 (A1)
- new net OUT02: C2.1, R2.2
- new net OUT03: C3.1, R3.2
- new net OUT04: C4.1, R4.2
- new net OUT05: C5.1, R5.2
- new net OUT06: C6.1, R6.2
- new net OUT07: C7.1, R7.2
- new net OUT08: C8.1, R8.2
Other:
- moved on the sheet: C1, C9, D1, D9, R1, R9
