File: PM-AI8-U/isolation.kicad_sch (KiCad schematic)
At the start: 5 parts, among them U2 CA-IS3641HW

Commit message: send to nextpcb
Parts:
- C14, C16: footprint Capacitor_SMD:C_1206_3216Metric_Pad1.33x1.80mm_HandSolder -> Capacitor_SMD:C_1210_3225Metric_Pad1.33x2.70mm_HandSolder; symbol kicad_inventree_lib:C_10uF_50V_1206 -> kicad_inventree_lib:C_10uF_50V_1210; part_ipn C_10uF_50V_1206 -> C_10uF_50V_1210
- U2: part_ipn http://inventree.network/part/115/ -> CA-IS3641HW
Changed lines of the file:
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@@
+	(wire
+		(pts
+			(xy 127 91.44) (xy 132.08 91.44)
+		)
+		(stroke
+			(width 0)
+			(type default)
+		)
+	)
 	(wire
 		(pts
@@
 		(pts
 			(xy 88.9 99.06) (xy 101.6 99.06)
-		)
-		(stroke
-			(width 0)
-			(type default)
-		)
-	)
-	(wire
-		(pts
-			(xy 127 91.44) (xy 132.08 91.44)
 		)
 		(stroke
@@
 	)
 	(symbol
-		(lib_id "kicad_inventree_lib:C_10uF_50V_1206")
+		(lib_id "kicad_inventree_lib:C_10uF_50V_1210")
 		(at 203.2 90.17 0)
 		(unit 1)
@@
 			)
 		)
-		(property "Footprint" "Capacitor_SMD:C_1206_3216Metric_Pad1.33x1.80mm_HandSolder"
+		(property "Footprint" "Capacitor_SMD:C_1210_3225Metric_Pad1.33x2.70mm_HandSolder"
 			(at 204.1652 93.98 0)
 			(effects
@@
 			)
 		)
-		(property "Datasheet" "http://inventree.network/part/116/"
+		(property "Datasheet" "http://inventree.network/part/125/"
 			(at 203.2 90.17 0)
 			(effects
@@
 			)
 		)
-		(property "part_ipn" "C_10uF_50V_1206"
+		(property "part_ipn" "C_10uF_50V_1210"
 			(at 203.2 90.17 0)
 			(effects
@@
 	)
 	(symbol
-		(lib_id "kicad_inventree_lib:C_10uF_50V_1206")
+		(lib_id "kicad_inventree_lib:C_10uF_50V_1210")
 		(at 101.6 90.17 0)
 		(unit 1)
@@
 			)
 		)
-		(property "Footprint" "Capacitor_SMD:C_1206_3216Metric_Pad1.33x1.80mm_HandSolder"
+		(property "Footprint" "Capacitor_SMD:C_1210_3225Metric_Pad1.33x2.70mm_HandSolder"
 			(at 102.5652 93.98 0)
 			(effects
@@
 			)
 		)
-		(property "Datasheet" "http://inventree.network/part/116/"
+		(property "Datasheet" "http://inventree.network/part/125/"
 			(at 101.6 90.17 0)
 			(effects
@@
 			)
 		)
-		(property "part_ipn" "C_10uF_50V_1206"
+		(property "part_ipn" "C_10uF_50V_1210"
 			(at 101.6 90.17 0)
 			(effects
@@
 			)
 		)
-		(property "part_ipn" "http://inventree.network/part/115/"
+		(property "part_ipn" "CA-IS3641HW"
 			(at 152.146 107.442 0)
 			(effects
