File: PM-AI8-U/voltage_input.kicad_sch (KiCad schematic)
At the start: 27 parts

Commit message: PM-AI8-U
Parts:
- removed C9: 4.7 nF, Capacitor_SMD:C_1206_3216Metric_Pad1.33x1.80mm_HandSolder, symbol kicad_inventree_lib:C_4.7nF_50V_1206
- removed D9: SMAJ33CA, Diode_SMD:D_SMA, symbol Diode:SMAJ33CA
- removed R9: 180R, Resistor_SMD:R_1206_3216Metric_Pad1.30x1.75mm_HandSolder, symbol kicad_inventree_lib:R_180R_1206_1%
Connections:
- net -: now also C3.2, D3.1 (A1)

Commit message: send to nextpcb
Parts:
- D1, D2, D3, D4, D5, D6, D7, D8: footprint Diode_SMD:D_SMA -> kicad_inventree_lib:SMASeries_LTF-M; symbol Diode:SMAJ33CA -> kicad_inventree_lib:SMAJ33CA; part_ipn (none) -> SMAJ33CA
Changed lines of the file:
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@@
 	)
 	(symbol
-		(lib_id "Diode:SMAJ33CA")
+		(lib_name "SMAJ33CA_4")
+		(lib_id "kicad_inventree_lib:SMAJ33CA")
 		(at 66.04 58.42 90)
 		(unit 1)
@@
 			)
 		)
-		(property "Footprint" "Diode_SMD:D_SMA"
+		(property "Footprint" "kicad_inventree_lib:SMASeries_LTF-M"
 			(at 71.12 58.42 0)
 			(effects
@@
 			)
 		)
-		(property "Datasheet" "https://www.littelfuse.com/media?resourcetype=datasheets&itemid=75e32973-b177-4ee3-a0ff-cedaf1abdb93&filename=smaj-datasheet"
+		(property "Datasheet" "http://inventree.network/part/123/"
 			(at 66.04 58.42 0)
 			(effects
@@
 			)
 		)
-		(property "Description" "400W bidirectional Transient Voltage Suppressor, 33.0Vr, SMA(DO-214AC)"
+		(property "Description" "7.5A 400W 53.3V 40.6V 33V SMA(DO-214AC) ESD and Surge Protection (TVS/ESD)"
+			(at 66.04 58.42 0)
+			(effects
+				(font
+					(size 1.27 1.27)
+				)
+				(hide yes)
+			)
+		)
+		(property "part_ipn" "SMAJ33CA"
 			(at 66.04 58.42 0)
 			(effects
@@
 	)
 	(symbol
-		(lib_id "Diode:SMAJ33CA")
+		(lib_name "SMAJ33CA_1")
+		(lib_id "kicad_inventree_lib:SMAJ33CA")
 		(at 66.04 33.02 90)
 		(unit 1)
@@
 			)
 		)
-		(property "Footprint" "Diode_SMD:D_SMA"
+		(property "Footprint" "kicad_inventree_lib:SMASeries_LTF-M"
 			(at 71.12 33.02 0)
 			(effects
@@
 			)
 		)
-		(property "Datasheet" "https://www.littelfuse.com/media?resourcetype=datasheets&itemid=75e32973-b177-4ee3-a0ff-cedaf1abdb93&filename=smaj-datasheet"
+		(property "Datasheet" "http://inventree.network/part/123/"
 			(at 66.04 33.02 0)
 			(effects
@@
 			)
 		)
-		(property "Description" "400W bidirectional Transient Voltage Suppressor, 33.0Vr, SMA(DO-214AC)"
+		(property "Description" "7.5A 400W 53.3V 40.6V 33V SMA(DO-214AC) ESD and Surge Protection (TVS/ESD)"
+			(at 66.04 33.02 0)
+			(effects
+				(font
+					(size 1.27 1.27)
+				)
+				(hide yes)
+			)
+		)
+		(property "part_ipn" "SMAJ33CA"
 			(at 66.04 33.02 0)
 			(effects
@@
 	)
 	(symbol
-		(lib_id "Diode:SMAJ33CA")
+		(lib_id "kicad_inventree_lib:SMAJ33CA")
 		(at 167.64 33.02 90)
 		(unit 1)
@@
 			)
 		)
-		(property "Footprint" "Diode_SMD:D_SMA"
+		(property "Footprint" "kicad_inventree_lib:SMASeries_LTF-M"
 			(at 172.72 33.02 0)
 			(effects
@@
 			)
 		)
-		(property "Datasheet" "https://www.littelfuse.com/media?resourcetype=datasheets&itemid=75e32973-b177-4ee3-a0ff-cedaf1abdb93&filename=smaj-datasheet"
+		(property "Datasheet" "http://inventree.network/part/123/"
 			(at 167.64 33.02 0)
 			(effects
@@
 			)
 		)
-		(property "Description" "400W bidirectional Transient Voltage Suppressor, 33.0Vr, SMA(DO-214AC)"
+		(property "Description" "7.5A 400W 53.3V 40.6V 33V SMA(DO-214AC) ESD and Surge Protection (TVS/ESD)"
+			(at 167.64 33.02 0)
+			(effects
+				(font
+					(size 1.27 1.27)
+				)
+				(hide yes)
+			)
+		)
+		(property "part_ipn" "SMAJ33CA"
 			(at 167.64 33.02 0)
 			(effects
@@
 	)
 	(symbol
-		(lib_id "Diode:SMAJ33CA")
+		(lib_id "kicad_inventree_lib:SMAJ33CA")
 		(at 167.64 83.82 90)
 		(unit 1)
@@
 			)
 		)
-		(property "Footprint" "Diode_SMD:D_SMA"
+		(property "Footprint" "kicad_inventree_lib:SMASeries_LTF-M"
 			(at 172.72 83.82 0)
 			(effects
@@
 			)
 		)
-		(property "Datasheet" "https://www.littelfuse.com/media?resourcetype=datasheets&itemid=75e32973-b177-4ee3-a0ff-cedaf1abdb93&filename=smaj-datasheet"
+		(property "Datasheet" "http://inventree.network/part/123/"
 			(at 167.64 83.82 0)
 			(effects
@@
 			)
 		)
-		(property "Description" "400W bidirectional Transient Voltage Suppressor, 33.0Vr, SMA(DO-214AC)"
+		(property "Description" "7.5A 400W 53.3V 40.6V 33V SMA(DO-214AC) ESD and Surge Protection (TVS/ESD)"
+			(at 167.64 83.82 0)
+			(effects
+				(font
+					(size 1.27 1.27)
+				)
+				(hide yes)
+			)
+		)
+		(property "part_ipn" "SMAJ33CA"
 			(at 167.64 83.82 0)
 			(effects
@@
 	)
 	(symbol
-		(lib_id "Diode:SMAJ33CA")
+		(lib_name "SMAJ33CA_3")
+		(lib_id "kicad_inventree_lib:SMAJ33CA")
 		(at 66.04 109.22 90)
 		(unit 1)
@@
 			)
 		)
-		(property "Footprint" "Diode_SMD:D_SMA"
+		(property "Footprint" "kicad_inventree_lib:SMASeries_LTF-M"
 			(at 71.12 109.22 0)
 			(effects
@@
 			)
 		)
-		(property "Datasheet" "https://www.littelfuse.com/media?resourcetype=datasheets&itemid=75e32973-b177-4ee3-a0ff-cedaf1abdb93&filename=smaj-datasheet"
+		(property "Datasheet" "http://inventree.network/part/123/"
 			(at 66.04 109.22 0)
 			(effects
@@
 			)
 		)
-		(property "Description" "400W bidirectional Transient Voltage Suppressor, 33.0Vr, SMA(DO-214AC)"
+		(property "Description" "7.5A 400W 53.3V 40.6V 33V SMA(DO-214AC) ESD and Surge Protection (TVS/ESD)"
 			(at 66.04 109.22 0)
 			(effects
@@
 			)
 		)
+		(property "part_ipn" "SMAJ33CA"
+			(at 66.04 109.22 0)
+			(effects
+				(font
+					(size 1.27 1.27)
+				)
+				(hide yes)
+			)
+		)
 		(pin "1"
 		)
@@
 	)
 	(symbol
-		(lib_id "Diode:SMAJ33CA")
+		(lib_name "SMAJ33CA_2")
+		(lib_id "kicad_inventree_lib:SMAJ33CA")
 		(at 66.04 83.82 90)
 		(unit 1)
@@
 			)
 		)
-		(property "Footprint" "Diode_SMD:D_SMA"
+		(property "Footprint" "kicad_inventree_lib:SMASeries_LTF-M"
 			(at 71.12 83.82 0)
 			(effects
@@
 			)
 		)
-		(property "Datasheet" "https://www.littelfuse.com/media?resourcetype=datasheets&itemid=75e32973-b177-4ee3-a0ff-cedaf1abdb93&filename=smaj-datasheet"
+		(property "Datasheet" "http://inventree.network/part/123/"
 			(at 66.04 83.82 0)
 			(effects
@@
 			)
 		)
-		(property "Description" "400W bidirectional Transient Voltage Suppressor, 33.0Vr, SMA(DO-214AC)"
+		(property "Description" "7.5A 400W 53.3V 40.6V 33V SMA(DO-214AC) ESD and Surge Protection (TVS/ESD)"
 			(at 66.04 83.82 0)
 			(effects
@@
 			)
 		)
+		(property "part_ipn" "SMAJ33CA"
+			(at 66.04 83.82 0)
+			(effects
+				(font
+					(size 1.27 1.27)
+				)
+				(hide yes)
+			)
+		)
 		(pin "1"
 		)
@@
 	)
 	(symbol
-		(lib_id "Diode:SMAJ33CA")
+		(lib_id "kicad_inventree_lib:SMAJ33CA")
 		(at 167.64 58.42 90)
 		(unit 1)
@@
 			)
 		)
-		(property "Footprint" "Diode_SMD:D_SMA"
+		(property "Footprint" "kicad_inventree_lib:SMASeries_LTF-M"
 			(at 172.72 58.42 0)
 			(effects
@@
 			)
 		)
-		(property "Datasheet" "https://www.littelfuse.com/media?resourcetype=datasheets&itemid=75e32973-b177-4ee3-a0ff-cedaf1abdb93&filename=smaj-datasheet"
+		(property "Datasheet" "http://inventree.network/part/123/"
 			(at 167.64 58.42 0)
 			(effects
@@
 			)
 		)
-		(property "Description" "400W bidirectional Transient Voltage Suppressor, 33.0Vr, SMA(DO-214AC)"
+		(property "Description" "7.5A 400W 53.3V 40.6V 33V SMA(DO-214AC) ESD and Surge Protection (TVS/ESD)"
+			(at 167.64 58.42 0)
+			(effects
+				(font
+					(size 1.27 1.27)
+				)
+				(hide yes)
+			)
+		)
+		(property "part_ipn" "SMAJ33CA"
 			(at 167.64 58.42 0)
 			(effects
@@
 	)
 	(symbol
-		(lib_id "Diode:SMAJ33CA")
+		(lib_id "kicad_inventree_lib:SMAJ33CA")
 		(at 167.64 109.22 90)
 		(unit 1)
@@
 			)
 		)
-		(property "Footprint" "Diode_SMD:D_SMA"
+		(property "Footprint" "kicad_inventree_lib:SMASeries_LTF-M"
 			(at 172.72 109.22 0)
 			(effects
@@
 			)
 		)
-		(property "Datasheet" "https://www.littelfuse.com/media?resourcetype=datasheets&itemid=75e32973-b177-4ee3-a0ff-cedaf1abdb93&filename=smaj-datasheet"
+		(property "Datasheet" "http://inventree.network/part/123/"
 			(at 167.64 109.22 0)
 			(effects
@@
 			)
 		)
-		(property "Description" "400W bidirectional Transient Voltage Suppressor, 33.0Vr, SMA(DO-214AC)"
+		(property "Description" "7.5A 400W 53.3V 40.6V 33V SMA(DO-214AC) ESD and Surge Protection (TVS/ESD)"
 			(at 167.64 109.22 0)
 			(effects
+				(font
+					(size 1.27 1.27)
+				)
+				(hide yes)
+			)
+		)
+		(property "part_ipn" "SMAJ33CA"
+			(at 167.64 109.22 0)
+			(effects
