File: PM-AI8-U/PM-AI8-U.kicad_sch (KiCad schematic)
At the start: 31 parts, among them J1 2EDGR-5.08-18P, J3 PinHeader P2.54 01x12 THT Str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, J4 PinHeader P2.54 01x12 THT Str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, J5 PinHeader_01x05_P2.54_THT_ang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, SW1 DSIC03LS-P, U1 AD4111BCPZ, U3 Weact ESP32-C3FH4

Commit message: send to nextpcb
Parts:
- removed J2: ~, kicad_inventree_lib:PM-front-02x08, symbol kicad_inventree_lib:PM-front-02x08
- removed SW1: DSIC03LS-P, kicad_inventree_lib:DSIC03LS-P, symbol kicad_inventree_lib:DSIC03LS-P
- added J2: ~, kicad_inventree_lib:PM-front-02x04, symbol kicad_inventree_lib:PM-front-02x04
- added SW1: DIP_SW-3P-P2.54-THT-Top, Button_Switch_THT:SW_DIP_SPSTx03_Slide_9.78x9.8mm_W7.62mm_P2.54mm, symbol kicad_inventree_lib:DIP_SW-3P-P2.54-THT-Top
- D10, D11, D12: value KPT-3216CGCK -> Green; footprint NextPCB:Kingbright_KPT-3216CGCK -> LED_SMD:LED_1206_3216Metric_Pad1.42x1.75mm_HandSolder; symbol kicad_inventree_lib:Kingbright_KPT-3216CGCK -> kicad_inventree_lib:LED_green_1206; part_ipn KPT-3216CGCK -> LED_green_1206
- D9: now left out of the parts list
Connections:
- net CS1 is gone; now on net CS: J3.6 (Pin_6)
- net +3.3V: now also SW1.4, SW1.5, SW1.6
- net A1: now also SW1.1
- net A2: now also SW1.2
- net A3: now also SW1.3
- net CS2: no longer names the net of J3.8 (Pin_8)
- net INT: no longer names the net of J3.7 (Pin_7)
- no-connect marks 18 -> 28
Other:
- note added: "Подключение фронтальной платы"

Commit message: PM-AI8-U
Parts:
- removed D13: B5819W, Diode_SMD:D_SOD-123, symbol kicad_inventree_lib:B5819W
- removed J3, J4: PinHeader P2.54 01x12 THT Straight, Connector_PinHeader_2.54mm:PinHeader_1x12_P2.54mm_Vertical, symbol kicad_inventree_lib:PinHeader_01x12_P2.54_THT_straight
- removed R15, R16, R17: 10k, Resistor_SMD:R_1206_3216Metric_Pad1.30x1.75mm_HandSolder, symbol kicad_inventree_lib:R_10k_1206_1%
- removed SW1: DIP_SW-3P-P2.54-THT-Top, Button_Switch_THT:SW_DIP_SPSTx03_Slide_9.78x9.8mm_W7.62mm_P2.54mm, symbol kicad_inventree_lib:DIP_SW-3P-P2.54-THT-Top
- removed U3: Weact ESP32-C3FH4, kicad_inventree_lib:Weact ESP32-C3FH4, symbol kicad_inventree_lib:Weact ESP32-C3FH4
- added PM1: ~, kicad_inventree_lib:PM-ESP32C3, symbol kicad_inventree_lib:PM-ESP32C3
Connections:
- net +3.3V: now also J5.4 (Pin_4), PM1.10 (+3.3V)
- net +5V: now also J5.3 (Pin_3); no longer J5.1 (Pin_1)
- net CLK: now also PM1.4 (GPIO9)
- net CS: now also PM1.5 (GPIO8)
- net GND: now also J2.7, J2.8, J5.5 (Pin_5), PM1.11 (GND), PM1.14 (GND); no longer J5.3 (Pin_3)
- net MISO: now also PM1.3 (GPIO3)
- net MOSI: now also PM1.2 (GPIO2)
- net SCL: now also J5.2 (Pin_2), PM1.13 (SCL); no longer J5.5 (Pin_5)
- net SDA: now also J5.1 (Pin_1), PM1.12 (SDA); no longer J5.4 (Pin_4)
- no-connect marks 28 -> 17
Other:
- note removed: "ESP32"
- note removed: "Задание адреса"
- moved on the sheet: J5
