File: PM-CPU-ESP-front/PM-CPU-ESP-front.kicad_sch (KiCad schematic)
At the start: 5 parts, among them J1 Conn_02x08_Odd_Even

Commit message: PM-CPU-ESP
Parts:
- removed J1: Conn_02x08_Odd_Even, NextPCB:Conn_02x08_pin, symbol NextPCB:Conn_02x08_pin
- removed R1: 270, Resistor_SMD:R_1206_3216Metric_Pad1.30x1.75mm_HandSolder, symbol NextPCB:R_270_0.25W
- removed R2: 120, Resistor_SMD:R_1206_3216Metric_Pad1.30x1.75mm_HandSolder, symbol NextPCB:R_120_0.25W
- added D1: KPT-3216CGCK, NextPCB:Kingbright_KPT-3216CGCK, symbol kicad_inventree_lib:Kingbright_KPT-3216CGCK
- added J1: PinHeader_02x08_P2.54_THT_Angle, Connector_PinHeader_2.54mm:PinHeader_2x08_P2.54mm_Horizontal, symbol kicad_inventree_lib:PinHeader_02x08_P2.54_THT_Angle
- added R1, R2, R3: 10k, Resistor_SMD:R_1206_3216Metric_Pad1.30x1.75mm_HandSolder, symbol kicad_inventree_lib:R_10k_1206_1%
- D2: renamed from D1; symbol NextPCB:Kingbright_KPT-3216CGCK -> kicad_inventree_lib:Kingbright_KPT-3216CGCK; part_ipn (none) -> KPT-3216CGCK
- D3: renamed from D2; symbol NextPCB:Kingbright_KPT-3216CGCK -> kicad_inventree_lib:Kingbright_KPT-3216CGCK; part_ipn (none) -> KPT-3216CGCK
Connections:
- net +3.3V: now also J1.5 (Pin_5), R3.2
- net +5V: now also J1.3 (Pin_3), R2.2
- net GND: now also D1.1 (K), J1.15 (Pin_15)
- net at D3.2 (A): now also R3.1
- net at D2.2 (A): now also R2.1
- new net: D1.2 (A), R1.1
- new net +24V: J1.1 (Pin_1), R1.2
- no-connect marks 11 -> 10
Other:
- note removed: "R = (3.3 - 2.1) / 0.01 = 120 Ом"
- note removed: "R = (5 - 2.1) / 0.01 = 290 Ом"

Commit message: send to nextpcb
Parts:
- removed D1, D2, D3: KPT-3216CGCK, NextPCB:Kingbright_KPT-3216CGCK, symbol kicad_inventree_lib:Kingbright_KPT-3216CGCK
- removed J1: PinHeader_02x08_P2.54_THT_Angle, Connector_PinHeader_2.54mm:PinHeader_2x08_P2.54mm_Horizontal, symbol kicad_inventree_lib:PinHeader_02x08_P2.54_THT_Angle
- added D1, D2, D3: Green, kicad_inventree_lib:LED_1206_3216Metric_ReverseMount_Hole1.8x2.4mm, symbol kicad_inventree_lib:LED_green_1206_reverse
- added J2: PinHeader_02x04_P2.54_THT_angle, Connector_PinHeader_2.54mm:PinHeader_2x04_P2.54mm_Horizontal, symbol kicad_inventree_lib:PinHeader_02x04_P2.54_THT_angle
Connections:
- net +24V: now also J2.1 (Pin_1)
- net +3.3V: now also J2.5 (Pin_5)
- net +5V: now also J2.3 (Pin_3)
- net GND: now also D1.1 (K), D2.1 (K), D3.1 (K), J2.7 (Pin_7)
- net at R2.1: now also D2.2 (A)
- net at R3.1: now also D3.2 (A)
- net at R1.1: now also D1.2 (A)
- no-connect marks 10 -> 4
