File: PM-RQ8/PM-RQ8.kicad_sch (KiCad schematic)
At the start: 32 parts, among them J1 2EDGK-5.08-02P, J17 2EDGR-5.08-18P, J18 S4B-PH-SM4-TB, J19 S4B-PH-SM4-TB, J2 2EDGK-5.08-02P, J20 Conn_01x03, J21 Conn_01x03, J22 Conn_01x03, J23 PHR-4, J24 PHR-4, J25 Conn_02x08_socket, J3 2EDGK-5.08-02P, J4 2EDGK-5.08-02P, J5 2EDGK-5.08-02P, J6 2EDGK-5.08-02P, J7 2EDGK-5.08-02P, J8 2EDGK-5.08-02P, K1 G5NB-1A-E_DC5, K2 G5NB-1A-E_DC5, K3 G5NB-1A-E_DC5, K4 G5NB-1A-E_DC5, K5 G5NB-1A-E_DC5, K6 G5NB-1A-E_DC5, K7 G5NB-1A-E_DC5, K8 G5NB-1A-E_DC5, U1 ULN2803A, U2 PCA9555PW, U3 64900001039

Commit message: PM_Bus
Parts:
- removed J18, J19: S4B-PH-SM4-TB, NextPCB:JST_S4B-PH-SM4-TB_JST_S4B-PH-SM4-TB, symbol NextPCB:JST_S4B-PH-SM4-TB
- removed J23, J24: PHR-4, symbol NextPCB:JST_PHR-4
- removed K1, K2, K3, K4, K5, K6, K7, K8: G5NB-1A-E_DC5, NextPCB:G5NB-1A-E_DC12_RELAY_G5NB-1A_DC5_OMR, symbol NextPCB:G5NB-1A-E_DC5
- added J9: PinHeader P2.54 01x08 THT Angle, Connector_PinHeader_2.54mm:PinHeader_1x08_P2.54mm_Horizontal, symbol kicad_inventree_lib:PinHeader P2.54 01x08 THT Angle
- added K1, K2, K3, K4, K5, K6, K7, K8: G5NB-1A-E-DC5, NextPCB:G5NB-1A-E_DC12_RELAY_G5NB-1A_DC5_OMR, symbol kicad_inventree_lib:G5NB-1A-E-DC5
Connections:
- net GND: now also J9.2 (Pin_2)
- net K1: now also K1.1
- net K2: now also K2.1
- net K3: now also K3.1
- net K4: now also K4.1
- net K5: now also K5.1
- net K6: now also K6.1
- net K7: now also K7.1
- net K8: now also K8.1
- net SCL: now also J9.4 (Pin_4)
- net SDA: now also J9.3 (Pin_3)
- net VDD: now also K1.4, K2.4, K3.4, K4.4, K5.4, K6.4, K7.4, K8.4
- net at J17.7 (Pin_7): now also K4.2
- net at J17.8 (Pin_8): now also K4.3
- net at J17.15 (Pin_15): now also K8.2
- net at J17.16 (Pin_16): now also K8.3
- net at J17.5 (Pin_5): now also K3.2
- net at J17.6 (Pin_6): now also K3.3
- net at J17.1 (Pin_1): now also K1.2
- net at J17.2 (Pin_2): now also K1.3
- net at J17.3 (Pin_3): now also K2.2
- net at J17.4 (Pin_4): now also K2.3
- net at U3.2: now also J9.1 (Pin_1)
- net at J17.13 (Pin_13): now also K7.2
- net at J17.14 (Pin_14): now also K7.3
- net at J17.10 (Pin_10): now also K5.3
- net at J17.11 (Pin_11): now also K6.2
- net at J17.12 (Pin_12): now also K6.3
- net at J17.9 (Pin_9): now also K5.2
- no-connect marks 42 -> 34

Commit message: PM-RQ8
Parts:
- removed J1, J2, J3, J4, J5, J6, J7, J8: 2EDGK-5.08-02P, symbol NextPCB:Degson_2EDGK-5.08-02P
- removed J17: 2EDGR-5.08-18P, NextPCB:Degson_2EDGR-5.08-18P, symbol NextPCB:Degson_2EDGR-5.08-18P
- removed J20, J21, J22: Conn_01x03, Connector_PinHeader_2.54mm:PinHeader_1x03_P2.54mm_Vertical_SMD_Pin1Left, symbol Connector_Generic:Conn_01x03
- removed J25: Conn_02x08_socket, Connector_PinSocket_2.54mm:PinSocket_2x08_P2.54mm_Vertical_SMD, symbol NextPCB:Conn_02x08_socket
- removed U1: ULN2803A, NextPCB:ULN2803A, symbol NextPCB:ULN2803A
- removed U2: PCA9555PW, Package_SO:TSSOP-24_4.4x7.8mm_P0.65mm, symbol NextPCB:PCA9555PW
- removed U3: 64900001039, NextPCB:Fuseholder, symbol NextPCB:Fuseholder
- added J1, J2, J3, J4, J5, J6, J7, J8: 2EDGK-5.08-02P, symbol kicad_inventree_lib:Degson_2EDGK-5.08-02P
- added J10: 2EDGR-5.08-18P, NextPCB:Degson_2EDGR-5.08-18P, symbol kicad_inventree_lib:Degson_2EDGR-5.08-18P
- added J11: FemaleHeader P2.54 02x08 SMD Straight, Connector_PinSocket_2.54mm:PinSocket_2x08_P2.54mm_Vertical_SMD, symbol kicad_inventree_lib:FemaleHeader P2.54 02x08 SMD Straight
- added J12, J13, J14: PinHeader_P2.54_01x03_SMD_Straight, Connector_PinHeader_2.54mm:PinHeader_1x03_P2.54mm_Vertical_SMD_Pin1Left, symbol kicad_inventree_lib:PinHeader P2.54 01x03 SMD Straight
- added U1: ULN2803A, NextPCB:ULN2803A, symbol kicad_inventree_lib:ULN2803A
- added U2: PCA9555PW, Package_SO:TSSOP-24_4.4x7.8mm_P0.65mm, symbol kicad_inventree_lib:PCA9555PW
- added U4: 64900001039, NextPCB:Fuseholder, symbol kicad_inventree_lib:Fuseholder
Connections:
- net A0: now also J12.2 (Pin_2), U2.21 (A0)
- net A1: now also J13.2 (Pin_2), U2.2 (A1)
- net A2: now also J14.2 (Pin_2), U2.3 (A2)
- net GND: now also J12.3 (Pin_3), J13.3 (Pin_3), J14.3 (Pin_3), U1.9 (GND), U2.12 (VSS)
- net K1: now also J11.1 (Pin_1), U1.18 (O1)
- net K2: now also J11.3 (Pin_3), U1.17 (O2)
- net K3: now also J11.5 (Pin_5), U1.16 (O3)
- net K4: now also J11.7 (Pin_7), U1.15 (O4)
- net K5: now also J11.9 (Pin_9), U1.14 (O5)
- net K6: now also J11.11 (Pin_11), U1.13 (O6)
- net K7: now also J11.13 (Pin_13), U1.12 (O7)
- net K8: now also J11.15 (Pin_15), U1.11 (O8)
- net SCL: now also U2.22 (SCL)
- net SDA: now also U2.23 (SDA)
- net VDD: now also J11.2 (Pin_2), J12.1 (Pin_1), J13.1 (Pin_1), J14.1 (Pin_1), U1.10 (COM), U2.24 (VDD), U4.1
- net at K5.2: now also J10.9 (Pin_9)
- net at K5.3: now also J10.10 (Pin_10)
- net at K3.2: now also J10.5 (Pin_5)
- net at K3.3: now also J10.6 (Pin_6)
- net at K8.2: now also J10.15 (Pin_15)
- net at K8.3: now also J10.16 (Pin_16)
- net at K2.2: now also J10.3 (Pin_3)
- net at K2.3: now also J10.4 (Pin_4)
- net at K4.2: now also J10.7 (Pin_7)
- net at K4.3: now also J10.8 (Pin_8)
- net at K1.2: now also J10.1 (Pin_1)
- net at K1.3: now also J10.2 (Pin_2)
- net at K6.2: now also J10.11 (Pin_11)
- net at K6.3: now also J10.12 (Pin_12)
- net at K7.2: now also J10.13 (Pin_13)
- net at K7.3: now also J10.14 (Pin_14)
- net at J9.1 (Pin_1): now also U4.2
- new net: U1.1 (I1), U2.4 (IO0_0)
- new net: U1.2 (I2), U2.5 (IO0_1)
- new net: U1.3 (I3), U2.6 (IO0_2)
- new net: U1.4 (I4), U2.7 (IO0_3)
- new net: U1.5 (I5), U2.8 (IO0_4)
- new net: U1.6 (I6), U2.9 (IO0_5)
- new net: U1.7 (I7), U2.10 (IO0_6)
- new net: U1.8 (I8), U2.11 (IO0_7)
- no-connect marks 34 -> 38
Other:
- moved on the sheet: J9

Commit message: InvenTree
Parts:
- removed J11: FemaleHeader P2.54 02x08 SMD Straight, Connector_PinSocket_2.54mm:PinSocket_2x08_P2.54mm_Vertical_SMD, symbol kicad_inventree_lib:FemaleHeader P2.54 02x08 SMD Straight
- added J11, J16, J17: Shunt 2.54 Open Top, symbol kicad_inventree_lib:Shunt 2.54 Open Top
- added J15: FemaleHeader P2.54 02x08 THT Straight, Connector_PinSocket_2.54mm:PinSocket_2x08_P2.54mm_Vertical, symbol kicad_inventree_lib:FemaleHeader P2.54 02x08 THT Straight
Connections:
- net K1: now also J15.1 (Pin_1)
- net K2: now also J15.3 (Pin_3)
- net K3: now also J15.5 (Pin_5)
- net K4: now also J15.7 (Pin_7)
- net K5: now also J15.9 (Pin_9)
- net K6: now also J15.11 (Pin_11)
- net K7: now also J15.13 (Pin_13)
- net K8: now also J15.15 (Pin_15)
- net VDD: now also J15.2 (Pin_2)

Commit message: PM-AI-xxx docs
Parts:
- removed J9: PinHeader P2.54 01x08 THT Angle, Connector_PinHeader_2.54mm:PinHeader_1x08_P2.54mm_Horizontal, symbol kicad_inventree_lib:PinHeader P2.54 01x08 THT Angle
- added J18: 2EDGK-5.08-02P, symbol kicad_inventree_lib:Degson_2EDGK-5.08-02P
- added J9: Conn_01x04_Pin, Connector_PinHeader_2.54mm:PinHeader_1x04_P2.54mm_Horizontal, symbol kicad_inventree_lib:PinHeader P2.54 01x04 THT Angle
Connections:
- net GND: now also J9.2 (Pin_2)
- net SCL: now also J9.4 (Pin_4)
- net SDA: now also J9.3 (Pin_3)
- net at U4.2: now also J9.1 (Pin_1)
- no-connect marks 38 -> 36
Changed lines of the file:
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@@
 	)
 	(no_connect
+		(at 38.1 73.66)
+	)
+	(no_connect
 		(at 38.1 63.5)
 	)
@@
 	)
 	(no_connect
-		(at 241.3 119.38)
-	)
-	(no_connect
 		(at 198.12 50.8)
 	)
@@
 	)
 	(no_connect
-		(at 241.3 114.3)
+		(at 38.1 76.2)
 	)
 	(no_connect
@@
 	)
 	(no_connect
-		(at 241.3 116.84)
-	)
-	(no_connect
 		(at 152.4 111.76)
 	)
@@
 	)
 	(no_connect
-		(at 241.3 121.92)
-	)
-	(no_connect
 		(at 38.1 38.1)
 	)
@@
 	)
 	(symbol
+		(lib_id "kicad_inventree_lib:Degson_2EDGK-5.08-02P")
+		(at 38.1 73.66 0)
+		(mirror y)
+		(unit 1)
+		(exclude_from_sim no)
+		(in_bom yes)
+		(on_board no)
+		(dnp no)
+		(property "Reference" "J18"
+			(at 33.528 73.66 0)
+			(effects
+				(font
+					(size 1.27 1.27)
+				)
+				(justify right)
+			)
+		)
+		(property "Value" "2EDGK-5.08-02P"
+			(at 18.542 75.946 0)
+			(effects
+				(font
+					(size 1.27 1.27)
+				)
+				(justify right)
+			)
+		)
+		(property "Footprint" ""
+			(at 38.1 73.66 0)
+			(effects
+				(font
+					(size 1.27 1.27)
+				)
+				(hide yes)
+			)
+		)
+		(property "Datasheet" "http://inventree.network/part/18/"
+			(at 38.1 73.66 0)
+			(effects
+				(font
+					(size 1.27 1.27)
+				)
+				(hide yes)
+			)
+		)
+		(property "Description" "Generic connector, single row, 01x02, script generated"
+			(at 38.1 73.66 0)
+			(effects
+				(font
+					(size 1.27 1.27)
+				)
+				(hide yes)
+			)
+		)
+		(property "NextPCB_url" "https://www.hqonline.com/product-detail/max-maixu--mx2edgk-5-08-02p-gn01-cu-y-a-1027943030"
+			(at 38.1 73.66 0)
+			(effects
+				(font
+					(size 1.27 1.27)
+				)
+				(hide yes)
+			)
+		)
+		(property "NextPCB_price" "0.11828"
+			(at 38.1 73.66 0)
+			(effects
+				(font
+					(size 1.27 1.27)
+				)
+				(hide yes)
+			)
+		)
+		(property "part_ipn" "2EDGK-5.08-02P"
+			(at 38.1 73.66 0)
+			(effects
+				(font
+					(size 1.27 1.27)
+				)
+				(hide yes)
+			)
+		)
+		(pin "2"
+		)
+		(pin "1"
+		)
+		(instances
+			(project "PM-RQ8"
+				(path "/a75183a9-ea53-46d5-9d29-d6271be85780"
+					(reference "J18")
+					(unit 1)
+				)
+			)
+		)
+	)
+	(symbol
 		(lib_id "power:VDD")
 		(at 151.13 22.86 0)
@@
 	)
 	(symbol
-		(lib_id "kicad_inventree_lib:Degson_2EDGK-5.08-02P")
-		(at 38.1 53.34 0)
+		(lib_id "kicad_inventree_lib:PinHeader P2.54 01x04 THT Angle")
+		(at 246.38 106.68 0)
 		(mirror y)
 		(unit 1)
 		(exclude_from_sim no)
 		(in_bom yes)
-		(on_board no)
+		(on_board yes)
 		(dnp no)
-		(property "Reference" "J5"
-			(at 33.528 53.34 0)
+		(fields_autoplaced yes)
+		(property "Reference" "J9"
+			(at 247.65 107.9499 0)
 			(effects
 				(font
@@
 			)
 		)
-		(property "Value" "2EDGK-5.08-02P"
-			(at 18.542 55.626 0)
+		(property "Value" "Conn_01x04_Pin"
+			(at 247.65 109.2199 0)
 			(effects
 				(font
@@
 				)
 				(justify right)
-			)
-		)
-		(property "Footprint" ""
-			(at 38.1 53.34 0)
-			(effects
-				(font
-					(size 1.27 1.27)
-				)
 				(hide yes)
 			)
 		)
-		(property "Datasheet" "http://inventree.network/part/18/"
-			(at 38.1 53.34 0)
+		(property "Footprint" "Connector_PinHeader_2.54mm:PinHeader_1x04_P2.54mm_Horizontal"
+			(at 246.38 106.68 0)
 			(effects
 				(font
@@
 			)
 		)
-		(property "Description" "Generic connector, single row, 01x02, script generated"
-			(at 38.1 53.34 0)
-			(effects
-				(font
-					(size 1.27 1.27)
-				)
-				(hide yes)
-			)
-		)
-		(property "NextPCB_url" "https://www.hqonline.com/product-detail/max-maixu--mx2edgk-5-08-02p-gn01-cu-y-a-1027943030"
-			(at 38.1 53.34 0)
+		(property "Datasheet" "http://inventree.network/part/9/"
+			(at 246.38 106.68 0)
 			(effects
 				(font
@@
 			)
 		)
-		(property "NextPCB_price" "0.11828"
-			(at 38.1 53.34 0)
+		(property "Description" "Generic connector, single row, 01x04, script generated"
+			(at 246.38 106.68 0)
 			(effects
 				(font
@@
 			)
 		)
-		(property "part_ipn" "2EDGK-5.08-02P"
-			(at 38.1 53.34 0)
+		(property "part_ipn" "PinHeader P2.54 01x04 THT Angle"
+			(at 246.38 106.68 0)
 			(effects
 				(font
@@
 		(pin "2"
 		)
+		(pin "3"
+		)
+		(pin "4"
+		)
 		(pin "1"
 		)
 		(instances
-			(project "PM-RQ8"
+			(project ""
 				(path "/a75183a9-ea53-46d5-9d29-d6271be85780"
-					(reference "J5")
+					(reference "J9")
 					(unit 1)
 				)
@@
 	)
 	(symbol
-		(lib_id "Mechanical:MountingHole")
-		(at 152.4 186.69 0)
+		(lib_id "kicad_inventree_lib:Degson_2EDGK-5.08-02P")
+		(at 38.1 53.34 0)
+		(mirror y)
 		(unit 1)
-		(exclude_from_sim yes)
-		(in_bom no)
-		(on_board yes)
+		(exclude_from_sim no)
+		(in_bom yes)
+		(on_board no)
 		(dnp no)
-		(fields_autoplaced yes)
-		(property "Reference" "H3"
-			(at 154.94 185.4199 0)
+		(property "Reference" "J5"
+			(at 33.528 53.34 0)
 			(effects
 				(font
 					(size 1.27 1.27)
 				)
-				(justify left)
+				(justify right)
 			)
 		)
-		(property "Value" "MountingHole"
-			(at 154.94 187.9599 0)
+		(property "Value" "2EDGK-5.08-02P"
+			(at 18.542 55.626 0)
 			(effects
 				(font
 					(size 1.27 1.27)
 				)
-				(justify left)
+				(justify right)
 			)
 		)
-		(property "Footprint" "MountingHole:MountingHole_3.2mm_M3"
-			(at 152.4 186.69 0)
+		(property "Footprint" ""
+			(at 38.1 53.34 0)
 			(effects
 				(font
@@
 			)
 		)
-		(property "Datasheet" "~"
-			(at 152.4 186.69 0)
+		(property "Datasheet" "http://inventree.network/part/18/"
+			(at 38.1 53.34 0)
 			(effects
 				(font
@@
 			)
 		)
-		(property "Description" "Mounting Hole without connection"
-			(at 152.4 186.69 0)
+		(property "Description" "Generic connector, single row, 01x02, script generated"
+			(at 38.1 53.34 0)
 			(effects
 				(font
@@
 			)
 		)
-		(property "NextPCB_url" ""
-			(at 152.4 186.69 0)
+		(property "NextPCB_url" "https://www.hqonline.com/product-detail/max-maixu--mx2edgk-5-08-02p-gn01-cu-y-a-1027943030"
+			(at 38.1 53.34 0)
 			(effects
 				(font
@@
 			)
 		)
-		(property "NextPCB_price" ""
-			(at 152.4 186.69 0)
+		(property "NextPCB_price" "0.11828"
+			(at 38.1 53.34 0)
 			(effects
 				(font
@@
 			)
 		)
-		(property "MANUFACTURER" ""
-			(at 152.4 186.69 0)
+		(property "part_ipn" "2EDGK-5.08-02P"
+			(at 38.1 53.34 0)
 			(effects
 				(font
@@
 			)
 		)
+		(pin "2"
+		)
+		(pin "1"
+		)
 		(instances
-			(project "PM-RQ8-base"
+			(project "PM-RQ8"
 				(path "/a75183a9-ea53-46d5-9d29-d6271be85780"
-					(reference "H3")
+					(reference "J5")
 					(unit 1)
 				)
@@
 	)
 	(symbol
-		(lib_id "kicad_inventree_lib:PinHeader P2.54 01x08 THT Angle")
-		(at 246.38 111.76 0)
-		(mirror y)
+		(lib_id "Mechanical:MountingHole")
+		(at 152.4 186.69 0)
 		(unit 1)
-		(exclude_from_sim no)
-		(in_bom yes)
+		(exclude_from_sim yes)
+		(in_bom no)
 		(on_board yes)
 		(dnp no)
-		(property "Reference" "J9"
-			(at 248.92 113.03 90)
+		(fields_autoplaced yes)
+		(property "Reference" "H3"
+			(at 154.94 185.4199 0)
 			(effects
 				(font
 					(size 1.27 1.27)
 				)
+				(justify left)
 			)
 		)
-		(property "Value" "PinHeader P2.54 01x08 THT Angle"
-			(at 245.745 101.6 0)
+		(property "Value" "MountingHole"
+			(at 154.94 187.9599 0)
+			(effects
+				(font
+					(size 1.27 1.27)
+				)
+				(justify left)
+			)
+		)
+		(property "Footprint" "MountingHole:MountingHole_3.2mm_M3"
+			(at 152.4 186.69 0)
 			(effects
 				(font
@@
 			)
 		)
-		(property "Footprint" "Connector_PinHeader_2.54mm:PinHeader_1x08_P2.54mm_Horizontal"
-			(at 246.38 111.76 0)
+		(property "Datasheet" "~"
+			(at 152.4 186.69 0)
 			(effects
 				(font
@@
 			)
 		)
-		(property "Datasheet" "http://inventree.network/part/11/"
-			(at 246.38 111.76 0)
+		(property "Description" "Mounting Hole without connection"
+			(at 152.4 186.69 0)
 			(effects
 				(font
@@
 			)
 		)
-		(property "Description" "Generic connector, single row, 01x08, script generated"
-			(at 246.38 111.76 0)
+		(property "NextPCB_url" ""
+			(at 152.4 186.69 0)
 			(effects
 				(font
@@
 			)
 		)
-		(property "part_ipn" "PinHeader P2.54 01x08 THT Angle"
-			(at 246.38 111.76 0)
+		(property "NextPCB_price" ""
+			(at 152.4 186.69 0)
 			(effects
 				(font
@@
 		)
 		(property "MANUFACTURER" ""
-			(at 246.38 111.76 0)
+			(at 152.4 186.69 0)
 			(effects
 				(font
@@
 			)
 		)
-		(pin "6"
-		)
-		(pin "1"
-		)
-		(pin "2"
-		)
-		(pin "8"
-		)
-		(pin "5"
-		)
-		(pin "7"
-		)
-		(pin "3"
-		)
-		(pin "4"
-		)
 		(instances
-			(project ""
+			(project "PM-RQ8-base"
 				(path "/a75183a9-ea53-46d5-9d29-d6271be85780"
-					(reference "J9")
+					(reference "H3")
 					(unit 1)
 				)

Commit message: send to nextpcb
Parts:
- removed J11, J16, J17: Shunt 2.54 Open Top, symbol kicad_inventree_lib:Shunt 2.54 Open Top
- removed J12, J13, J14: PinHeader_P2.54_01x03_SMD_Straight, Connector_PinHeader_2.54mm:PinHeader_1x03_P2.54mm_Vertical_SMD_Pin1Left, symbol kicad_inventree_lib:PinHeader P2.54 01x03 SMD Straight
- removed J15: FemaleHeader P2.54 02x08 THT Straight, Connector_PinSocket_2.54mm:PinSocket_2x08_P2.54mm_Vertical, symbol kicad_inventree_lib:FemaleHeader P2.54 02x08 THT Straight
- removed J9: Conn_01x04_Pin, Connector_PinHeader_2.54mm:PinHeader_1x04_P2.54mm_Horizontal, symbol kicad_inventree_lib:PinHeader P2.54 01x04 THT Angle
- removed U4: 64900001039, NextPCB:Fuseholder, symbol kicad_inventree_lib:Fuseholder
- added C3: 1uF, Capacitor_SMD:C_1206_3216Metric_Pad1.33x1.80mm_HandSolder, symbol kicad_inventree_lib:C_1uF_50V_1206
- added D1, D2, D3, D4, D5, D6, D7, D8: BAT20J, kicad_inventree_lib:SOD-323_STM-M, symbol kicad_inventree_lib:BAT20J
- added J1: ~, kicad_inventree_lib:PM-front-02x04, symbol kicad_inventree_lib:PM-front-02x04
- added J2: PinHeader_01x05_P2.54_THT_angle, Connector_PinHeader_2.54mm:PinHeader_1x05_P2.54mm_Horizontal, symbol kicad_inventree_lib:PinHeader_01x05_P2.54_THT_angle
- added J9: U254-051T-4BH83-S1S, kicad_inventree_lib:CONN5_H83-S1S_XKB, symbol kicad_inventree_lib:XKG_U254-051T-4BH83-S1S
- added R1, R2: 10k, Resistor_SMD:R_1206_3216Metric_Pad1.30x1.75mm_HandSolder, symbol kicad_inventree_lib:R_10k_1206_1%
- added SW2, SW4: Button, kicad_inventree_lib:SW_TS-1088_XNP-M, symbol kicad_inventree_lib:TS-1088-AR02016
- added U3: ESP32-C3-WROOM-02U-N4, ESP32-C3-WROOM-02U_EXP, symbol kicad_inventree_lib:ESP32-C3-WROOM-02U-N4
- renumbered J1 to J100, J2 to J20
Connections:
- net GND: now also C3.2, J2.3 (Pin_3), J9.5 (GND), SW2.1, SW4.1
- net K1: now also D1.1
- net K2: now also D2.1
- net K3: now also D3.1
- net K4: now also D4.1
- net K5: now also D5.1
- net K6: now also D6.1
- net K7: now also D7.1
- net K8: now also D8.1
- net SCL: now also J2.5 (Pin_5)
- net SDA: now also J2.4 (Pin_4)
- net VDD: now also J1.1; no longer K1.4, K2.4, K3.4, K4.4, K5.4, K6.4, K7.4, K8.4, U1.10 (COM), U2.24 (VDD)
- net at K5.2: now also J10.10 (Pin_10); no longer J10.9 (Pin_9)
- net at K5.3: now also J10.9 (Pin_9); no longer J10.10 (Pin_10)
- net at K3.2: now also J10.6 (Pin_6); no longer J10.5 (Pin_5)
- net at K3.3: now also J10.5 (Pin_5); no longer J10.6 (Pin_6)
- net at K8.2: now also J10.16 (Pin_16); no longer J10.15 (Pin_15)
- net at K8.3: now also J10.15 (Pin_15); no longer J10.16 (Pin_16)
- net at K2.2: now also J10.4 (Pin_4); no longer J10.3 (Pin_3)
- net at K2.3: now also J10.3 (Pin_3); no longer J10.4 (Pin_4)
- net at K4.2: now also J10.8 (Pin_8); no longer J10.7 (Pin_7)
- net at K4.3: now also J10.7 (Pin_7); no longer J10.8 (Pin_8)
- net at K1.2: now also J10.2 (Pin_2); no longer J10.1 (Pin_1)
- net at K1.3: now also J10.1 (Pin_1); no longer J10.2 (Pin_2)
- net at J10.11 (Pin_11): now also K6.3; no longer K6.2
- net at J10.12 (Pin_12): now also K6.2; no longer K6.3
- net at J10.13 (Pin_13): now also K7.3; no longer K7.2
- net at J10.14 (Pin_14): now also K7.2; no longer K7.3
- new net +3.3V: J2.2 (Pin_2), R1.1, R2.1, U3.1 (3V3)
- new net +5V: D1.2, D2.2, D3.2, D4.2, D5.2, D6.2, D7.2, D8.2, J2.1 (Pin_1), K1.4, K2.4, K3.4, K4.4, K5.4, K6.4, K7.4, K8.4, U1.10 (COM), U2.24 (VDD)
- new net MCU_BOOT: R2.2, SW4.2, U3.8 (IO9)
- new net MCU_EN: C3.1, R1.2, SW2.2, U3.2 (EN)
- new net USB_DN: J9.2 (D-), U3.13 (IO18_(USB_D-))
- new net USB_DP: J9.3 (D+), U3.14 (IO19_(USB_D+))
- no-connect marks 36 -> 34
Other:
- moved on the sheet: H1, H2, H3, H4, J10, J100, J18, J20, J3, J4, J5, J6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

Commit message: PM-PS
Parts:
- removed C3: 1uF, Capacitor_SMD:C_1206_3216Metric_Pad1.33x1.80mm_HandSolder, symbol kicad_inventree_lib:C_1uF_50V_1206
- removed J9: U254-051T-4BH83-S1S, kicad_inventree_lib:CONN5_H83-S1S_XKB, symbol kicad_inventree_lib:XKG_U254-051T-4BH83-S1S
- removed R1, R2: 10k, Resistor_SMD:R_1206_3216Metric_Pad1.30x1.75mm_HandSolder, symbol kicad_inventree_lib:R_10k_1206_1%
- removed SW2, SW4: Button, kicad_inventree_lib:SW_TS-1088_XNP-M, symbol kicad_inventree_lib:TS-1088-AR02016
- removed U3: ESP32-C3-WROOM-02U-N4, ESP32-C3-WROOM-02U_EXP, symbol kicad_inventree_lib:ESP32-C3-WROOM-02U-N4
- added U4: TXS0108EPW, Package_SO:TSSOP-20_4.4x6.5mm_P0.65mm, symbol Logic_LevelTranslator:TXS0108EPW
- added U5: TXB0104D, Package_SO:SOIC-14_3.9x8.7mm_P1.27mm, symbol Logic_LevelTranslator:TXB0104D
Connections:
- no-connect marks 34 -> 32
Other:
- added sheet ESP32 (ESP32.kicad_sch)
- note added: "TXS0108EPWR"

Commit message: PM-RQ8
Parts:
- removed H4: MountingHole, MountingHole:MountingHole_3.2mm_M3, symbol Mechanical:MountingHole
- removed U2: PCA9555PW, Package_SO:TSSOP-24_4.4x7.8mm_P0.65mm, symbol kicad_inventree_lib:PCA9555PW
- removed U4: TXS0108EPW, Package_SO:TSSOP-20_4.4x6.5mm_P0.65mm, symbol Logic_LevelTranslator:TXS0108EPW
- removed U5: TXB0104D, Package_SO:SOIC-14_3.9x8.7mm_P1.27mm, symbol Logic_LevelTranslator:TXB0104D
- added PE1: PE, kicad_inventree_lib:PE, symbol kicad_inventree_lib:PE
- added U6: MCP23S17_ML, Package_DFN_QFN:QFN-28-1EP_6x6mm_P0.65mm_EP4.25x4.25mm, symbol kicad_inventree_lib:MCP23S17_ML
- K1, K2, K3, K4, K5, K6, K7, K8: footprint NextPCB:G5NB-1A-E_DC12_RELAY_G5NB-1A_DC5_OMR -> kicad_inventree_lib:G5NB-1A-E_DC12_RELAY_G5NB-1A_DC5_OMR
Connections:
- net +3.3V: now also U6.5 (VDD)
- net GND: now also U6.29 (EP), U6.6 (VSS)
- net at U1.1 (I1): now also U6.17 (GPA0)
- net at U1.2 (I2): now also U6.18 (GPA1)
- net at U1.3 (I3): now also U6.19 (GPA2)
- net at U1.4 (I4): now also U6.20 (GPA3)
- net at U1.5 (I5): now also U6.21 (GPA4)
- net at U1.6 (I6): now also U6.22 (GPA5)
- net at U1.7 (I7): now also U6.23 (GPA6)
- net at U1.8 (I8): now also U6.24 (GPA7)
- net PE: now reaches J10.17 (Pin_17)
- net PE: now also J10.18 (Pin_18), PE1.1
- new net CS: U6.7 (~{CS})
- new net INT: U6.15 (INTB)
- new net MISO: U6.10 (SO)
- new net MOSI: U6.9 (SI)
- new net SCK: U6.8 (SCK)
- no-connect marks 32 -> 38
Other:
- sheet ESP32 ports: added GPIO0, GPIO1, GPIO10, GPIO2, GPIO3, GPIO4, GPIO5, GPIO6, GPIO7, GPIO8, GPIO9; removed none
- note removed: "TXS0108EPWR"
- moved on the sheet: D1, D2, D3, D4, D5, D6, D7, D8, H1, H2, H3, J1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
