File: PM-RQ8/PM-RQ8.kicad_sch (KiCad schematic)
At the start: 34 parts, among them J10 2EDGR-5.08-18P, J100 2EDGK-5.08-02P, J18 2EDGK-5.08-02P, J2 PinHeader_01x05_P2.54_THT_ang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, J20 2EDGK-5.08-02P, J3 2EDGK-5.08-02P, J4 2EDGK-5.08-02P, J5 2EDGK-5.08-02P, J6 2EDGK-5.08-02P, J7 2EDGK-5.08-02P, J8 2EDGK-5.08-02P, K1 G5NB-1A-E-DC5, K2 G5NB-1A-E-DC5, K3 G5NB-1A-E-DC5, K4 G5NB-1A-E-DC5, K5 G5NB-1A-E-DC5, K6 G5NB-1A-E-DC5, K7 G5NB-1A-E-DC5, K8 G5NB-1A-E-DC5, U1 ULN2803A, U6 MCP23S17_ML

Commit message: PM-ESPC3
Connections:
- net +3.3V: now also J2.4 (Pin_4); no longer J2.2 (Pin_2)
- net +5V: now also J2.3 (Pin_3); no longer J2.1 (Pin_1)
- net GND: now also J2.5 (Pin_5); no longer J2.3 (Pin_3)
- net K1: now also U1.11 (O8); no longer U1.18 (O1)
- net K2: now also U1.12 (O7); no longer U1.17 (O2)
- net K3: now also U1.13 (O6); no longer U1.16 (O3)
- net K4: now also U1.14 (O5); no longer U1.15 (O4)
- net K5: now also U1.15 (O4); no longer U1.14 (O5)
- net K6: now also U1.16 (O3); no longer U1.13 (O6)
- net K7: now also U1.17 (O2); no longer U1.12 (O7)
- net K8: now also U1.18 (O1); no longer U1.11 (O8)
- net PE: now also J10.10 (Pin_10), J10.9 (Pin_9); no longer J10.17 (Pin_17), J10.18 (Pin_18)
- net SCL: now also J2.2 (Pin_2); no longer J2.5 (Pin_5)
- net SDA: now also J2.1 (Pin_1); no longer J2.4 (Pin_4)
- net at K5.2: now also J10.12 (Pin_12); no longer J10.10 (Pin_10)
- net at K5.3: now also J10.11 (Pin_11); no longer J10.9 (Pin_9)
- net at K8.2: now also J10.18 (Pin_18); no longer J10.16 (Pin_16)
- net at K8.3: now also J10.17 (Pin_17); no longer J10.15 (Pin_15)
- net K1_exp: now reaches U6.17 (GPA0)
- net K1_exp: now also U1.8 (I8); no longer U1.1 (I1)
- net K2_exp: now reaches U6.18 (GPA1)
- net K2_exp: now also U1.7 (I7); no longer U1.2 (I2)
- net K3_exp: now reaches U6.19 (GPA2)
- net K3_exp: now also U1.6 (I6); no longer U1.3 (I3)
- net K4_exp: now reaches U6.20 (GPA3)
- net K4_exp: now also U1.5 (I5); no longer U1.4 (I4)
- net K5_exp: now reaches U6.21 (GPA4)
- net K5_exp: now also U1.4 (I4); no longer U1.5 (I5)
- net K6_exp: now reaches U6.22 (GPA5)
- net K6_exp: now also U1.3 (I3); no longer U1.6 (I6)
- net K7_exp: now reaches U6.23 (GPA6)
- net K7_exp: now also U1.2 (I2); no longer U1.7 (I7)
- net K8_exp: now reaches U6.24 (GPA7)
- net K8_exp: now also U1.1 (I1); no longer U1.8 (I8)
- net at K6.3: now also J10.13 (Pin_13); no longer J10.11 (Pin_11)
- net at K6.2: now also J10.14 (Pin_14); no longer J10.12 (Pin_12)
- net at K7.3: now also J10.15 (Pin_15); no longer J10.13 (Pin_13)
- net at K7.2: now also J10.16 (Pin_16); no longer J10.14 (Pin_14)
- no-connect marks 38 -> 37
Other:
- sheet ESP32 ports: added SCL, SDA; removed GPIO0, GPIO1, GPIO10
- moved on the sheet: U6
