File: PM-RQ8/PM-RQ8.kicad_pcb (KiCad board)
At the start: 2 copper layers, 99.1 x 99.1 mm, 23 parts, among them J17 2EDGR-5.08-18P, J20 Conn_01x03, J21 Conn_01x03, J22 Conn_01x03, J25 Conn_02x08_socket, J9 PinHeader P2.54 01x08 THT Ang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, K1 G5NB-1A-E-DC5, K2 G5NB-1A-E-DC5, K3 G5NB-1A-E-DC5, K4 G5NB-1A-E-DC5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

Commit message: PM-RQ8
Parts:
- removed J17: 2EDGR-5.08-18P, NextPCB:Degson_2EDGR-5.08-18P
- removed J20, J21, J22: Conn_01x03, Connector_PinHeader_2.54mm:PinHeader_1x03_P2.54mm_Vertical_SMD_Pin1Left
- removed J25: Conn_02x08_socket, Connector_PinSocket_2.54mm:PinSocket_2x08_P2.54mm_Vertical_SMD
- added J10: 2EDGR-5.08-18P, NextPCB:Degson_2EDGR-5.08-18P, F.Cu at (81.3, 58.4)
- added J11: FemaleHeader P2.54 02x08 SMD Straight, Connector_PinSocket_2.54mm:PinSocket_2x08_P2.54mm_Vertical_SMD, F.Cu at (91.5, 100.3)
- added J12: PinHeader_P2.54_01x03_SMD_Straight, Connector_PinHeader_2.54mm:PinHeader_1x03_P2.54mm_Vertical_SMD_Pin1Left, F.Cu at (144.8, 116.8)
- added J13: PinHeader_P2.54_01x03_SMD_Straight, Connector_PinHeader_2.54mm:PinHeader_1x03_P2.54mm_Vertical_SMD_Pin1Left, F.Cu at (152.4, 116.8)
- added J14: PinHeader_P2.54_01x03_SMD_Straight, Connector_PinHeader_2.54mm:PinHeader_1x03_P2.54mm_Vertical_SMD_Pin1Left, F.Cu at (160.0, 116.8)
- moved U1 5.68 mm to (154.9, 68.6)
- moved U2 3.59 mm to (154.9, 86.4)

Commit message: InvenTree
Parts:
- removed J11: FemaleHeader P2.54 02x08 SMD Straight, Connector_PinSocket_2.54mm:PinSocket_2x08_P2.54mm_Vertical_SMD
- removed U3: 64900001039, NextPCB:Fuseholder
- added J15: FemaleHeader P2.54 02x08 THT Straight, Connector_PinSocket_2.54mm:PinSocket_2x08_P2.54mm_Vertical, F.Cu at (41.9, 91.5)
- added U4: 64900001039, NextPCB:Fuseholder, F.Cu at (119.4, 76.2)
- moved J12 73.8 mm to (96.5, 61.0)
- moved J13 73.8 mm to (104.1, 61.0)
- moved J14 73.8 mm to (111.8, 61.0)
- moved U1 62.0 mm to (104.1, 104.1)
- moved U2 51.4 mm to (104.1, 78.7)
- moved K1 50.8 mm to (66.2, 63.1)
- moved K2 50.8 mm to (66.2, 74.5)
- moved K3 50.8 mm to (66.2, 86.0)
- moved K4 50.8 mm to (66.2, 97.4)
- moved K5 50.8 mm to (66.2, 108.8)
- moved K6 50.8 mm to (66.2, 120.3)
- moved K7 50.8 mm to (66.2, 131.7)
- moved K8 50.8 mm to (66.2, 143.1)
- moved H1 50.8 mm to (61.0, 54.6)
- moved H4 50.8 mm to (61.0, 146.1)
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Routing:
- net VDD: track 0.00 -> 231.8 mm, vias 0 -> 3
- net /K1: track 0.00 -> 108.4 mm, vias 0 -> 1
- net /K8: track 0.00 -> 103.4 mm, vias 0 -> 1
- net /K2: track 0.00 -> 88.7 mm, vias 0 -> 1
- net /K7: track 0.00 -> 87.8 mm, vias 0 -> 1
- net GND: track 0.00 -> 85.3 mm, vias 0 -> 5
- net /K6: track 0.00 -> 75.6 mm, vias 0 -> 1
- net /K3: track 0.00 -> 74.4 mm, vias 0 -> 1
- net /K4: track 0.00 -> 68.4 mm, vias 0 -> 1
- net /K5: track 0.00 -> 66.1 mm, vias 0 -> 1
- net /SDA: track 0.00 -> 31.0 mm, vias 0 -> 1
- net /SCL: track 0.00 -> 30.9 mm, vias 0 -> 1
- net Net-(U1-I1): track 0.00 -> 29.3 mm
- net Net-(U1-I8): track 0.00 -> 29.2 mm
- net Net-(U1-I2): track 0.00 -> 29.0 mm
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- added copper zone on B.Cu, net (none)
- added copper zone on F.Cu, net (none)
- removed copper zone on B.Cu, net GND
- removed copper zone on F.Cu, net VDD

Commit message: PM-AI-xxx docs
Parts:
- J9: value PinHeader P2.54 01x08 THT Angle -> Conn_01x04_Pin; footprint Connector_PinHeader_2.54mm:PinHeader_1x08_P2.54mm_Horizontal -> Connector_PinHeader_2.54mm:PinHeader_1x04_P2.54mm_Horizontal
- moved J9 5.08 mm to (120.1, 96.5)
Routing:
- net VDD: track 231.8 -> 216.7 mm, vias 3 -> 0
- net /A0: track 26.3 -> 18.1 mm
- net /K1: track 108.4 -> 103.3 mm
- net Net-(J9-Pin_1): track 8.05 -> 13.1 mm
- net /SCL: track 30.9 -> 36.0 mm
- net /K8: track 103.4 -> 100.4 mm, vias 1 -> 0
- net /SDA: track 31.0 -> 33.8 mm
- net /K4: track 68.4 -> 67.6 mm, vias 1 -> 0
- net /A2: track 25.3 -> 26.1 mm, vias 0 -> 2
- net /K5: track 66.1 -> 65.5 mm, vias 1 -> 0
- net /K6: track 75.6 -> 75.1 mm, vias 1 -> 0
- net Net-(U1-I5): track 28.2 -> 27.7 mm, vias 0 -> 2
- net Net-(U1-I4): track 28.4 -> 27.9 mm, vias 0 -> 2
- net Net-(U1-I3): track 28.7 -> 28.2 mm, vias 0 -> 2
- net Net-(U1-I1): track 29.3 -> 28.7 mm, vias 0 -> 2
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Other:
- board text removed: "CLK"
- board text removed: "CS"
- board text removed: "MISO"
- board text removed: "MOSI"

Commit message: send to nextpcb
Parts:
- removed J12, J13, J14: PinHeader_P2.54_01x03_SMD_Straight, Connector_PinHeader_2.54mm:PinHeader_1x03_P2.54mm_Vertical_SMD_Pin1Left
- removed J15: FemaleHeader P2.54 02x08 THT Straight, Connector_PinSocket_2.54mm:PinSocket_2x08_P2.54mm_Vertical
- removed U4: 64900001039, NextPCB:Fuseholder
- removed logo_kicad: KiCad-Logo2_8mm_SilkScreen, Symbol:KiCad-Logo2_8mm_SilkScreen
- removed logo_oshw: OSHW-Symbol_13.4x12mm_SilkScreen, Symbol:OSHW-Symbol_13.4x12mm_SilkScreen
- added C3: 1uF, Capacitor_SMD:C_1206_3216Metric_Pad1.33x1.80mm_HandSolder, B.Cu at (119.4, 124.5)
- added D1: BAT20J, kicad_inventree_lib:SOD-323_STM-M, F.Cu at (76.2, 61.1)
- added D2: BAT20J, kicad_inventree_lib:SOD-323_STM-M, F.Cu at (76.2, 68.6)
- added D3: BAT20J, kicad_inventree_lib:SOD-323_STM-M, F.Cu at (76.2, 76.2)
- added D4: BAT20J, kicad_inventree_lib:SOD-323_STM-M, F.Cu at (76.2, 83.8)
- added D5: BAT20J, kicad_inventree_lib:SOD-323_STM-M, F.Cu at (76.2, 116.8)
- added D6: BAT20J, kicad_inventree_lib:SOD-323_STM-M, F.Cu at (76.2, 124.5)
- added D7: BAT20J, kicad_inventree_lib:SOD-323_STM-M, F.Cu at (76.2, 132.1)
- added D8: BAT20J, kicad_inventree_lib:SOD-323_STM-M, F.Cu at (76.2, 139.7)
- added J1: ~, kicad_inventree_lib:PM-front-02x04, F.Cu at (39.4, 100.3)
- added J2: PinHeader_01x05_P2.54_THT_angle, Connector_PinHeader_2.54mm:PinHeader_1x05_P2.54mm_Horizontal, F.Cu at (120.7, 95.2)
- added R1: 10k, Resistor_SMD:R_1206_3216Metric_Pad1.30x1.75mm_HandSolder, B.Cu at (119.4, 120.7)
- added SW2: Button, kicad_inventree_lib:SW_TS-1088_XNP-M, B.Cu at (101.6, 142.2)
- added U3: ESP32-C3-WROOM-02U-N4, kicad_inventree_lib:ESP32-C3-WROOM-02U_EXP, B.Cu at (101.7, 125.1)
- added kicad_logo: KiCad-Logo2_5mm_SilkScreen, Symbol:KiCad-Logo2_5mm_SilkScreen, B.Cu at (119.4, 66.0)
- added oshw_logo: OSHW-Symbol_6.7x6mm_SilkScreen, Symbol:OSHW-Symbol_6.7x6mm_SilkScreen, B.Cu at (119.4, 78.7)
- J9: value Conn_01x04_Pin -> U254-051T-4BH83-S1S; footprint Connector_PinHeader_2.54mm:PinHeader_1x04_P2.54mm_Horizontal -> kicad_inventree_lib:CONN5_H83-S1S_XKB; moved to B.Cu
- moved J9 44.2 mm to (113.1, 140.1), turned to 180 degrees
- moved U1 25.7 mm to (78.7, 100.3), turned to 0 degrees
- moved K4 19.4 mm to (50.3, 86.4)
- moved K5 18.9 mm to (50.3, 119.0)
- moved K3 17.5 mm to (50.3, 78.7)
- moved K6 17.2 mm to (50.3, 126.6)
- moved H1 16.5 mm to (44.5, 54.6)
- moved H4 16.5 mm to (44.5, 146.1)
- moved K2 16.3 mm to (50.3, 71.1)
- moved K7 16.2 mm to (50.3, 134.2)
- moved K8 16.0 mm to (50.3, 141.9)
- moved K1 16.0 mm to (50.3, 63.5)
Connections:
- net VDD renamed +5V
- J9 pad 1: Net-(J9-Pin_1) -> unconnected-(J9-VBUS-Pad1)
- J9 pad 2: GND -> /USB_DN
- J9 pad 3: /SDA -> /USB_DP
- J9 pad 4: /SCL -> unconnected-(J9-ID-Pad4)
- K1 pad 2: Net-(J10-Pin_1) -> Net-(J10-Pin_2)
- K1 pad 3: Net-(J10-Pin_2) -> Net-(J10-Pin_1)
- K2 pad 2: Net-(J10-Pin_3) -> Net-(J10-Pin_4)
- K2 pad 3: Net-(J10-Pin_4) -> Net-(J10-Pin_3)
- K3 pad 2: Net-(J10-Pin_5) -> Net-(J10-Pin_6)
- K3 pad 3: Net-(J10-Pin_6) -> Net-(J10-Pin_5)
- K4 pad 2: Net-(J10-Pin_7) -> Net-(J10-Pin_8)
- K4 pad 3: Net-(J10-Pin_8) -> Net-(J10-Pin_7)
- K5 pad 2: Net-(J10-Pin_9) -> Net-(J10-Pin_10)
- K5 pad 3: Net-(J10-Pin_10) -> Net-(J10-Pin_9)
- K6 pad 2: Net-(J10-Pin_11) -> Net-(J10-Pin_12)
- K6 pad 3: Net-(J10-Pin_12) -> Net-(J10-Pin_11)
- K7 pad 2: Net-(J10-Pin_13) -> Net-(J10-Pin_14)
- K7 pad 3: Net-(J10-Pin_14) -> Net-(J10-Pin_13)
- K8 pad 2: Net-(J10-Pin_15) -> Net-(J10-Pin_16)
- K8 pad 3: Net-(J10-Pin_16) -> Net-(J10-Pin_15)
Routing:
- net +5V: track 216.7 -> 0.00 mm
- net /K1: track 103.3 -> 0.00 mm, vias 1 -> 0
- net /K8: track 100.4 -> 0.00 mm
- net /K2: track 88.7 -> 0.00 mm, vias 1 -> 0
- net /K7: track 87.8 -> 0.00 mm
- net GND: track 84.9 -> 0.00 mm
- net /K6: track 75.1 -> 0.00 mm
- net /K3: track 74.2 -> 0.00 mm
- net /K4: track 67.6 -> 0.00 mm
- net /K5: track 65.5 -> 0.00 mm
- net Net-(J10-Pin_9): track 55.9 -> 0.00 mm
- net Net-(J10-Pin_15): track 46.2 -> 0.00 mm
- net Net-(J10-Pin_11): track 46.1 -> 0.00 mm
- net Net-(J10-Pin_13): track 45.7 -> 0.00 mm
- net Net-(J10-Pin_7): track 45.6 -> 0.00 mm
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- added copper zone on B.Cu, net GND
- added copper zone on F.Cu, net GND
- removed copper zone on B.Cu, net (none)
- removed copper zone on F.Cu, net (none)
Other:
- outline, holes or cut-outs redrawn
- board text added: "+3.3V"
- board text removed: "A0"
- board text removed: "A1"
- board text removed: "A2"
- board text removed: "V"

Commit message: PM-PS
Parts:
- added C1: 1uF, Capacitor_SMD:C_1206_3216Metric_Pad1.33x1.80mm_HandSolder, B.Cu at (116.8, 121.9)
- added C2: 10uF, Capacitor_SMD:C_1206_3216Metric_Pad1.33x1.80mm_HandSolder, B.Cu at (109.2, 116.8)
- added R2: 10k, Resistor_SMD:R_1206_3216Metric_Pad1.30x1.75mm_HandSolder, B.Cu at (116.8, 132.1)
- added R3: 330R, Resistor_SMD:R_1206_3216Metric_Pad1.30x1.75mm_HandSolder, B.Cu at (116.8, 137.2)
- added R4: 10k, Resistor_SMD:R_1206_3216Metric_Pad1.30x1.75mm_HandSolder, B.Cu at (116.8, 127.0)
- added R5: 10k, Resistor_SMD:R_1206_3216Metric_Pad1.30x1.75mm_HandSolder, B.Cu at (86.4, 124.5)
- added SW4: Button, kicad_inventree_lib:SW_TS-1088_XNP-M, B.Cu at (94.0, 142.2)
- moved C3 19.3 mm to (101.6, 116.8), turned to 180 degrees
- moved R1 4.58 mm to (116.8, 116.8)
- moved U3 2.56 mm to (101.5, 127.7)
Connections:
- net /USB_DN renamed /ESP32/USB_DN
- net /USB_DP renamed /ESP32/USB_DP
- C3 pad 1: /MCU_EN -> +3.3V
- R1 pad 2: /MCU_EN -> /ESP32/EN
- SW2 pad 2: /MCU_EN -> Net-(R3-Pad2)
- U3 pad 10: unconnected-(U3-IO10-Pad10) -> /ESP32/GPIO10
- U3 pad 15: unconnected-(U3-IO3-Pad15) -> /ESP32/GPIO3
- U3 pad 16: unconnected-(U3-IO2-Pad16) -> /ESP32/GPIO2
- U3 pad 17: unconnected-(U3-IO1-Pad17) -> /ESP32/GPIO1
- U3 pad 18: unconnected-(U3-IO0-Pad18) -> /ESP32/GPIO0
- U3 pad 2: /MCU_EN -> /ESP32/EN
- U3 pad 3: unconnected-(U3-IO4-Pad3) -> /ESP32/GPIO4
- U3 pad 4: unconnected-(U3-IO5-Pad4) -> /ESP32/GPIO5
- U3 pad 5: unconnected-(U3-IO6-Pad5) -> /ESP32/GPIO6
- U3 pad 6: unconnected-(U3-IO7-Pad6) -> /ESP32/GPIO7
- U3 pad 7: unconnected-(U3-IO8-Pad7) -> /ESP32/GPIO8
- U3 pad 8: unconnected-(U3-IO9-Pad8) -> /ESP32/GPIO9
- U3 pad 9: unconnected-(U3-GND-Pad9) -> GND
- U3 pad EPAD: unconnected-(U3-PadEPAD) -> GND
Routing:
- net /ESP32/USB_DN: track 28.7 -> 0.00 mm
- net /ESP32/USB_DP: track 28.6 -> 0.00 mm

Commit message: PM-RQ8
Parts:
- removed H4: MountingHole, MountingHole:MountingHole_3.2mm_M3
- removed U2: PCA9555PW, Package_SO:TSSOP-24_4.4x7.8mm_P0.65mm
- added PE1: PE, kicad_inventree_lib:PE, F.Cu at (44.5, 146.1)
- added R6: 10k, Resistor_SMD:R_1206_3216Metric_Pad1.30x1.75mm_HandSolder, B.Cu at (77.7, 153.4)
- added R7: 10k, Resistor_SMD:R_1206_3216Metric_Pad1.30x1.75mm_HandSolder, B.Cu at (77.7, 156.7)
- added R8: 10k, Resistor_SMD:R_1206_3216Metric_Pad1.30x1.75mm_HandSolder, B.Cu at (77.7, 160.0)
- added SW5: DIP_SW-3P-P2.54-THT-Top, Button_Switch_THT:SW_DIP_SPSTx03_Slide_9.78x9.8mm_W7.62mm_P2.54mm, B.Cu at (108.0, 135.9)
- added U6: MCP23S17_ML, Package_DFN_QFN:QFN-28-1EP_6x6mm_P0.65mm_EP4.25x4.25mm, F.Cu at (97.8, 100.3)
- K1, K2, K3, K4, K5, K6, K7, K8: footprint NextPCB:G5NB-1A-E_DC12_RELAY_G5NB-1A_DC5_OMR -> kicad_inventree_lib:G5NB-1A-E_DC12_RELAY_G5NB-1A_DC5_OMR
- moved J9 25.4 mm to (87.7, 140.1)
- moved SW4 20.9 mm to (114.3, 137.2)
- moved SW2 18.5 mm to (119.4, 137.2)
- moved R2 5.08 mm to (116.8, 127.0)
- moved U3 5.08 mm to (101.5, 122.6)
- moved C1 5.08 mm to (116.8, 116.8)
- moved C2 5.08 mm to (109.2, 111.8)
- moved C3 5.08 mm to (101.6, 111.8)
- moved R1 5.08 mm to (116.8, 111.8)
- moved R4 5.08 mm to (116.8, 121.9)
- moved R5 5.08 mm to (86.4, 119.4)
- moved R3 5.08 mm to (116.8, 132.1)
Connections:
- net /ESP32/GPIO2 renamed /MOSI
- J10 pad 17: unconnected-(J10-Pin_17-Pad17) -> /PE
- J10 pad 18: unconnected-(J10-Pin_18-Pad18) -> /PE
- U3 pad 15: /ESP32/GPIO3 -> /MISO
- U3 pad 17: /ESP32/GPIO1 -> /SCL
- U3 pad 18: /ESP32/GPIO0 -> /SDA
- U3 pad 3: /ESP32/GPIO4 -> /SCK
- U3 pad 4: /ESP32/GPIO5 -> /CS
- U3 pad 5: /ESP32/GPIO6 -> /INT
Routing:
- net Net-(J10-Pin_10): track 0.00 -> 32.7 mm
- net Net-(J10-Pin_8): track 0.00 -> 32.1 mm
- net Net-(J10-Pin_12): track 0.00 -> 31.3 mm
- net Net-(J10-Pin_9): track 0.00 -> 30.8 mm
- net Net-(J10-Pin_6): track 0.00 -> 30.7 mm
- net Net-(J10-Pin_14): track 0.00 -> 30.2 mm
- net Net-(J10-Pin_4): track 0.00 -> 29.6 mm
- net Net-(J10-Pin_16): track 0.00 -> 29.1 mm
- net Net-(J10-Pin_2): track 0.00 -> 28.5 mm
- net Net-(J10-Pin_11): track 0.00 -> 25.0 mm
- net Net-(J10-Pin_13): track 0.00 -> 23.8 mm
- net Net-(J10-Pin_15): track 0.00 -> 22.8 mm
- net Net-(J10-Pin_7): track 0.00 -> 22.6 mm
- net Net-(J10-Pin_5): track 0.00 -> 21.5 mm
- net Net-(J10-Pin_3): track 0.00 -> 20.5 mm
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- added copper zone on B.Cu, net /PE
- added copper zone on F.Cu, net /PE
Other:
- board text added: "1"
- board text added: "2"
- board text added: "20+"
- board text added: "4"
- board text added: "Address"
- board text added: "OFF"
- board text added: "ON"

Commit message: PM-ESPC3
Parts:
- added REF**: PinHeader_1x13_P2.54mm_Vertical, Connector_PinHeader_2.54mm:PinHeader_1x13_P2.54mm_Vertical, F.Cu at (120.7, 61.0)
- added SW5: DIP_SW-3P-P2.54-THT-Top, Button_Switch_THT:SW_DIP_SPSTx03_Slide_9.78x9.8mm_W7.62mm_P2.54mm, B.Cu at (114.3, 55.9)
- moved R8 106.3 mm to (99.1, 55.9), turned to -90 degrees
- moved R7 102.2 mm to (94.0, 55.9), turned to -90 degrees
- moved R6 98.2 mm to (88.9, 55.9), turned to -90 degrees
- moved J9 83.4 mm to (105.4, 58.6), turned to 0 degrees
- moved kicad_logo 81.3 mm to (99.1, 144.8), turned to 180 degrees
- moved SW5 69.5 mm to (96.5, 67.3)
- moved R5 69.4 mm to (114.3, 55.9), turned to -90 degrees
- moved oshw_logo 66.5 mm to (111.8, 144.8), turned to 180 degrees
- moved SW2 59.2 mm to (88.9, 86.4), turned to -90 degrees
- moved U3 52.1 mm to (108.6, 71.0), turned to 90 degrees
- moved R3 51.1 mm to (94.0, 86.4), turned to -90 degrees
- moved SW4 51.1 mm to (119.4, 86.4)
- moved C3 44.4 mm to (119.4, 71.1), turned to 90 degrees
- moved R2 44.4 mm to (99.1, 86.4), turned to 90 degrees
- moved R4 37.8 mm to (104.1, 86.4), turned to 90 degrees
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Connections:
- J10 pad 10: Net-(J10-Pin_10) -> /PE
- J10 pad 17: /PE -> Net-(J10-Pin_17)
- J10 pad 18: /PE -> Net-(J10-Pin_18)
- J10 pad 9: Net-(J10-Pin_9) -> /PE
- J2 pad 1: +5V -> /SDA
- J2 pad 2: +3.3V -> /SCL
- J2 pad 3: GND -> +5V
- J2 pad 4: /SDA -> +3.3V
- J2 pad 5: /SCL -> GND
- K5 pad 2: Net-(J10-Pin_10) -> Net-(J10-Pin_12)
- K5 pad 3: Net-(J10-Pin_9) -> Net-(J10-Pin_11)
- K6 pad 2: Net-(J10-Pin_12) -> Net-(J10-Pin_14)
- K6 pad 3: Net-(J10-Pin_11) -> Net-(J10-Pin_13)
- K7 pad 2: Net-(J10-Pin_14) -> Net-(J10-Pin_16)
- K7 pad 3: Net-(J10-Pin_13) -> Net-(J10-Pin_15)
- K8 pad 2: Net-(J10-Pin_16) -> Net-(J10-Pin_18)
- K8 pad 3: Net-(J10-Pin_15) -> Net-(J10-Pin_17)
- R4 pad 2: /ESP32/GPIO8 -> /CS
- R5 pad 2: /MOSI -> /ESP32/GPIO2
- U1 pad 1: Net-(U1-I1) -> /K8_exp
- U1 pad 11: /K8 -> /K1
- U1 pad 12: /K7 -> /K2
- U1 pad 13: /K6 -> /K3
- U1 pad 14: /K5 -> /K4
- U1 pad 15: /K4 -> /K5
- U1 pad 16: /K3 -> /K6
- U1 pad 17: /K2 -> /K7
- U1 pad 18: /K1 -> /K8
- U1 pad 2: Net-(U1-I2) -> /K7_exp
- U1 pad 3: Net-(U1-I3) -> /K6_exp
- U1 pad 4: Net-(U1-I4) -> /K5_exp
- U1 pad 5: Net-(U1-I5) -> /K4_exp
- U1 pad 6: Net-(U1-I6) -> /K3_exp
- U1 pad 7: Net-(U1-I7) -> /K2_exp
- U1 pad 8: Net-(U1-I8) -> /K1_exp
- U3 pad 10: /ESP32/GPIO10 -> /ESP32/A1
- U3 pad 11: unconnected-(U3-RXD-Pad11) -> /ESP32/A2
- U3 pad 12: unconnected-(U3-TXD-Pad12) -> /ESP32/A3
- U3 pad 15: /MISO -> /INT
- U3 pad 16: /MOSI -> /ESP32/GPIO2
- U3 pad 3: /SCK -> /MOSI
- U3 pad 4: /CS -> /MISO
- U3 pad 5: /INT -> /SCK
- U3 pad 7: /ESP32/GPIO8 -> /CS
- U6 pad 17: Net-(U1-I1) -> /K1_exp
- U6 pad 18: Net-(U1-I2) -> /K2_exp
- U6 pad 19: Net-(U1-I3) -> /K3_exp
- U6 pad 20: Net-(U1-I4) -> /K4_exp
- U6 pad 21: Net-(U1-I5) -> /K5_exp
- U6 pad 22: Net-(U1-I6) -> /K6_exp
- U6 pad 23: Net-(U1-I7) -> /K7_exp
- U6 pad 24: Net-(U1-I8) -> /K8_exp
Routing:
- net +5V: track 0.00 -> 201.8 mm
- net +3.3V: track 0.00 -> 130.7 mm
- net /K1: track 0.00 -> 46.0 mm
- net /K8: track 0.00 -> 43.0 mm, vias 0 -> 1
- net /SCL: track 0.00 -> 42.4 mm
- net /K2: track 0.00 -> 39.7 mm
- net /INT: track 0.00 -> 39.2 mm, vias 0 -> 1
- net /K7: track 0.00 -> 37.3 mm, vias 0 -> 1
- net /SDA: track 0.00 -> 35.6 mm, vias 0 -> 1
- net /K3: track 0.00 -> 33.3 mm
- net /K6: track 0.00 -> 32.9 mm
- net Net-(J10-Pin_10): track 32.7 -> 0.00 mm
- net Net-(J10-Pin_9): track 30.8 -> 0.00 mm
- net Net-(J10-Pin_18): track 0.00 -> 29.8 mm
- net /K4: track 0.00 -> 26.8 mm
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
Commit message: PM-ESPC3
Parts:
- removed C1, C3: 1uF, Capacitor_SMD:C_1206_3216Metric_Pad1.33x1.80mm_HandSolder
- removed C2: 10uF, Capacitor_SMD:C_1206_3216Metric_Pad1.33x1.80mm_HandSolder
- removed J9: U254-051T-4BH83-S1S, kicad_inventree_lib:CONN5_H83-S1S_XKB
- removed R1, R2, R4, R5, R6, R7, R8: 10k, Resistor_SMD:R_1206_3216Metric_Pad1.30x1.75mm_HandSolder
- removed R3: 330R, Resistor_SMD:R_1206_3216Metric_Pad1.30x1.75mm_HandSolder
- removed REF**: PinHeader_1x13_P2.54mm_Vertical, Connector_PinHeader_2.54mm:PinHeader_1x13_P2.54mm_Vertical
- removed SW2, SW4: Button, kicad_inventree_lib:SW_TS-1088_XNP-M
- removed SW5 (x2): DIP_SW-3P-P2.54-THT-Top, Button_Switch_THT:SW_DIP_SPSTx03_Slide_9.78x9.8mm_W7.62mm_P2.54mm
- removed U3: ESP32-C3-WROOM-02U-N4, kicad_inventree_lib:ESP32-C3-WROOM-02U_EXP
- added PM1: ~, kicad_inventree_lib:PM-ESP32C3, B.Cu at (106.7, 50.8)
Routing:
- net +5V: track 201.8 -> 0.00 mm
- net +3.3V: track 130.7 -> 0.00 mm
- net /K1: track 46.0 -> 0.00 mm
- net /K8: track 43.0 -> 0.00 mm, vias 1 -> 0
- net /SCL: track 42.4 -> 0.00 mm
- net /K2: track 39.7 -> 0.00 mm
- net /INT: track 39.2 -> 0.00 mm, vias 1 -> 0
- net /K7: track 37.3 -> 0.00 mm, vias 1 -> 0
- net /SDA: track 35.6 -> 0.00 mm, vias 1 -> 0
- net /K3: track 33.3 -> 0.00 mm
- net /K6: track 32.9 -> 0.00 mm
- net /K4: track 26.8 -> 0.00 mm
- net /K5: track 25.2 -> 0.00 mm, vias 1 -> 0
- net /ESP32/A1: track 24.6 -> 0.00 mm
- net /ESP32/A2: track 24.5 -> 0.00 mm
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Other:
- outline, holes or cut-outs redrawn
- board text removed: "Address"
