File: PM-DI16-DC24sink/PM-DI16-DC24sink.kicad_pcb (KiCad board)
At the start: 2 copper layers, 99.1 x 99.1 mm, 87 parts, among them J2 2EDGR-5.08-18P, J3 Conn_01x04_Pin, J4 PinHeader P2.54 01x12 THT Str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, J5 PinHeader P2.54 01x12 THT Str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, U1 MCP23S17_ML, U10 Weact ESP32-C3FH4, U2 ISO1212DBQ, U3 ISO1212DBQ, U4 ISO1212DBQ, U5 ISO1212DBQ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

Commit message: PM-DI16-DC24sink
Parts:
- removed J1: ~, kicad_inventree_lib:PM-front-02x08
- added J6: ~, kicad_inventree_lib:PM-front-02x10, F.Cu at (40.6, 88.9)
- added R36: 10k, Resistor_SMD:R_1206_3216Metric_Pad1.30x1.75mm_HandSolder, B.Cu at (82.3, 130.6)
- added R37: 10k, Resistor_SMD:R_1206_3216Metric_Pad1.30x1.75mm_HandSolder, B.Cu at (82.3, 133.9)
- added R38: 10k, Resistor_SMD:R_1206_3216Metric_Pad1.30x1.75mm_HandSolder, B.Cu at (82.3, 137.2)
- added R39: 10k, Resistor_SMD:R_1206_3216Metric_Pad1.30x1.75mm_HandSolder, B.Cu at (82.3, 140.4)
- added R40: 10k, Resistor_SMD:R_1206_3216Metric_Pad1.30x1.75mm_HandSolder, B.Cu at (82.3, 143.7)
- added R41: 100, Resistor_SMD:R_1206_3216Metric_Pad1.30x1.75mm_HandSolder, F.Cu at (120.4, 83.8)
- added SW1: DSIC05LS-P, kicad_inventree_lib:DSIC05LS-P, B.Cu at (55.0, 137.2)
- J3: value Conn_01x04_Pin -> PinHeader_01x05_P2.54_THT_angle; footprint Connector_PinHeader_2.54mm:PinHeader_1x04_P2.54mm_Horizontal -> Connector_PinHeader_2.54mm:PinHeader_1x05_P2.54mm_Horizontal
- moved C1 5.08 mm to (66.0, 55.9)
- moved C19 5.08 mm to (66.0, 63.5)
- moved C2 5.08 mm to (66.0, 71.1)
- moved C20 5.08 mm to (66.0, 55.9)
- moved C23 5.08 mm to (66.0, 78.7)
- moved C24 5.08 mm to (66.0, 71.1)
- moved C27 5.08 mm to (66.0, 94.0)
- moved C28 5.08 mm to (66.0, 86.4)
- moved C3 5.08 mm to (66.0, 86.4)
- moved C31 5.08 mm to (66.0, 109.2)
- moved C32 5.08 mm to (66.0, 101.6)
- moved C4 5.08 mm to (66.0, 101.6)
- moved C5 5.08 mm to (66.0, 63.5)
- moved C6 5.08 mm to (66.0, 78.7)
- moved C7 5.08 mm to (66.0, 94.0)
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Connections:
- J3 pad 2: GND -> unconnected-(J3-Pin_2-Pad2)
- J3 pad 3: /SDA -> GND
- J3 pad 4: /SCL -> /SDA
- J4 pad 7: /RST -> /A1
- J4 pad 8: unconnected-(J4-Pin_8-Pad8) -> /A2
- J5 pad 5: unconnected-(J5-Pin_5-Pad5) -> /A5
- J5 pad 6: unconnected-(J5-Pin_6-Pad6) -> /A4
- J5 pad 7: unconnected-(J5-Pin_7-Pad7) -> /A3
- U1 pad 9: /MISO -> Net-(U1-SI)
Routing:
- net +5V: track 0.00 -> 246.3 mm, vias 0 -> 4
- net /OUT01: track 0.00 -> 170.1 mm, vias 0 -> 2
- net /OUT10: track 0.00 -> 157.5 mm, vias 0 -> 2
- net /OUT09: track 0.00 -> 155.7 mm, vias 0 -> 2
- net /OUT02: track 0.00 -> 154.2 mm, vias 0 -> 2
- net /OUT14: track 0.00 -> 142.9 mm, vias 0 -> 1
- net /OUT03: track 0.00 -> 139.0 mm, vias 0 -> 1
- net /OUT11: track 0.00 -> 138.5 mm, vias 0 -> 3
- net /OUT12: track 0.00 -> 137.7 mm, vias 0 -> 2
- net /OUT04: track 0.00 -> 134.9 mm, vias 0 -> 1
- net /OUT13: track 0.00 -> 124.5 mm, vias 0 -> 1
- net /OUT05: track 0.00 -> 121.4 mm, vias 0 -> 1
- net /OUT06: track 0.00 -> 121.1 mm, vias 0 -> 2
- net /OUT16: track 0.00 -> 116.8 mm, vias 0 -> 1
- net /OUT15: track 0.00 -> 113.6 mm, vias 0 -> 2
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Other:
- copper layers 2 -> 4
- board text added: "1"
- board text added: "16"
- board text added: "2"
- board text added: "4"
- board text added: "8"
- board text added: "Address"
- board text added: "OFF"
- board text added: "ON"

Commit message: PM-DI16-DC24sink
Parts:
- removed H4: MountingHole, MountingHole:MountingHole_3.2mm_M3
- removed J6: ~, kicad_inventree_lib:PM-front-02x10
- removed R33, R34, R35, R41: 100, Resistor_SMD:R_1206_3216Metric_Pad1.30x1.75mm_HandSolder
- removed R39, R40: 10k, Resistor_SMD:R_1206_3216Metric_Pad1.30x1.75mm_HandSolder
- added C33: 4.7nF 2kV, Capacitor_SMD:C_1812_4532Metric_Pad1.57x3.40mm_HandSolder, B.Cu at (39.4, 137.2)
- added D2: ~, kicad_inventree_lib:PE, F.Cu at (44.5, 146.1)
- added J1: ~, kicad_inventree_lib:PM-front-02x08, F.Cu at (40.6, 91.4)
- added REF**: OSHW-Symbol_6.7x6mm_SilkScreen, Symbol:OSHW-Symbol_6.7x6mm_SilkScreen, B.Cu at (97.8, 54.6)
- added REF**: KiCad-Logo2_5mm_SilkScreen, Symbol:KiCad-Logo2_5mm_SilkScreen, B.Cu at (109.2, 54.6)
- SW1: value DSIC05LS-P -> DSIC03LS-P; footprint kicad_inventree_lib:DSIC05LS-P -> kicad_inventree_lib:DSIC03LS-P
- moved R38 36.6 mm to (114.3, 119.4)
- moved R37 33.4 mm to (114.3, 124.5)
- moved R36 32.0 mm to (114.3, 129.5)
- moved SW1 14.4 mm to (69.4, 137.2), turned to 90 degrees
- moved C17 7.62 mm to (91.4, 66.0)
- moved C18 7.62 mm to (96.5, 66.0)
- moved C19 7.62 mm to (66.0, 71.1)
- moved C21 7.62 mm to (91.4, 81.3)
- moved C22 7.62 mm to (96.5, 81.3)
- moved C23 7.62 mm to (66.0, 86.4)
- moved C28 7.62 mm to (66.0, 94.0)
- moved C29 7.62 mm to (91.4, 111.8)
- moved C30 7.62 mm to (96.5, 111.8)
- moved C31 7.62 mm to (66.0, 116.8)
- moved C32 7.62 mm to (66.0, 109.2)
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Connections:
- J4 pad 3: Net-(J4-Pin_3) -> /MOSI
- J4 pad 5: Net-(J4-Pin_5) -> /CLK
- J4 pad 6: Net-(J4-Pin_6) -> /CS1
- J4 pad 7: /A1 -> /INT
- J4 pad 8: /A2 -> /CS2
- J5 pad 5: /A5 -> /A3
- J5 pad 6: /A4 -> /A2
- J5 pad 7: /A3 -> /A1
- R19 pad 1: /IN09 -> /IN03
- R20 pad 1: /IN10 -> /IN04
- R23 pad 1: /IN11 -> /IN07
- R24 pad 1: /IN12 -> /IN08
- R27 pad 1: /IN13 -> /IN11
- R28 pad 1: /IN14 -> /IN12
- R3 pad 1: /IN03 -> /IN05
- R4 pad 1: /IN04 -> /IN06
- R5 pad 1: /IN05 -> /IN09
- R6 pad 1: /IN06 -> /IN10
- R7 pad 1: /IN07 -> /IN13
- R8 pad 1: /IN08 -> /IN14
- SW1 pad 1: /A5 -> /A3
- SW1 pad 2: /A4 -> /A2
- SW1 pad 3: /A3 -> /A1
- SW1 pad 4: /A2 -> +3.3V
- SW1 pad 5: /A1 -> +3.3V
- U1 pad 16: unconnected-(U1-INTA-Pad16) -> /INT
- U1 pad 9: Net-(U1-SI) -> /MISO
- U3 pad 4: /OUT04 -> /OUT06
- U3 pad 5: /OUT03 -> /OUT05
- U4 pad 4: /OUT06 -> /OUT10
- U4 pad 5: /OUT05 -> /OUT09
- U5 pad 4: /OUT08 -> /OUT14
- U5 pad 5: /OUT07 -> /OUT13
- U6 pad 4: /OUT09 -> /OUT03
- U6 pad 5: /OUT10 -> /OUT04
- U7 pad 4: /OUT11 -> /OUT07
- U7 pad 5: /OUT12 -> /OUT08
- U8 pad 4: /OUT13 -> /OUT11
- U8 pad 5: /OUT14 -> /OUT12
Routing:
- net /OUT01: track 170.1 -> 41.2 mm, vias 2 -> 0
- net /OUT10: track 157.5 -> 30.4 mm, vias 2 -> 0
- net /OUT09: track 155.7 -> 30.4 mm, vias 2 -> 0
- net /MOSI: track 37.1 -> 154.7 mm, vias 1 -> 2
- net /CLK: track 40.3 -> 156.8 mm, vias 1 -> 2
- net /MISO: track 41.3 -> 157.3 mm
- net /OUT02: track 154.2 -> 40.4 mm, vias 2 -> 0
- net /CS2: track 0.00 -> 113.0 mm
- net /OUT11: track 138.5 -> 33.3 mm, vias 3 -> 1
- net /OUT12: track 137.7 -> 33.0 mm, vias 2 -> 1
- net /OUT03: track 139.0 -> 35.1 mm
- net /OUT14: track 142.9 -> 40.4 mm, vias 1 -> 0
- net /OUT04: track 134.9 -> 34.2 mm
- net +5V: track 246.3 -> 346.5 mm, vias 4 -> 5
- net /OUT05: track 121.4 -> 30.4 mm, vias 1 -> 0
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- added copper zone on B.Cu, net PE
- added copper zone on F.Cu, net PE
Other:
- outline, holes or cut-outs redrawn
- copper layers 4 -> 2
- board text added: "+3.3V"
- board text added: "+5V"
- board text added: "10+"
- board text added: "GND"
- board text added: "PE"
- board text added: "PM-DI16-DC24sink v0.0.1"
- board text added: "SCL"
- board text added: "SDA"
- board text removed: "16"
- board text removed: "8"

Commit message: send to nextpcb
Parts:
- removed J1: ~, kicad_inventree_lib:PM-front-02x08
- removed REF**: OSHW-Symbol_6.7x6mm_SilkScreen, Symbol:OSHW-Symbol_6.7x6mm_SilkScreen
- removed REF**: KiCad-Logo2_5mm_SilkScreen, Symbol:KiCad-Logo2_5mm_SilkScreen
- removed U1: MCP23S17_ML, Package_DFN_QFN:QFN-28-1EP_6x6mm_P0.65mm_EP4.25x4.25mm
- added J6: ~, kicad_inventree_lib:PM-front-02x04, F.Cu at (39.4, 100.3)
- added U11: MCP23S17_ML, Package_DFN_QFN:QFN-28-1EP_6x6mm_P0.65mm_EP4.25x4.25mm, F.Cu at (114.3, 81.3)
- SW1: value DSIC03LS-P -> DIP_SW-3P-P2.54-THT-Top; footprint kicad_inventree_lib:DSIC03LS-P -> Button_Switch_THT:SW_DIP_SPSTx03_Slide_9.78x9.8mm_W7.62mm_P2.54mm
- moved SW1 1.52 mm to (68.6, 135.9), turned to 180 degrees
Connections:
- SW1 pad 1: /A3 -> /A1
- SW1 pad 3: /A1 -> /A3
Routing:
- net /IN14: track 78.6 -> 68.4 mm
- net /IN13: track 67.3 -> 57.5 mm
- net /IN16: track 96.3 -> 86.7 mm
- net /IN15: track 85.1 -> 76.1 mm
- net /IN12: track 63.8 -> 55.3 mm
- net /A3: track 50.7 -> 58.3 mm, vias 1 -> 0
- net /IN10: track 46.0 -> 38.7 mm
- net /A1: track 56.1 -> 48.9 mm, vias 1 -> 0
- net /IN11: track 52.6 -> 45.4 mm
- net /MISO: track 157.3 -> 151.4 mm
- net /IN09: track 38.4 -> 34.0 mm
- net /A2: track 49.6 -> 53.5 mm, vias 1 -> 0
- net /IN08: track 34.1 -> 30.7 mm
- net /MOSI: track 154.7 -> 151.9 mm
- net /CLK: track 156.8 -> 159.1 mm
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
Commit message: PM-DI16
Parts:
- removed D1: B5819W, Diode_SMD:D_SOD-123
- removed D2: ~, kicad_inventree_lib:PE
- removed J3: PinHeader_01x05_P2.54_THT_angle, Connector_PinHeader_2.54mm:PinHeader_1x05_P2.54mm_Horizontal
- removed J4, J5: PinHeader P2.54 01x12 THT Straight, Connector_PinHeader_2.54mm:PinHeader_1x12_P2.54mm_Vertical
- removed R36, R37, R38: 10k, Resistor_SMD:R_1206_3216Metric_Pad1.30x1.75mm_HandSolder
- removed SW1: DIP_SW-3P-P2.54-THT-Top, Button_Switch_THT:SW_DIP_SPSTx03_Slide_9.78x9.8mm_W7.62mm_P2.54mm
- removed U10: Weact ESP32-C3FH4, kicad_inventree_lib:Weact ESP32-C3FH4
- added J1: PinHeader_01x05_P2.54_THT_angle, Connector_PinHeader_2.54mm:PinHeader_1x05_P2.54mm_Horizontal, F.Cu at (120.7, 95.2)
- added PE1: PE, kicad_inventree_lib:PE, F.Cu at (44.5, 146.1)
- added PM1: ~, kicad_inventree_lib:PM-ESP32C3, B.Cu at (106.7, 50.8)
- C33: moved to F.Cu
- moved U11 30.6 mm to (111.8, 111.8)
- moved C12 27.9 mm to (96.5, 132.1)
- moved C16 27.9 mm to (91.4, 132.1)
- moved C24 27.9 mm to (66.0, 106.7)
- moved C6 27.9 mm to (66.0, 106.7)
- moved R12 27.9 mm to (71.1, 106.7)
- moved R21 27.9 mm to (71.1, 106.7)
- moved R23 27.9 mm to (58.4, 106.7)
- moved R4 27.9 mm to (58.4, 106.7)
- moved U5 27.9 mm to (81.3, 132.1)
- moved C10 27.9 mm to (96.5, 101.6)
- moved C11 27.9 mm to (96.5, 116.8)
- moved C13 27.9 mm to (91.4, 86.4)
- moved C14 27.9 mm to (91.4, 101.6)
- moved C15 27.9 mm to (91.4, 116.8)
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Connections:
- J6 pad 1: +5V -> +3.3V
- J6 pad 2: /MOSI -> +3.3V
- J6 pad 3: unconnected-(J6-Pad3) -> /MOSI
- J6 pad 4: /MISO -> /SCK
- J6 pad 5: unconnected-(J6-Pad5) -> /MISO
- J6 pad 6: /CLK -> /CS2
- J6 pad 8: /CS2 -> GND
- U11 pad 10: /MOSI -> /MISO
- U11 pad 5: +5V -> +3.3V
- U11 pad 7: /CS -> /CS1
- U11 pad 8: /CLK -> /SCK
- U11 pad 9: /MISO -> /MOSI
Routing:
- net /CLK: track 159.1 -> 0.00 mm, vias 2 -> 0
- net /SCK: track 0.00 -> 142.6 mm, vias 0 -> 1
- net +5V: track 347.2 -> 245.9 mm, vias 3 -> 4
- net +3.3V: track 54.9 -> 141.1 mm, vias 0 -> 1
- net /IN01: track 28.6 -> 96.3 mm
- net /A3: track 58.3 -> 0.00 mm
- net /IN02: track 26.9 -> 85.1 mm
- net /IN16: track 86.7 -> 32.2 mm
- net /A2: track 53.5 -> 0.00 mm
- net /IN03: track 28.0 -> 78.6 mm
- net /A1: track 48.9 -> 0.00 mm
- net /CS1: track 0.00 -> 48.9 mm, vias 0 -> 1
- net /IN15: track 76.1 -> 30.1 mm
- net /IN04: track 26.9 -> 67.3 mm
- net /IN14: track 68.4 -> 32.2 mm
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Other:
- board text removed: "1"
- board text removed: "10+"
- board text removed: "2"
- board text removed: "4"
- board text removed: "Address"
- board text removed: "OFF"
- board text removed: "ON"

Commit message: PM-RQ8
Parts:
- added kicad_logo: KiCad-Logo2_5mm_SilkScreen, Symbol:KiCad-Logo2_5mm_SilkScreen, B.Cu at (120.7, 125.7)
- added oshw_logo: OSHW-Symbol_6.7x6mm_SilkScreen, Symbol:OSHW-Symbol_6.7x6mm_SilkScreen, B.Cu at (120.7, 138.4)
Routing:
- net GND: vias 12 -> 18
Other:
- outline, holes or cut-outs redrawn
- board text added: "0V"
- board text added: "1"
- board text added: "10+"
- board text added: "2"
- board text added: "4"
- board text added: "CS"
- board text added: "MISO"
- board text added: "MOSI"
- board text added: "OFF"
- board text added: "ON"
- board text added: "PM-DI16-DC24sink v0.0.2"
- board text added: "SCK"
- board text added: "a.0"
- board text added: "a.1"
- board text added: "a.2"
- board text added: "a.3"
- board text added: "a.4"
- board text added: "a.5"
- board text added: "a.6"
- board text added: "a.7"
- board text added: "b.0"
- board text added: "b.1"
- board text added: "b.2"
- board text added: "b.3"
- board text added: "b.4"
- board text added: "b.5"
- board text added: "b.6"
- board text added: "b.7"
- board text removed: "PM-DI16-DC24sink v0.0.1"

Commit message: send to nextpcb
Connections:
- C10 pad 2: +5V -> +3.3V
- C11 pad 2: +5V -> +3.3V
- C12 pad 2: +5V -> +3.3V
- C13 pad 2: +5V -> +3.3V
- C14 pad 2: +5V -> +3.3V
- C15 pad 2: +5V -> +3.3V
- C16 pad 2: +5V -> +3.3V
- C17 pad 1: +5V -> +3.3V
- C18 pad 1: +5V -> +3.3V
- C21 pad 1: +5V -> +3.3V
- C22 pad 1: +5V -> +3.3V
- C25 pad 1: +5V -> +3.3V
- C26 pad 1: +5V -> +3.3V
- C29 pad 1: +5V -> +3.3V
- C30 pad 1: +5V -> +3.3V
- C9 pad 2: +5V -> +3.3V
- U11 pad 14: +5V -> +3.3V
- U2 pad 2: +5V -> +3.3V
- U2 pad 3: +5V -> +3.3V
- U3 pad 2: +5V -> +3.3V
- U3 pad 3: +5V -> +3.3V
- U4 pad 2: +5V -> +3.3V
- U4 pad 3: +5V -> +3.3V
- U5 pad 2: +5V -> +3.3V
- U5 pad 3: +5V -> +3.3V
- U6 pad 2: +5V -> +3.3V
- U6 pad 3: +5V -> +3.3V
- U7 pad 2: +5V -> +3.3V
- U7 pad 3: +5V -> +3.3V
- U8 pad 2: +5V -> +3.3V
- U8 pad 3: +5V -> +3.3V
- U9 pad 2: +5V -> +3.3V
- U9 pad 3: +5V -> +3.3V
Routing:
- net +5V: track 245.9 -> 0.00 mm, vias 4 -> 0
- net +3.3V: track 141.1 -> 368.2 mm, vias 1 -> 2
- net /MOSI: track 160.9 -> 150.4 mm, vias 0 -> 1
- net /SCK: track 142.5 -> 150.2 mm, vias 1 -> 2
- net /OUT11: track 29.4 -> 32.9 mm
- net /MISO: track 158.9 -> 156.4 mm, vias 0 -> 1
- net /OUT16: track 42.1 -> 39.7 mm
- net /OUT15: track 41.3 -> 42.8 mm
- net /CS1: track 48.9 -> 47.4 mm
- net /CS2: track 104.0 -> 102.7 mm
- net /OUT04: track 32.7 -> 33.3 mm
- net /INT: track 36.0 -> 35.9 mm, vias 1 -> 0
- net GND: vias 18 -> 19
