File: PM-DI16-DC24sink/PM-DI16-DC24sink.kicad_sch (KiCad schematic)
At the start: 15 parts, among them J2 2EDGR-5.08-18P, J3 Conn_01x04_Pin, J4 PinHeader P2.54 01x12 THT Str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, J5 PinHeader P2.54 01x12 THT Str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, U1 MCP23S17_ML, U10 Weact ESP32-C3FH4

Commit message: PM-DI16-DC24sink
Parts:
- removed J1: ~, kicad_inventree_lib:PM-front-02x08, symbol kicad_inventree_lib:PM-front-02x08
- removed J3: Conn_01x04_Pin, Connector_PinHeader_2.54mm:PinHeader_1x04_P2.54mm_Horizontal, symbol kicad_inventree_lib:PinHeader P2.54 01x04 THT Angle
- added J3: PinHeader_01x05_P2.54_THT_angle, Connector_PinHeader_2.54mm:PinHeader_1x05_P2.54mm_Horizontal, symbol kicad_inventree_lib:PinHeader_01x05_P2.54_THT_angle
- added J6: ~, kicad_inventree_lib:PM-front-02x10, symbol kicad_inventree_lib:PM-front-02x10
- added R36, R37, R38, R39, R40: 10k, Resistor_SMD:R_1206_3216Metric_Pad1.30x1.75mm_HandSolder, symbol kicad_inventree_lib:R_10k_1206_1%
- added R41: 100, Resistor_SMD:R_1206_3216Metric_Pad1.30x1.75mm_HandSolder, symbol kicad_inventree_lib:R_100_1206_1%
- added SW1: DSIC05LS-P, kicad_inventree_lib:DSIC05LS-P, symbol kicad_inventree_lib:DSIC05LS-P
Connections:
- net +3.3V: now also SW1.10, SW1.6, SW1.7, SW1.8, SW1.9
- net +5V: now also J3.1 (Pin_1)
- net GND: now also J3.3 (Pin_3)
- net MISO: now also R41.2; no longer U1.9 (SI)
- net OUT01: now also J6.2
- net OUT02: now also J6.4
- net OUT03: now also J6.6
- net OUT04: now also J6.8
- net OUT05: now also J6.10
- net OUT06: now also J6.12
- net OUT07: now also J6.14
- net OUT08: now also J6.16
- net OUT09: now also J6.1
- net OUT10: now also J6.3
- net OUT11: now also J6.5
- net OUT12: now also J6.7
- net OUT13: now also J6.9
- net OUT14: now also J6.11
- net OUT15: now also J6.13
- net OUT16: now also J6.15
- net SCL: now also J3.5 (Pin_5)
- net SDA: now also J3.4 (Pin_4)
- net A5: now reaches J5.5 (Pin_5)
- net A5: now also R40.2, SW1.1
- net A4: now reaches J5.6 (Pin_6)
- net A4: now also R39.2, SW1.2
- net A3: now reaches J5.7 (Pin_7)
- net A3: now also R38.2, SW1.3
- net A2: now reaches J4.8 (Pin_8)
- net A2: now also R37.2, SW1.4
- net RST renamed A1
- net A1: now also R36.2, SW1.5
- new net: R41.1, U1.9 (SI)
- new net DGND: R36.1, R37.1, R38.1, R39.1, R40.1
- no-connect marks 12 -> 13
Other:
- note added: "Задание адреса"

Commit message: PM-DI16-DC24sink
Parts:
- removed H4: MountingHole, MountingHole:MountingHole_3.2mm_M3, symbol Mechanical:MountingHole
- removed J6: ~, kicad_inventree_lib:PM-front-02x10, symbol kicad_inventree_lib:PM-front-02x10
- removed R33, R34, R35, R41: 100, Resistor_SMD:R_1206_3216Metric_Pad1.30x1.75mm_HandSolder, symbol kicad_inventree_lib:R_100_1206_1%
- removed R39, R40: 10k, Resistor_SMD:R_1206_3216Metric_Pad1.30x1.75mm_HandSolder, symbol kicad_inventree_lib:R_10k_1206_1%
- removed SW1: DSIC05LS-P, kicad_inventree_lib:DSIC05LS-P, symbol kicad_inventree_lib:DSIC05LS-P
- added C33: 4.7nF 2kV, Capacitor_SMD:C_1812_4532Metric_Pad1.57x3.40mm_HandSolder, symbol kicad_inventree_lib:C_4.7nF_2kV_1812
- added D2: ~, kicad_inventree_lib:PE, symbol kicad_inventree_lib:PE
- added J1: ~, kicad_inventree_lib:PM-front-02x08, symbol kicad_inventree_lib:PM-front-02x08
- added SW1: DSIC03LS-P, kicad_inventree_lib:DSIC03LS-P, symbol kicad_inventree_lib:DSIC03LS-P
Connections:
- net A4 is gone; now on net A2: J5.6 (Pin_6)
- net A5 is gone; now on net A3: J5.5 (Pin_5)
- net +3.3V: now also SW1.4, SW1.5, SW1.6
- net +5V: now also J1.1
- net A1: now also J5.7 (Pin_7), SW1.3; no longer J4.7 (Pin_7)
- net A2: now also SW1.2; no longer J4.8 (Pin_8)
- net A3: now also SW1.1; no longer J5.7 (Pin_7)
- net CLK: now also J4.5 (Pin_5), J1.6
- net FGND: now also C33.2
- net GND: now also J1.15
- net MISO: now also U1.9 (SI), J1.4
- net MOSI: now also J4.3 (Pin_3), J1.2
- net PE: now also C33.1, D2.1
- net CS1: now reaches J4.6 (Pin_6)
- net INT: now reaches U1.16 (INTA)
- net INT: now also J4.7 (Pin_7)
- new net CS2: J1.8, J4.8 (Pin_8)
- no-connect marks 13 -> 18
Other:
- moved on the sheet: R36, R37, R38

Commit message: send to nextpcb
Parts:
- removed J1: ~, kicad_inventree_lib:PM-front-02x08, symbol kicad_inventree_lib:PM-front-02x08
- removed SW1: DSIC03LS-P, kicad_inventree_lib:DSIC03LS-P, symbol kicad_inventree_lib:DSIC03LS-P
- removed U1: MCP23S17_ML, Package_DFN_QFN:QFN-28-1EP_6x6mm_P0.65mm_EP4.25x4.25mm, symbol Interface_Expansion:MCP23S17_ML
- added J6: ~, kicad_inventree_lib:PM-front-02x04, symbol kicad_inventree_lib:PM-front-02x04
- added SW1: DIP_SW-3P-P2.54-THT-Top, Button_Switch_THT:SW_DIP_SPSTx03_Slide_9.78x9.8mm_W7.62mm_P2.54mm, symbol kicad_inventree_lib:DIP_SW-3P-P2.54-THT-Top
- added U11: MCP23S17_ML, Package_DFN_QFN:QFN-28-1EP_6x6mm_P0.65mm_EP4.25x4.25mm, symbol kicad_inventree_lib:MCP23S17_ML
- D2: now left out of the parts list
Connections:
- net +3.3V: now also SW1.4, SW1.5, SW1.6
- net +5V: now also J6.1, U11.14 (~{RESET}), U11.5 (VDD)
- net A1: now also SW1.1
- net A2: now also SW1.2
- net A3: now also SW1.3
- net CLK: now also J6.6, U11.8 (SCK)
- net CS: now also U11.7 (~{CS})
- net CS2: now also J6.8
- net GND: now also J6.7, U11.11 (A0), U11.12 (A1), U11.13 (A2), U11.29 (EP), U11.6 (VSS)
- net INT: now also U11.16 (INTA)
- net MISO: now also J6.4, U11.9 (SI)
- net MOSI: now also J6.2, U11.10 (SO)
- net OUT01: now also U11.17 (GPA0)
- net OUT02: now also U11.18 (GPA1)
- net OUT03: now also U11.19 (GPA2)
- net OUT04: now also U11.20 (GPA3)
- net OUT05: now also U11.21 (GPA4)
- net OUT06: now also U11.22 (GPA5)
- net OUT07: now also U11.23 (GPA6)
- net OUT08: now also U11.24 (GPA7)
- net OUT09: now also U11.25 (GPB0)
- net OUT10: now also U11.26 (GPB1)
- net OUT11: now also U11.27 (GPB2)
- net OUT12: now also U11.28 (GPB3)
- net OUT13: now also U11.1 (GPB4)
- net OUT14: now also U11.2 (GPB5)
- net OUT15: now also U11.3 (GPB6)
- net OUT16: now also U11.4 (GPB7)
- no-connect marks 18 -> 10
Other:
- note added: "Фронтальная плата"

Commit message: PM-DI16
Parts:
- removed D1: B5819W, Diode_SMD:D_SOD-123, symbol kicad_inventree_lib:B5819W
- removed D2: ~, kicad_inventree_lib:PE, symbol kicad_inventree_lib:PE
- removed J3: PinHeader_01x05_P2.54_THT_angle, Connector_PinHeader_2.54mm:PinHeader_1x05_P2.54mm_Horizontal, symbol kicad_inventree_lib:PinHeader_01x05_P2.54_THT_angle
- removed J4, J5: PinHeader P2.54 01x12 THT Straight, Connector_PinHeader_2.54mm:PinHeader_1x12_P2.54mm_Vertical, symbol kicad_inventree_lib:PinHeader_01x12_P2.54_THT_straight
- removed R36, R37, R38: 10k, Resistor_SMD:R_1206_3216Metric_Pad1.30x1.75mm_HandSolder, symbol kicad_inventree_lib:R_10k_1206_1%
- removed SW1: DIP_SW-3P-P2.54-THT-Top, Button_Switch_THT:SW_DIP_SPSTx03_Slide_9.78x9.8mm_W7.62mm_P2.54mm, symbol kicad_inventree_lib:DIP_SW-3P-P2.54-THT-Top
- removed U10: Weact ESP32-C3FH4, kicad_inventree_lib:Weact ESP32-C3FH4, symbol kicad_inventree_lib:Weact ESP32-C3FH4
- added J1: PinHeader_01x05_P2.54_THT_angle, Connector_PinHeader_2.54mm:PinHeader_1x05_P2.54mm_Horizontal, symbol kicad_inventree_lib:PinHeader_01x05_P2.54_THT_angle
- added PE1: PE, kicad_inventree_lib:PE, symbol kicad_inventree_lib:PE
- added PM1: ~, kicad_inventree_lib:PM-ESP32C3, symbol kicad_inventree_lib:PM-ESP32C3
Connections:
- net CS is gone; now on net CS1: U11.7 (~{CS})
- net +3.3V: now also J6.1, J6.2, U11.5 (VDD), J1.4 (Pin_4), PM1.10 (+3.3V)
- net +5V: now also J1.3 (Pin_3); no longer J6.1, U11.5 (VDD)
- net CS1: now also PM1.5 (GPIO8)
- net CS2: now also J6.6, PM1.6 (GPIO7); no longer J6.8
- net GND: now also J6.8, J1.5 (Pin_5), PM1.11 (GND), PM1.14 (GND)
- net INT: now also PM1.7 (GPIO6)
- net MISO: now also J6.5, U11.10 (SO), PM1.3 (GPIO3); no longer J6.4, U11.9 (SI)
- net MOSI: now also J6.3, U11.9 (SI), PM1.2 (GPIO2); no longer J6.2, U11.10 (SO)
- net PE: now also PE1.1
- net SCL: now also J1.2 (Pin_2), PM1.13 (SCL)
- net SDA: now also J1.1 (Pin_1), PM1.12 (SDA)
- net CLK renamed SCK
- net SCK: now also J6.4, PM1.4 (GPIO9); no longer J6.6
- no-connect marks 10 -> 4
Other:
- note removed: "ESP32"
- note removed: "Задание адреса"
- moved on the sheet: U11

Commit message: PM-RQ8
Other:
- added sheet external_connection (external_connection.kicad_sch)
Changed lines of the file:
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@@
+		)
+	)
+	(sheet
+		(at 25.4 254)
+		(size 25.4 25.4)
+		(fields_autoplaced yes)
+		(stroke
+			(width 0.1524)
+			(type solid)
+		)
+		(fill
+			(color 0 0 0 0.0000)
+		)
+		(property "Sheetname" "external_connection"
+			(at 25.4 253.2884 0)
+			(effects
+				(font
+					(size 1.27 1.27)
+				)
+				(justify left bottom)
+			)
+		)
+		(property "Sheetfile" "external_connection.kicad_sch"
+			(at 25.4 279.9846 0)
+			(effects
+				(font
+					(size 1.27 1.27)
+				)
+				(justify left top)
+			)
+		)
+		(instances
+			(project "PM-DI16-DC24sink"
+				(path "/1246bd54-589f-4393-89ee-2c32c8dfdfba"
+					(page "3")
+				)
+			)
 		)
 	)

Commit message: send to nextpcb
Parts:
- PM1: part_ipn (none) -> PM-ESP32C3
Connections:
- net +3.3V: now also U11.14 (~{RESET})
- net +5V: no longer U11.14 (~{RESET})
Other:
- sheet isolation ports: added FGND, GND, Vcc1; removed none
