File: PM-AI1-W_v0.0.1/PM-AI1-W.kicad_sch (KiCad schematic)
At the start: 44 parts, among them J1 2EDGK-5.08-08P, J4 2EDGR-5.08-08P, Q1 BSH112, Q2 BSH201, Q4 BSH112, Q7 BSH201, U1 AD7195BCPZ, U3 CA-IS3641HW, U4 CJA1117B-3.3

Commit message: PM-Debug
Other:
- moved on the sheet: H1, H2, H3, H4

Commit message: update
Other:
- title: (none) -> ${article} v${version}
Changed lines of the file:
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@@
 	(generator_version "8.0")
 	(paper "A3")
+	(title_block
+		(title "${article} v${version}")
+	)
 	(junction
 		(at 63.5 43.18)

Commit message: send to nextpcb
Parts:
- removed C1, C11, C13, C19, C20, C21, C22: 0.1uF, Capacitor_SMD:C_1206_3216Metric_Pad1.33x1.80mm_HandSolder, symbol kicad_inventree_lib:C_100nF_1206
- removed C12, C14: 1uF, Capacitor_SMD:C_1206_3216Metric_Pad1.33x1.80mm_HandSolder, symbol kicad_inventree_lib:C_1uF_1206
- added C1, C11, C13, C16, C19, C20, C21: 100nF, Capacitor_SMD:C_1206_3216Metric_Pad1.33x1.80mm_HandSolder, symbol kicad_inventree_lib:C_100nF_50V_1206
- added C12, C14: 1uF, Capacitor_SMD:C_1206_3216Metric_Pad1.33x1.80mm_HandSolder, symbol kicad_inventree_lib:C_1uF_16V_1206
Connections:
- net +5V_ISO: now also C20.1
- net AD_AIN1: now also C14.1
- net AD_REFIN(+): now also C11.1, C12.1
- net AD_REFIN(-): now also C12.2, C13.1
- net AGND: now also C1.1, C11.2, C13.2, C14.2, C16.2, C19.2, C20.2, C21.2
- net AVDD: now also C1.2, C16.1, C21.1
- net DVDD: now also C19.1
