File: PM-Debug_v0.0.1/PM-Debug_v0.0.1.kicad_sch (KiCad schematic)
At the start: 8 parts, among them J1 AFA07-S10FCC-00, J2 Conn_01x10_Pin, J4 PinHeader_01x08_P2.54_THT_Str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, J5 Conn_01x03_Pin, U1 CJA1117B-3.3

Commit message: send to nextpcb
Parts:
- removed J3: ~, kicad_inventree_lib:HC-WK88-H16-1X2-DB, symbol kicad_inventree_lib:HC-WK88-H16-1X2-DB
- removed J4: PinHeader_01x08_P2.54_THT_Straight, Connector_PinHeader_2.54mm:PinHeader_1x08_P2.54mm_Vertical, symbol kicad_inventree_lib:PinHeader_01x08_P2.54_THT_Straight
- added J3: AFA07-S10FCC-00, kicad_inventree_lib:CONN10_AFA07-S10_JUS, symbol kicad_inventree_lib:AFA07-S10FCC-00
- added J4: Conn_01x10_Pin, Connector_PinHeader_2.54mm:PinHeader_1x10_P2.54mm_Vertical, symbol Connector:Conn_01x10_Pin
- J1: part_ipn (none) -> AFA07-S10FCC-00
Connections:
- new net: J3.1 (Pin_1), J4.1 (Pin_1)
- new net: J3.10 (Pin_10), J4.10 (Pin_10)
- new net: J3.2 (Pin_2), J4.2 (Pin_2)
- new net: J3.3 (Pin_3), J4.3 (Pin_3)
- new net: J3.4 (Pin_4), J4.4 (Pin_4)
- new net: J3.5 (Pin_5), J4.5 (Pin_5)
- new net: J3.6 (Pin_6), J4.6 (Pin_6)
- new net: J3.7 (Pin_7), J4.7 (Pin_7)
- new net: J3.8 (Pin_8), J4.8 (Pin_8)
- new net: J3.9 (Pin_9), J4.9 (Pin_9)
Other:
- moved on the sheet: C1, C2, J5, U1
