File: PM-LED8_v0.0.1/PM-LED8.kicad_sch (KiCad schematic)
At the start: 24 parts, among them J1 AFA07-S10FCC-00, J2 AFA07-S10FCC-00, J3 AFA07-S10FCC-00, J4 AFA07-S10FCC-00

Commit message: send to nextpcb
Parts:
- J1, J2, J3, J4: part_ipn (none) -> AFA07-S10FCC-00
Changed lines of the file:
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@@
+			)
+		)
+		(property "part_ipn" "AFA07-S10FCC-00"
+			(at 152.4 86.36 0)
+			(effects
+				(font
+					(size 1.27 1.27)
+				)
+				(hide yes)
 			)
 		)
@@
 			)
 		)
+		(property "part_ipn" "AFA07-S10FCC-00"
+			(at 152.4 58.42 0)
+			(effects
+				(font
+					(size 1.27 1.27)
+				)
+				(hide yes)
+			)
+		)
 		(pin "9"
 		)
@@
 			)
 		)
+		(property "part_ipn" "AFA07-S10FCC-00"
+			(at 152.4 114.3 0)
+			(effects
+				(font
+					(size 1.27 1.27)
+				)
+				(hide yes)
+			)
+		)
 		(pin "9"
 		)
@@
 			(at 152.4 30.48 0)
 			(effects
+				(font
+					(size 1.27 1.27)
+				)
+				(hide yes)
+			)
+		)
+		(property "part_ipn" "AFA07-S10FCC-00"
+			(at 152.4 30.48 0)
+			(effects
