File: PM-CPU-RP_v0.0.3/PM-CPU-RP.kicad_sch (KiCad schematic)
At the start: 13 parts, among them J1 PinHeader_01x05_P2.54_THT_ang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, J3 FemaleHeader_02x20_P2.54_SMD_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, J7 2EDGK-5.08-02P, J8 2EDGR-5.08-02P

Commit message: PM-CPU-RP
Parts:
- removed J1: PinHeader_01x05_P2.54_THT_angle, Connector_PinHeader_2.54mm:PinHeader_1x05_P2.54mm_Horizontal, symbol kicad_inventree_lib:PinHeader_01x05_P2.54_THT_angle
- removed J2: ~, kicad_inventree_lib:PM-front-02x04, symbol kicad_inventree_lib:PM-front-02x04
- removed R1, R2: 3k3, Resistor_SMD:R_1206_3216Metric_Pad1.30x1.75mm_HandSolder, symbol kicad_inventree_lib:R_3k3_1206_1%
- added C2, C3: 22uF, kicad_inventree_lib:C_2220_5750Metric_Pad1.97x5.40mm_HandSolder, symbol kicad_inventree_lib:C_22uF_50V_2220
- added H4, H5, H6, H7: MountingHole, MountingHole:MountingHole_2.2mm_M2, symbol Mechanical:MountingHole
- added J1, J2: R-RJ11R04P-A802, kicad_inventree_lib:R-RJ11R04P-A802, symbol kicad_inventree_lib:R-RJ11R04P-A802
- added J4: K7805-2000R3, kicad_inventree_lib:K7805-2000R3, symbol kicad_inventree_lib:K7805-2000R3
- added J5: 2EDGK-5.08-02P, symbol kicad_inventree_lib:Degson_2EDGK-5.08-02P
- added J6: 2EDGR-5.08-02P, NextPCB:Degson_2EDGR-5.08-02P, symbol kicad_inventree_lib:Degson_2EDGR-5.08-02P
- added U1: 64900001039, NextPCB:Fuseholder, symbol kicad_inventree_lib:Fuseholder
Connections:
- net +3.3V: now also D1.1 (3V3)
- net +5V: now also C3.1, J4.3 (+VO)
- net GND: now also C2.2, C3.2, J1.4 (Pin_4), J2.4 (Pin_4), J4.2 (GND), J6.2 (Pin_2)
- net SCL: now also J1.2 (Pin_2), J2.2 (Pin_2)
- net SDA: now also J1.3 (Pin_3), J2.3 (Pin_3)
- new net: C2.1, J4.1 (VIN), U1.2
- new net +24V: J6.1 (Pin_1), U1.1
- no-connect marks 78 -> 71
Other:
- note added: "Крепление платы светодиодов"
- note added: "Регулятор напряжения DC24 / DC5"
- note removed: "Подключение внутренней шины"
- moved on the sheet: J3, J7, J8

Commit message: update
Parts:
- removed H4, H5, H6, H7: MountingHole, MountingHole:MountingHole_2.2mm_M2, symbol Mechanical:MountingHole
- removed J7: 2EDGK-5.08-02P, symbol kicad_inventree_lib:Degson_2EDGK-5.08-02P
- removed J8: 2EDGR-5.08-02P, NextPCB:Degson_2EDGR-5.08-02P, symbol kicad_inventree_lib:Degson_2EDGR-5.08-02P
Connections:
- no-connect marks 71 -> 69
Other:
- added sheet subplates (subplates.kicad_sch)
- note removed: "Крепление платы светодиодов"

Commit message: update
Parts:
- added J7: Conn_02x05_Odd_Even, Connector_PinHeader_2.54mm:PinHeader_2x05_P2.54mm_Horizontal, symbol Connector_Generic:Conn_02x05_Odd_Even
- added R1, R10, R12, R4, R6, R8: 330R, Resistor_SMD:R_1206_3216Metric_Pad1.30x1.75mm_HandSolder, symbol kicad_inventree_lib:R_330R_1206_1%
- added R11, R3, R5, R7, R9: 10k, Resistor_SMD:R_1206_3216Metric_Pad1.30x1.75mm_HandSolder, symbol kicad_inventree_lib:R_10k_1206_1%
- added R2: 4k7, Resistor_SMD:R_1206_3216Metric_Pad1.30x1.75mm_HandSolder, symbol kicad_inventree_lib:R_4k7_1206_1%
Connections:
- net +24V: now also R2.1
- net +5V: now also R1.1
- net GND: now also R11.1, R3.1, R5.1, R7.1, R9.1
- net LED_2: now reaches D1.10 (GPIO15/UART_RX)
- net LED_3: now reaches D1.11 (GPIO17)
- net KEY_IN_0: now reaches D1.26 (GPIO7/SPI_CE1)
- net KEY_IN_0: now also R3.2, R4.1
- net KEY_OUT_0: now reaches D1.29 (GPIO5)
- net KEY_OUT_0: now also J7.2 (Pin_2)
- net KEY_OUT_1: now reaches D1.31 (GPIO6)
- net KEY_OUT_1: now also J7.4 (Pin_4)
- net KEY_IN_1: now reaches D1.32 (GPIO12/PWM0)
- net KEY_IN_1: now also R5.2, R6.1
- net KEY_OUT_2: now reaches D1.33 (GPIO13/PWM1)
- net KEY_OUT_2: now also J7.6 (Pin_6)
- net KEY_OUT_3: now reaches D1.35 (GPIO19/PCM_FS)
- net KEY_OUT_3: now also J7.8 (Pin_8)
- net KEY_IN_2: now reaches D1.36 (GPIO16)
- net KEY_IN_2: now also R7.2, R8.1
- net KEY_OUT_4: now reaches D1.37 (GPIO26)
- net KEY_OUT_4: now also J7.10 (Pin_10)
- net KEY_IN_3: now reaches D1.38 (GPIO20/PCM_DIN)
- net KEY_IN_3: now also R10.1, R9.2
- net KEY_IN_4: now reaches D1.40 (GPIO20/PCM_DOUT)
- net KEY_IN_4: now also R11.2, R12.1
- net LED_0: now reaches D1.7 (GPIO4/GPCLK0)
- net LED_1: now reaches D1.8 (GPIO14/UART_TX)
- net at J2.1 (Pin_1): now also J1.1 (Pin_1)
- new net: J7.1 (Pin_1), R4.2
- new net: J7.3 (Pin_3), R6.2
- new net: J7.5 (Pin_5), R8.2
- new net: J7.7 (Pin_7), R10.2
- new net: J7.9 (Pin_9), R12.2
- new net subplates/LED_24V: R2.2
- new net subplates/LED_5V: R1.2
- no-connect marks 69 -> 55
Other:
- sheet subplates ports: added GND, LED_0, LED_1, LED_2, LED_24V, LED_3, LED_5V; removed none
- moved on the sheet: D1, J3

Commit message: PM-CPU-RP
Parts:
- removed J1, J2: R-RJ11R04P-A802, kicad_inventree_lib:R-RJ11R04P-A802, symbol kicad_inventree_lib:R-RJ11R04P-A802
- removed J7: Conn_02x05_Odd_Even, Connector_PinHeader_2.54mm:PinHeader_2x05_P2.54mm_Horizontal, symbol Connector_Generic:Conn_02x05_Odd_Even
- removed R10, R12, R4, R6, R8: 330R, Resistor_SMD:R_1206_3216Metric_Pad1.30x1.75mm_HandSolder, symbol kicad_inventree_lib:R_330R_1206_1%
- removed R11, R3, R5, R7, R9: 10k, Resistor_SMD:R_1206_3216Metric_Pad1.30x1.75mm_HandSolder, symbol kicad_inventree_lib:R_10k_1206_1%
- added XG1: DG141R-2.54-10P, kicad_inventree_lib:DG141R-2.54-10P, symbol kicad_inventree_lib:DG141R-2.54-10P

Commit message: update PM-RP
Parts:
- added C4, C6, C8: 10uF, Capacitor_SMD:C_1206_3216Metric_Pad1.33x1.80mm_HandSolder, symbol kicad_inventree_lib:C_10uF_16V_1206
- added C5, C7: 100nF, Capacitor_SMD:C_1206_3216Metric_Pad1.33x1.80mm_HandSolder, symbol kicad_inventree_lib:C_100nF_50V_1206
- added CR1: SM712, SOT23-3_LTF, symbol kicad_inventree_lib:SM712
- added J1: ~, kicad_inventree_lib:BS-12-A1AJ002-F, symbol kicad_inventree_lib:BS-12-A1AJ002-F
- added JP1, JP2, JP3, JP4, JP5: SolderJumper_2_Open, Jumper:SolderJumper-2_P1.3mm_Open_RoundedPad1.0x1.5mm, symbol Jumper:SolderJumper_2_Open
- added R3, R4, R5, R6: 10k, Resistor_SMD:R_1206_3216Metric_Pad1.30x1.75mm_HandSolder, symbol kicad_inventree_lib:R_10k_1206_1%
- added U3: W25Q32JVSSIQ, kicad_inventree_lib:SOIC-8_5P28X5P28_WIN-M, symbol kicad_inventree_lib:W25Q32JVSSIQ
- added U4: CA-IS3641HW, kicad_inventree_lib:SOIC16-WBW_CLG-M, symbol kicad_inventree_lib:CA-IS3641HW
- added U5: MAX3485, Package_SO:SOIC-8_3.9x4.9mm_P1.27mm, symbol Interface_UART:MAX3485
- added U6: DS3231, Package_SO:SOIC-16W_7.5x10.3mm_P1.27mm, symbol kicad_inventree_lib:DS3231
- added U7: SN74LVC2G14DBVR, kicad_inventree_lib:DBV6-M, symbol kicad_inventree_lib:SN74LVC2G14DBVR
Connections:
- net +3.3V: now also D1.17 (3V3), C4.1, C5.1, C6.1, JP1.1 (A), R3.1, R4.1, R5.1, U3.8 (VCC), U4.1 (VDD), U6.2 (VCC), U6.4 (~{RST}), U7.5 (VCC)
- net GND: now also C4.2, C5.2, C6.2, J1.2, JP5.1 (A), U3.4 (GND), U4.2 (GNDA), U4.8 (GNDA), U6.10 (GND), U6.11 (GND), U6.12 (GND), U6.13 (GND), U6.5 (GND), U6.6 (GND), U6.7 (GND), U6.8 (GND), U6.9 (GND), U7.2 (GND)
- net LED_0: now also D1.15 (GPIO22); no longer D1.7 (GPIO4/GPCLK0)
- net LED_1: now also D1.16 (GPIO23); no longer D1.8 (GPIO14/UART_TX)
- net LED_2: now also D1.18 (GPIO24); no longer D1.10 (GPIO15/UART_RX)
- net PE: now also XG1.10 (Pin_10), XG1.5 (Pin_5)
- net SCL: now also U6.16 (SCL)
- net SDA: now also U6.15 (SDA)
- net SPI_MOSI: now reaches D1.19 (GPIO10/SPI_MOSI)
- net SPI_MOSI: now also U3.5 (DI(IO0))
- net SPI_MISO: now reaches D1.21 (GPIO9/SPI_MISO)
- net SPI_MISO: now also U3.2 (DO(IO1))
- net SPI_SCK: now reaches D1.23 (GPIO11/SPI_SCLK)
- net SPI_SCK: now also U3.6 (CLK)
- net SPI_CS0: now reaches D1.24 (GPIO8/SPI_CE0)
- net SPI_CS0: now also R5.2, U3.1 (/CS)
- net RS485_A: now reaches XG1.3 (Pin_3)
- net RS485_A: now also XG1.8 (Pin_8), CR1.1, U5.6 (A)
- net RS485_B: now reaches XG1.4 (Pin_4)
- net RS485_B: now also XG1.9 (Pin_9), CR1.2, U5.7 (B)
- net KEY_IN_0: no longer names the net of D1.26 (GPIO7/SPI_CE1)
- net KEY_IN_1: no longer names the net of D1.32 (GPIO12/PWM0)
- net KEY_IN_2: no longer names the net of D1.36 (GPIO16)
- net KEY_IN_3: no longer names the net of D1.38 (GPIO20/PCM_DIN)
- net KEY_IN_4: no longer names the net of D1.40 (GPIO20/PCM_DOUT)
- net KEY_OUT_0: no longer names the net of D1.29 (GPIO5)
- net KEY_OUT_1: no longer names the net of D1.31 (GPIO6)
- net KEY_OUT_2: no longer names the net of D1.33 (GPIO13/PWM1)
- net KEY_OUT_3: no longer names the net of D1.35 (GPIO19/PCM_FS)
- net KEY_OUT_4: no longer names the net of D1.37 (GPIO26)
- net LED_3: no longer names the net of D1.11 (GPIO17)
- new net: J1.1, U6.14 (VBAT)
- new net: R4.2, U3.3 (/WP(IO2))
- new net: R3.2, U3.7 (/HOLD_(IO3))
- new net +3.3V_ISO: C7.1, C8.1, JP1.2 (B), U4.16 (VISO), U5.8 (VCC)
- new net GND_ISO: C7.2, C8.2, CR1.3, JP5.2 (B), R6.2, U4.10 (SEL), U4.15 (GNDB), U4.9 (GNDB), U5.5 (GND)
- new net UART_RTS: JP3.1 (A), U4.4 (VI2)
- new net UART_RTS_ISO: JP3.2 (B), R6.1, U4.13 (VO2), U5.2 (~{RE}), U5.3 (DE)
- new net UART_RX: D1.10 (GPIO15/UART_RX), JP4.1 (A), U4.6 (VO4), U7.1 (1A)
- new net UART_RX_ISO: JP4.2 (B), U4.11 (VI4), U5.1 (RO)
- new net UART_TX: D1.8 (GPIO14/UART_TX), JP2.1 (A), U4.3 (VI1), U7.3 (2A)
- new net UART_TX_ISO: JP2.2 (B), U4.14 (VO1), U5.4 (DI)
- new net subplates/LED_RX: U7.6 (1Y)
- new net subplates/LED_TX: U7.4 (2Y)
- no-connect marks 55 -> 68
Other:
- sheet subplates ports: added LED_3V3, LED_RX, LED_TX; removed LED_3
- note added: "RS-485"
- note added: "Внешняя Flash память"
- note added: "Изоляция UART"
- note added: "Часы реального времени"
- moved on the sheet: H1, H2, H3, R1, R2, XG1
