File: archive/PM-ESPC3_v0.0.2/PM-ESPC3.kicad_pcb (KiCad board)
At the start: 2 copper layers, 39.8 x 95.8 mm, 48 parts, among them J1 U254-051T-4BH83-S1S, J2 AFA07-S10FCC-00, J5 AFA07-S10FCC-00, J8 AFA07-S10FCC-00, SW1 Button, SW2 Button, SW4 DIP 3 pos, U1 ESP32-C3-WROOM-02U-N4, U2 CJA1117B-3.3, U3 MAX3485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

Commit message: new version
Parts:
- removed ? (x4): , clipboard:b0caab98-8a23-470e-b26d-76b441dffb16
