File: current/PM-AI4-W_v0.0.2/PM-AI4-W.kicad_sch (KiCad schematic)
At the start: 65 parts, among them J1 AFA07-S10FCC-00, U1 AD7190BRUZ, U2 AD7190BRUZ, U3 CA-IS3761HW, U4 CA-IS3105W

Commit message: update
Parts:
- removed XG1, XG2, XG3, XG4: DG141R-2.54-07P, kicad_inventree_lib:DG141R-2.54-07P, symbol kicad_inventree_lib:DG141R-2.54-07P
- added J4, J5: 15EDGRHC-THR-3.5-14P, kicad_inventree_lib:15EDGRHC-THR-3.5-14P, symbol kicad_inventree_lib:15EDGRHC-THR-3.5-14P
- added JP1, JP2, JP3, JP4, JP5, JP6, JP7, JP8: SolderJumper_2_Open, Jumper:SolderJumper-2_P1.3mm_Open_RoundedPad1.0x1.5mm, symbol Jumper:SolderJumper_2_Open
Connections:
- net 0.EXC-: now also J4.13 (Pin_10), J4.6 (Pin_9)
- net 0.SENSE+: now also J4.5 (Pin_9)
- net 0.SENSE-: now also J4.4
- net 0.SIG+: now also J4.3
- net 0.SIG-: now also J4.2 (Pin_3)
- net 1.SENSE+: now also J4.12 (Pin_10)
- net 1.SENSE-: now also J4.11 (Pin_8)
- net 1.SIG+: now also J4.10 (Pin_6)
- net 1.SIG-: now also J4.9 (Pin_4)
- net 2.EXC-: now also J5.13 (Pin_10), J5.6 (Pin_9)
- net 2.SENSE+: now also J5.5 (Pin_9)
- net 2.SENSE-: now also J5.4
- net 2.SIG+: now also J5.3
- net 2.SIG-: now also J5.2 (Pin_3)
- net 3.SENSE+: now also J5.12 (Pin_10)
- net 3.SENSE-: now also J5.11 (Pin_8)
- net 3.SIG+: now also J5.10 (Pin_6)
- net 3.SIG-: now also J5.9 (Pin_4)
- net AGND: now also J4.1 (Pin_1), J4.8 (Pin_2), J5.1 (Pin_1), J5.8 (Pin_2)
- net AVDD: now also J4.14 (Pin_10), J4.7 (Pin_9), J5.14 (Pin_10), J5.7 (Pin_9)
- net CS0: now also JP1.1 (A), JP5.1 (A); no longer R11.2, U3.4 (VI3)
- net CS1: now also JP2.1 (A), JP6.1 (A); no longer R10.2, U3.5 (VI4)
- new net: JP1.2 (B), JP2.2 (B), JP3.2 (B), JP4.2 (B), R10.2, U3.4 (VI3)
- new net: JP5.2 (B), JP6.2 (B), JP7.2 (B), JP8.2 (B), R11.2, U3.5 (VI4)
- new net CS2: JP3.1 (A), JP7.1 (A)
- new net CS3: JP4.1 (A), JP8.1 (A)
- no-connect marks 35 -> 15
Other:
- sheet subplates ports: added CS2, CS3; removed none
- note added: "Изменить 10uF тип на X7R - увеличить посадочное место"
- moved on the sheet: C1, C10, C13, C14, C15, C16, C17, C18, C19, C2, C20, C21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
