File: current/PM-CPU-RP_v0.0.4/PM-CPU-RP.kicad_pcb (KiCad board)
At the start: 2 copper layers, 80 x 100 mm, 34 parts, among them J10 AFA07-S10FCC-00, J11 Conn_01x10_Pin, J12 15EDGRC-3.5-05P, J2 15EDGRC-3.5-10P, J3 15EDGRHC-THR-3.5-10P, J4 K7805-2000R3, J5 Conn_01x03_Pin, J9 AFA07-S10FCC-00, U1 64900001039, U2 PM-LED8_v0.0.2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

Commit message: update
Parts:
- J2: value 15EDGRC-3.5-10P -> 15EDGRC-3.5-05P; footprint kicad_inventree_lib:15EDGRC-3.5-10P -> kicad_inventree_lib:15EDGRC-3.5-05P
- moved J2 17.5 mm to (106.7, 82.6)
- moved kicad_logo 4.53 mm to (72.4, 144.8)
- moved oshw_logo 4.53 mm to (83.4, 144.8)
- moved RN1 2.54 mm to (54.6, 72.4)
- moved J1 0.90 mm to (66.5, 60.3)
Connections:
- J2 pad 2: GND -> /SCL
- J2 pad 3: GND -> /SDA
- J2 pad 4: GND -> +3.3V
- J2 pad 5: GND -> +5V
Routing:
- net GND: track 0.00 -> 18.2 mm, vias 0 -> 1
- net +3.3V: track 211.7 -> 208.4 mm
- net /SPI0_CS0: track 31.4 -> 28.3 mm
- net /SPI1_CS2: track 66.6 -> 64.8 mm
- net /Vbat: track 15.0 -> 13.4 mm
