File: current/PM_CPU-RP-v0.0.4/PM_CPU-RP.kicad_pcb (KiCad board)
At the start: 2 copper layers, 80 x 100 mm, 34 parts, among them J11 Conn_01x10_Pin, J12 15EDGRC-3.5-05P, J2 15EDGRC-3.5-05P, J3 15EDGRHC-THR-3.5-10P, J4 K7805-2000R3, J5 Conn_01x03_Pin, J7 AFA07-S10FCC-00, J8 AFA07-S10FCC-00, J9 AFA07-S10FCC-00, U1 64900001039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

Commit message: update
Parts:
- J11: value Conn_01x10_Pin -> PinHeader_01x10_P1.00_THT_straight
- J5: value Conn_01x03_Pin -> PinHeader_01x03_P1.00_THT_straight
Connections:
- net +3.3V renamed +3.3V_CPU
- net +3.3V_ISO renamed +3.3V_BUS
- net GND renamed GND_CPU
- net GND_ISO renamed GND_BUS
