File: current/PM-Keybard_v0.0.2/PM-Keybard.kicad_sch (KiCad schematic)
At the start: 72 parts, among them J1 AFA07-S10FCC-00, J2 FFC_10P_P1.0_100mm_straight, SW0.0 TS-1187A-B-A-B, SW0.1 TS-1187A-B-A-B, SW0.2 TS-1187A-B-A-B, SW0.3 TS-1187A-B-A-B, SW0.4 TS-1187A-B-A-B, SW0.5 TS-1187A-B-A-B, SW0.6 TS-1187A-B-A-B, SW0.7 TS-1187A-B-A-B, SW1.0 TS-1187A-B-A-B, SW1.1 TS-1187A-B-A-B, SW1.2 TS-1187A-B-A-B, SW1.3 TS-1187A-B-A-B, SW1.4 TS-1187A-B-A-B, SW1.5 TS-1187A-B-A-B, SW1.6 TS-1187A-B-A-B, SW1.7 TS-1187A-B-A-B, SW2.0 TS-1187A-B-A-B, SW2.1 TS-1187A-B-A-B, SW2.2 TS-1187A-B-A-B, SW2.3 TS-1187A-B-A-B, SW2.4 TS-1187A-B-A-B, SW2.5 TS-1187A-B-A-B, SW2.6 TS-1187A-B-A-B, SW2.7 TS-1187A-B-A-B, SW3.0 TS-1187A-B-A-B, SW3.1 TS-1187A-B-A-B, SW3.2 TS-1187A-B-A-B, SW3.3 TS-1187A-B-A-B, SW3.4 TS-1187A-B-A-B, SW3.5 TS-1187A-B-A-B, SW3.6 TS-1187A-B-A-B, SW3.7 TS-1187A-B-A-B, SW4.0 TS-1187A-B-A-B, SW4.1 TS-1187A-B-A-B, SW4.2 TS-1187A-B-A-B, SW4.3 TS-1187A-B-A-B, SW4.4 TS-1187A-B-A-B, SW4.5 TS-1187A-B-A-B, SW4.6 TS-1187A-B-A-B, SW4.7 TS-1187A-B-A-B, SW5.0 TS-1187A-B-A-B, SW5.1 TS-1187A-B-A-B, SW5.2 TS-1187A-B-A-B, SW5.3 TS-1187A-B-A-B, SW5.4 TS-1187A-B-A-B, SW5.5 TS-1187A-B-A-B, SW5.6 TS-1187A-B-A-B, SW5.7 TS-1187A-B-A-B, SW6.0 TS-1187A-B-A-B, SW6.1 TS-1187A-B-A-B, SW6.2 TS-1187A-B-A-B, SW6.3 TS-1187A-B-A-B, SW6.4 TS-1187A-B-A-B, SW6.5 TS-1187A-B-A-B, SW6.6 TS-1187A-B-A-B, SW6.7 TS-1187A-B-A-B, SW7.0 TS-1187A-B-A-B, SW7.1 TS-1187A-B-A-B, SW7.2 TS-1187A-B-A-B, SW7.3 TS-1187A-B-A-B, SW7.4 TS-1187A-B-A-B, SW7.5 TS-1187A-B-A-B, SW7.6 TS-1187A-B-A-B, SW7.7 TS-1187A-B-A-B, U1 MCP23S17_SO

Commit message: PM_DBG
Parts:
- removed J1: AFA07-S10FCC-00, kicad_inventree_lib:CONN10_AFA07-S10_JUS, symbol kicad_inventree_lib:AFA07-S10FCC-00
- removed J2: FFC_10P_P1.0_100mm_straight, symbol kicad_inventree_lib:FFC_10P_P1.0_100mm_straight
- removed SW0.7, SW1.7, SW2.7, SW3.7, SW4.7, SW5.7, SW6.7, SW7.0, SW7.1, SW7.2, SW7.3, SW7.4, SW7.5, SW7.6, SW7.7: TS-1187A-B-A-B, TS-1187A-B-A-B_XKB, symbol kicad_inventree_lib:TS-1187A-B-A-B
- removed U1: MCP23S17_SO, Package_SO:SOIC-28W_7.5x17.9mm_P1.27mm, symbol kicad_inventree_lib:MCP23S17_SO
- added J1, J3: AFA07-S12FCC-00, kicad_inventree_lib:CONN10_AFA07-S12_JUS, symbol kicad_inventree_lib:AFA07-S12FCC-00
- added J2: FFC_12P_P1.0_100mm_straight, symbol kicad_inventree_lib:FFC_12P_P1.0_100mm_straight
- added U1: MCP23S17_SS, kicad_inventree_lib:SSOP28_MC_MCH, symbol kicad_inventree_lib:MCP23S17_SS
- U2: footprint kicad_inventree_lib:PM-ESP32C3_v0.0.2 -> kicad_inventree_lib:PM-ESP32C3_v0.0.5; symbol kicad_inventree_lib:PM-ESP32C3_v0.0.2 -> kicad_inventree_lib:PM-ESP32C3_v0.0.5; part_ipn PM-ESP32C3_v0.0.2 -> PM_MCU-ESP32_C3-v0.0.5; now left out of the parts list
Connections:
- net C0: now also U1.1 (GPB0)
- net C1: now also U1.2 (GPB1)
- net C2: now also U1.3 (GPB2)
- net C3: now also U1.4 (GPB3)
- net C4: now also U1.5 (GPB4)
- net C5: now also U1.6 (GPB5)
- net C6: now also U1.7 (GPB6)
- net C7: now also U1.8 (GPB7)
- net CS: now also U1.11 (~{CS})
- net MISO: now also J1.9 (Pin_9), J3.5 (Pin_5), U1.14 (SO)
- net MOSI: now also J1.10 (Pin_10), J3.4 (Pin_4), U1.13 (SI)
- net R0: now also U1.21 (GPA0)
- net R1: now also U1.22 (GPA1)
- net R2: now also U1.23 (GPA2)
- net R3: now also U1.24 (GPA3)
- net R4: now also U1.25 (GPA4)
- net R5: now also U1.26 (GPA5)
- net R6: now also U1.27 (GPA6)
- net R7: now also U1.28 (GPA7)
- net SCK: now also J1.8 (Pin_8), J3.6 (Pin_6), U1.12 (SCK)
- new net +3.3V_MCU: J1.11 (Pin_11), J3.3 (Pin_3), U1.18 (~{RESET}), U1.9 (VDD)
- new net +5V_MCU: J1.12 (Pin_11), J3.2 (Pin_2)
- new net CS0: J1.7 (Pin_7)
- new net CS1: J1.6 (Pin_6)
- new net CS2: J1.5 (Pin_5)
- new net CS3: J1.4 (Pin_4)
- new net CS_DISP: J3.7 (Pin_7)
- new net GND_MCU: J1.1 (Pin_1), J1.13 (Pin_11), J1.2 (Pin_2), J3.1 (Pin_1), J3.12 (Pin_11), J3.13 (Pin_11), U1.10 (VSS), U1.15 (A0), U1.16 (A1), U1.17 (A2)
- new net INT: J1.3 (Pin_3), J3.11 (Pin_11)
- no-connect marks 134 -> 103
Other:
- note added: "Подключение дисплея"
- moved on the sheet: U2
