File: current/PM_CNV-AI8_IU-v0.0.1/PM_CNV-AI8_IU.kicad_sch (KiCad schematic)
At the start: 71 parts, among them J1 AFA07-S10FCC-00, J2 AFA07-S10FCC-00, J3 PinHeader_01x10_P1.00_THT_str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, J4 15EDGRHC-THR-3.5-16P, J5 15EDGRHC-THR-3.5-16P, J6 15EDGRC-3.5-05P, U2 CA-IS3105W, U3 CA-IS3741HW, U4 ADS8688

Commit message: update docs
Parts:
- added U5: AD7190BRUZ, kicad_inventree_lib:RU_24_ADI-M, symbol kicad_inventree_lib:AD7190BRUZ
