File: template/front_v3/front.kicad_sch (KiCad schematic)
At the start: 6 parts

Commit message: update docs
Parts:
- removed H1, H2, H3, H4: MountingHole, MountingHole:MountingHole_2.2mm_M2, symbol Mechanical:MountingHole
- removed H5, H6: MountingHole, MountingHole:MountingHole_3.2mm_M3, symbol Mechanical:MountingHole
- added H5, H6, H7, H8: MountingHole_M2, kicad_inventree_lib:MountingHole_M2, symbol kicad_inventree_lib:MountingHole_M2
