File: current/PM_CNV-RQ8-v0.0.6/PM_CNV-RQ8.kicad_pcb (KiCad board)
At the start: 2 copper layers, 80 x 100 mm, 36 parts, among them J1 PinHeader_01x10_P1.00_THT_str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, J18 AFA07-S10FCC-00, J19 AFA07-S10FCC-00, J2 AFA07-S10FCC-00, J20 PinHeader_01x10_P1.00_THT_str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, J3 AFA07-S10FCC-00, J6 AFA07-S10FCC-00, J7 15EDGRC-3.5-10P, J8 15EDGRC-3.5-10P, K1 G5NB-1A-E-DC5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

Commit message: remove pagebreak level 2
Parts:
- removed J18, J19, J6: AFA07-S10FCC-00, kicad_inventree_lib:CONN10_AFA07-S10_JUS
- removed J20: PinHeader_01x10_P1.00_THT_straight, Connector_PinHeader_1.00mm:PinHeader_1x10_P1.00mm_Vertical
- removed JP5, JP6, JP7: SolderJumper_3_Open, Jumper:SolderJumper-3_P1.3mm_Open_RoundedPad1.0x1.5mm
- added U5: SN74LVC2G14DBVR, kicad_inventree_lib:DBV6-M, F.Cu at (55.9, 60.8)
- J1: value PinHeader_01x10_P1.00_THT_straight -> AFA07-S12FCC-00; footprint Connector_PinHeader_1.00mm:PinHeader_1x10_P1.00mm_Vertical -> kicad_inventree_lib:CONN10_AFA07-S12_JUS
- J2, J3: value AFA07-S10FCC-00 -> AFA07-S12FCC-00; footprint kicad_inventree_lib:CONN10_AFA07-S10_JUS -> kicad_inventree_lib:CONN10_AFA07-S12_JUS
- U3: footprint kicad_inventree_lib:PM-LED_v0.0.2 -> kicad_inventree_lib:PM_LED-xx-v0.0.1
- moved U1 20.4 mm to (54.9, 88.3)
- moved C2 20.3 mm to (53.4, 81.3)
- moved J3 20.0 mm to (64.9, 70.3)
- moved U2 13.4 mm to (53.2, 110.3)
- moved J1 8.32 mm to (44.9, 70.3), turned to 90 degrees
Connections:
- C1 pad 2: GND -> GND_MCU
- C2 pad 1: +3.3V -> +3.3V_MCU
- C2 pad 2: GND -> GND_MCU
- J1 pad 1: +5V -> GND_MCU
- J1 pad 10: GND -> +3.3V_MCU
- J1 pad 2: +3.3V -> /INT
- J1 pad 3: /MOSI -> /CS3
- J1 pad 4: /MISO -> /CS2
- J1 pad 5: /SCK -> /CS1
- J1 pad 7: /CS1 -> /SCK
- J1 pad 8: /CS2 -> /MISO
- J1 pad 9: /CS3 -> /MOSI
- J2 pad 1: +5V -> GND_MCU
- J2 pad 10: GND -> /CS3
- J2 pad 11: GND -> /INT
- J2 pad 2: +3.3V -> +5V_MCU
- J2 pad 3: /MOSI -> +3.3V_MCU
- J2 pad 4: /MISO -> /MOSI
- J2 pad 5: /SCK -> /MISO
- J2 pad 6: /CS0 -> /SCK
- J2 pad 7: /CS1 -> /CS0
- J2 pad 8: /CS2 -> /CS1
- J2 pad 9: /CS3 -> /CS2
- J3 pad 1: GND -> GND_MCU
- J3 pad 10: +5V -> /K2_led
- J3 pad 11: GND -> /K1_led
- J3 pad 2: /CS3 -> /MISO_LED
- J3 pad 3: /CS2 -> /CS_LED
- J3 pad 4: /CS1 -> /K8_led
- J3 pad 5: /CS0 -> /K7_led
- J3 pad 6: /SCK -> /K6_led
- J3 pad 7: /MISO -> /K5_led
- J3 pad 8: /MOSI -> /K4_led
- J3 pad 9: +3.3V -> /K3_led
- K1 pad 1: GND -> GND_MCU
- K2 pad 1: GND -> GND_MCU
- K3 pad 1: GND -> GND_MCU
- K4 pad 1: GND -> GND_MCU
- K5 pad 1: GND -> GND_MCU
- K6 pad 1: GND -> GND_MCU
- K7 pad 1: GND -> GND_MCU
- K8 pad 1: GND -> GND_MCU
- U1 pad 10: GND -> GND_MCU
- U1 pad 15: /A0 -> GND_MCU
- U1 pad 16: /A1 -> GND_MCU
- U1 pad 17: /A2 -> GND_MCU
- U1 pad 18: +3.3V -> +3.3V_MCU
- U1 pad 9: +3.3V -> +3.3V_MCU
- U2 pad 10: GND -> GND_MCU
- U2 pad 9: +5V -> +5V_MCU
Routing:
- net +3.3V: track 92.2 -> 0.00 mm, vias 1 -> 0
- net +5V: track 77.7 -> 0.00 mm
- net +3.3V_MCU: track 0.00 -> 63.7 mm, vias 0 -> 4
- net +5V_MCU: track 0.00 -> 49.9 mm, vias 0 -> 4
- net /MOSI: track 59.6 -> 26.0 mm
- net /SCK: track 58.7 -> 27.4 mm, vias 2 -> 1
- net /MISO_LED: track 0.00 -> 27.3 mm
- net /CS_LED: track 0.00 -> 25.8 mm
- net /K8_led: track 34.1 -> 13.6 mm
- net /K1_led: track 43.0 -> 22.5 mm
- net /K2_led: track 41.7 -> 21.3 mm
- net /K4_led: track 39.2 -> 18.7 mm
- net /K5_led: track 37.9 -> 17.4 mm
- net /K6_led: track 36.7 -> 16.2 mm
- net /K7_led: track 35.4 -> 14.9 mm
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- added copper zone on B.Cu, net +3.3V_MCU
- added copper zone on F.Cu, net +3.3V_MCU
- added copper zone on B.Cu, net +5V_MCU
- added copper zone on F.Cu, net +5V_MCU
- added copper zone on B.Cu, net GND_MCU
- added copper zone on F.Cu, net GND_MCU
- removed copper zone on B.Cu, net GND
- removed copper zone on F.Cu, net GND
