File: current/PM_CNV-RQ8-v0.0.6/PM_CNV-RQ8.kicad_sch (KiCad schematic)
At the start: 46 parts, among them J1 PinHeader_01x10_P1.00_THT_str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, J10 2EDGK-5.08-02P, J11 2EDGK-5.08-02P, J12 2EDGK-5.08-02P, J13 2EDGK-5.08-02P, J14 2EDGK-5.08-02P, J15 2EDGK-5.08-02P, J16 2EDGK-5.08-02P, J17 2EDGK-5.08-02P, J18 AFA07-S10FCC-00, J19 AFA07-S10FCC-00, J2 AFA07-S10FCC-00, J20 PinHeader_01x10_P1.00_THT_str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, J3 AFA07-S10FCC-00, J4 FFC_10P_P1.0_50mm_reverse, J5 FFC_10P_P1.0_100mm_straight, J6 AFA07-S10FCC-00, J7 15EDGRC-3.5-10P, J8 15EDGRC-3.5-10P, J9 2EDGK-5.08-02P, K1 G5NB-1A-E-DC5, K2 G5NB-1A-E-DC5, K3 G5NB-1A-E-DC5, K4 G5NB-1A-E-DC5, K5 G5NB-1A-E-DC5, K6 G5NB-1A-E-DC5, K7 G5NB-1A-E-DC5, K8 G5NB-1A-E-DC5, U1 MCP23S17_SS, U2 TBD62783AFG, U3 PM-LED8_v0.0.2, U5 MCP23017_SS

Commit message: remove pagebreak level 2
Parts:
- removed J1, J20: PinHeader_01x10_P1.00_THT_straight, Connector_PinHeader_1.00mm:PinHeader_1x10_P1.00mm_Vertical, symbol kicad_inventree_lib:PinHeader_01x10_P1.00_THT_straight
- removed J18, J19, J2, J3, J6: AFA07-S10FCC-00, kicad_inventree_lib:CONN10_AFA07-S10_JUS, symbol kicad_inventree_lib:AFA07-S10FCC-00
- removed J5: FFC_10P_P1.0_100mm_straight, symbol kicad_inventree_lib:FFC_10P_P1.0_100mm_straight
- removed JP5, JP6, JP7: SolderJumper_3_Open, Jumper:SolderJumper-3_P1.3mm_Open_RoundedPad1.0x1.5mm, symbol Jumper:SolderJumper_3_Open
- removed U5: MCP23017_SS, kicad_inventree_lib:SSOP28_MC_MCH, symbol kicad_inventree_lib:MCP23017_SS
- added D1, D2, D3, D4, D5, D6, D7, D8: XL-1606SYGC, kicad_inventree_lib:XL-1606, symbol kicad_inventree_lib:XL-1606SYGC
- added J1, J2, J3: AFA07-S12FCC-00, kicad_inventree_lib:CONN10_AFA07-S12_JUS, symbol kicad_inventree_lib:AFA07-S12FCC-00
- added J5: FFC_12P_P1.0_100mm_straight, symbol kicad_inventree_lib:FFC_12P_P1.0_100mm_straight
- added R34, R35, R36, R37, R38, R39, R40, R41: 680R, Resistor_SMD:R_0603_1608Metric, symbol kicad_inventree_lib:R_680R_0603_1%
- added U5: SN74LVC2G14DBVR, kicad_inventree_lib:DBV6-M, symbol kicad_inventree_lib:SN74LVC2G14DBVR
- U3: footprint kicad_inventree_lib:PM-LED_v0.0.2 -> kicad_inventree_lib:PM_LED-xx-v0.0.1; symbol kicad_inventree_lib:PM-LED8_v0.0.2 -> kicad_inventree_lib:PM_LED-10-v0.0.1; part_ipn PM-LED8_v0.0.1 -> PM_LED-10-v0.0.1; now in the parts list
- U4: part_ipn PM-ESP32C3_v0.0.4 -> PM_MCU-ESP32_C3-v0.0.5
Connections:
- net A1 is gone; now on net GND_MCU: U1.16 (A1)
- net A2 is gone; now on net GND_MCU: U1.17 (A2)
- net GND is gone; now on net GND_MCU: C1.2, C2.2, K1.1, K2.1, K3.1, K4.1, K5.1, K6.1, K7.1, K8.1, U1.10 (VSS), U2.10 (GND)
- net CS: now also U5.3 (2A)
- net CS0: now also J1.6 (Pin_6), J2.7 (Pin_7)
- net CS1: now also J1.5 (Pin_5), J2.8 (Pin_8)
- net CS2: now also J1.4 (Pin_4), J2.9 (Pin_9)
- net CS3: now also J1.3 (Pin_3), J2.10 (Pin_10)
- net K1_led: now also J3.11 (Pin_11)
- net K2_led: now also J3.10 (Pin_10)
- net K3_led: now also J3.9 (Pin_9)
- net K4_led: now also J3.8 (Pin_8)
- net K5_led: now also J3.7 (Pin_7)
- net K6_led: now also J3.6 (Pin_6)
- net K7_led: now also J3.5 (Pin_5)
- net K8_led: now also J3.4 (Pin_4)
- net MISO: now also J1.8 (Pin_8), J2.5 (Pin_5), U5.1 (1A)
- net MOSI: now also J1.9 (Pin_9), J2.4 (Pin_4)
- net SCK: now also J1.7 (Pin_7), J2.6 (Pin_6)
- net +3.3V renamed +3.3V_MCU
- net +3.3V_MCU: now also J1.10 (Pin_10), J2.3 (Pin_3), U5.5 (VCC)
- net +5V renamed +5V_MCU
- net +5V_MCU: now also J1.11 (Pin_11), J2.2 (Pin_2)
- net A0 renamed GND_MCU
- net GND_MCU: now also J1.1 (Pin_1), J1.12 (Pin_11), J1.13 (Pin_11), J2.1 (Pin_1), J2.12 (Pin_11), J2.13 (Pin_11), J3.1 (Pin_1), J3.12 (Pin_11), J3.13 (Pin_11), U5.2 (GND)
- new net: D1.2 (A), R34.2
- new net: D5.2 (A), R38.2
- new net: D6.2 (A), R39.2
- new net: D2.2 (A), R35.2
- new net: D8.2 (A), R41.2
- new net: D7.2 (A), R40.2
- new net: D4.2 (A), R37.2
- new net: D3.2 (A), R36.2
- new net CS_LED: J3.3 (Pin_3), U5.4 (2Y)
- new net INT: J1.2 (Pin_2), J2.11 (Pin_11)
- new net MISO_LED: J3.2 (Pin_2), U5.6 (1Y)
- no-connect marks 64 -> 36
Other:
- note added: "CNV"
- note added: "MCU"
- note removed: "Расширение GPIO (I2C)"
- moved on the sheet: C1, JP1, JP2, JP3, JP4, U3, U4
