File: current/PM_CNV-AI4_W-v0.0.2/PM_CNV-AI4_W.kicad_pcb (KiCad board)
At the start: 2 copper layers, 79.8 x 99.8 mm, 74 parts, among them J1 AFA07-S10FCC-00, J2 AFA07-S10FCC-00, J4 15EDGRHC-THR-3.5-14P, J5 15EDGRHC-THR-3.5-14P, U1 AD7190BRUZ, U2 AD7190BRUZ, U3 CA-IS3761HW, U4 CA-IS3105W, U5 PM-LED8_v0.0.2

Commit message: PM_CNV-AI4_W-v0.0.2
Parts:
- removed C10, C4: 10 uF, kicad_inventree_lib:TAJA_AVX-M
- removed C2, C8: 100nF, Capacitor_SMD:C_0603_1608Metric
- removed C22, C24, C31, C33, C34, C36: 10nF, Capacitor_SMD:C_0603_1608Metric
- removed C23, C32, C35: 1uF, Capacitor_SMD:C_0603_1608Metric
- removed J1: AFA07-S10FCC-00, kicad_inventree_lib:CONN10_AFA07-S10_JUS
- removed JP5, JP6, JP7, JP8: SolderJumper_2_Open, Jumper:SolderJumper-2_P1.3mm_Open_RoundedPad1.0x1.5mm
- removed R10: 10k, Resistor_SMD:R_0603_1608Metric
- removed U3: CA-IS3761HW, kicad_inventree_lib:SOIC16-WBW_CLG-M
- added J6: AFA07-S12FCC-00, kicad_inventree_lib:CONN10_AFA07-S12_JUS, F.Cu at (34.9, 110.3)
- added J7: AFA07-S12FCC-00, kicad_inventree_lib:CONN10_AFA07-S12_JUS, B.Cu at (34.9, 70.3)
- added SP1: ~, kicad_inventree_lib:PM_LED-xx-v0.0.1, F.Cu at (89.9, 100.3)
- added U7: AD7193BRUZ, kicad_inventree_lib:RU_28_ADI, F.Cu at (71.1, 100.3)
- added U8: CA-IS3741HW, kicad_inventree_lib:SOIC16-WBW_CLG-M, F.Cu at (51.9, 77.3)
- C12, C37: footprint Capacitor_SMD:C_0603_1608Metric -> Capacitor_SMD:C_0805_2012Metric
- J2: value AFA07-S10FCC-00 -> AFA07-S12FCC-00; footprint kicad_inventree_lib:CONN10_AFA07-S10_JUS -> kicad_inventree_lib:CONN10_AFA07-S12_JUS
- U1, U2: value AD7190BRUZ -> 5117; footprint kicad_inventree_lib:RU_24_ADI-M -> kicad_inventree_lib:5117
- U5: value PM-LED8_v0.0.2 -> SN74LVC2G14DBVR; footprint kicad_inventree_lib:PM-LED_v0.0.2 -> kicad_inventree_lib:DBV6-M
- U6: footprint kicad_inventree_lib:PM-ESP32C3_v0.0.4 -> kicad_inventree_lib:PM-ESP32C3_v0.0.5
- moved R11 40.9 mm to (64.9, 113.3), turned to 90 degrees
- moved U2 34.1 mm to (46.9, 90.3), turned to 0 degrees
- moved U1 27.1 mm to (49.9, 100.3), turned to 0 degrees
- moved U5 24.7 mm to (68.9, 113.3), turned to -90 degrees
- moved JP1 18.0 mm to (40.9, 65.8)
- moved JP2 17.6 mm to (40.9, 68.8)
- moved C40 17.4 mm to (66.9, 85.3), turned to 90 degrees
- moved JP3 17.1 mm to (40.9, 71.8)
- moved JP4 16.7 mm to (40.9, 74.8)
- moved C1 16.4 mm to (62.9, 92.3)
- moved C9 16.0 mm to (68.9, 92.3)
- moved R9 15.7 mm to (69.9, 85.3), turned to -90 degrees
- moved C3 14.9 mm to (65.9, 92.3)
- moved C7 14.9 mm to (71.9, 92.3)
- moved C30 11.6 mm to (81.9, 110.3), turned to 180 degrees
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Connections:
- net Net-(JP1-B) renamed /CS_MCU
- C1 pad 1: +5V_ISO -> +5V_CNV
- C1 pad 2: AGND -> GND_CNV
- C11 pad 1: +5V -> +5V_MCU
- C11 pad 2: GND -> GND_MCU
- C12 pad 1: +5V -> +5V_MCU
- C12 pad 2: GND -> GND_MCU
- C13 pad 1: AGND -> /AIN7
- C13 pad 2: /AD_0_AIN2 -> GND_CNV
- C14 pad 1: /AD_0_AIN2 -> /AIN7
- C14 pad 2: /AD_0_AIN3 -> /AIN8
- C15 pad 1: /AD_0_AIN3 -> /AIN8
- C15 pad 2: AGND -> GND_CNV
- C16 pad 1: AGND -> /AIN5
- C16 pad 2: /AD_0_AIN0 -> GND_CNV
- C17 pad 1: /AD_0_AIN0 -> /AIN5
- C17 pad 2: /AD_0_AIN1 -> /AIN6
- C18 pad 1: /AD_0_AIN1 -> /AIN6
- C18 pad 2: AGND -> GND_CNV
- C19 pad 1: AGND -> /SENSE+
- C19 pad 2: /0.SENSE+ -> GND_CNV
- C20 pad 1: /0.SENSE+ -> /SENSE+
- C20 pad 2: /0.SENSE- -> /SENSE-
- C21 pad 1: /0.SENSE- -> /SENSE-
- C21 pad 2: AGND -> GND_CNV
- C25 pad 1: AGND -> /AIN3
- C25 pad 2: /AD_1_AIN2 -> GND_CNV
- C26 pad 1: /AD_1_AIN2 -> /AIN3
- C26 pad 2: /AD_1_AIN3 -> /AIN4
- C27 pad 1: /AD_1_AIN3 -> /AIN4
- C27 pad 2: AGND -> GND_CNV
- C28 pad 1: AGND -> /AIN1
- C28 pad 2: /AD_1_AIN0 -> GND_CNV
- C29 pad 1: /AD_1_AIN0 -> /AIN1
- C29 pad 2: /AD_1_AIN1 -> /AIN2
- C3 pad 1: +5V_ISO -> +5V_CNV
- C3 pad 2: AGND -> GND_CNV
- C30 pad 1: /AD_1_AIN1 -> /AIN2
- C30 pad 2: AGND -> GND_CNV
- C37 pad 1: +5V_ISO -> +5V_CNV
- C37 pad 2: AGND -> GND_CNV
- C38 pad 1: +5V_ISO -> +5V_CNV
- C38 pad 2: AGND -> GND_CNV
- C39 pad 1: +5V_ISO -> +5V_CNV
- C39 pad 2: AGND -> GND_CNV
- C40 pad 1: AVDD -> +5V_CNV_FLT
- C40 pad 2: AGND -> GND_CNV
- C5 pad 1: +3.3V -> +3.3V_MCU
- C5 pad 2: GND -> GND_MCU
- C6 pad 1: +5V_ISO -> DGND
- C6 pad 2: AGND -> +5V_CNV
- C7 pad 1: AVDD -> +5V_CNV_FLT
- C7 pad 2: AGND -> GND_CNV
- C9 pad 1: AVDD -> +5V_CNV_FLT
- C9 pad 2: AGND -> GND_CNV
- J2 pad 1: GND -> GND_MCU
- J2 pad 10: +5V -> +3.3V_MCU
- J2 pad 11: GND -> +5V_MCU
- J2 pad 2: /CS3 -> /INT_MCU
- J2 pad 3: /CS2 -> /CS3_MCU
- J2 pad 4: /CS1 -> /CS2_MCU
- J2 pad 5: /CS0 -> /CS1_MCU
- J2 pad 6: /SCK -> /CS0_MCU
- J2 pad 7: /MISO -> /SCK_MCU
- J2 pad 8: /MOSI -> /MISO_MCU
- J2 pad 9: +3.3V -> /MOSI_MCU
- J4 pad 1: AGND -> GND_CNV
- J4 pad 11: /1.SENSE- -> /SENSE-
- J4 pad 12: /1.SENSE+ -> /SENSE+
- J4 pad 13: /0.EXC- -> /EXC-
- J4 pad 14: AVDD -> +5V_CNV_FLT
- J4 pad 4: /0.SENSE- -> /SENSE-
- J4 pad 5: /0.SENSE+ -> /SENSE+
- J4 pad 6: /0.EXC- -> /EXC-
- J4 pad 7: AVDD -> +5V_CNV_FLT
- J4 pad 8: AGND -> GND_CNV
- J5 pad 1: AGND -> GND_CNV
- J5 pad 11: /3.SENSE- -> /SENSE-
- J5 pad 12: /3.SENSE+ -> /SENSE+
- J5 pad 13: /2.EXC- -> /EXC-
- J5 pad 14: AVDD -> +5V_CNV_FLT
- J5 pad 4: /2.SENSE- -> /SENSE-
- J5 pad 5: /2.SENSE+ -> /SENSE+
- J5 pad 6: /2.EXC- -> /EXC-
- J5 pad 7: AVDD -> +5V_CNV_FLT
- J5 pad 8: AGND -> GND_CNV
- JP1 pad 1: /CS0 -> /CS0_MCU
- JP2 pad 1: /CS1 -> /CS1_MCU
- JP3 pad 1: /CS2 -> /CS2_MCU
- JP4 pad 1: /CS3 -> /CS3_MCU
- L1 pad 2: +5V_ISO -> +5V_CNV
- R1 pad 1: /AD_0_AIN2 -> /AIN7
- R11 pad 1: +3.3V -> +5V_CNV
- R11 pad 2: Net-(JP5-B) -> /CS_CNV
- R2 pad 1: /AD_0_AIN3 -> /AIN8
- R3 pad 1: /AD_0_AIN0 -> /AIN5
- R4 pad 1: /AD_0_AIN1 -> /AIN6
- R5 pad 1: /AD_1_AIN2 -> /AIN3
- R6 pad 1: /AD_1_AIN3 -> /AIN4
- R7 pad 1: /AD_1_AIN0 -> /AIN1
- R8 pad 1: /AD_1_AIN1 -> /AIN2
- R9 pad 2: AVDD -> +5V_CNV_FLT
- U1 pad 1: unconnected-(U1-MCLK1-Pad1) -> GND_CNV
- U2 pad 1: unconnected-(U2-MCLK1-Pad1) -> GND_MCU
- U4 pad 1: +5V -> +5V_MCU
- U4 pad 10: AGND -> GND_CNV
- U4 pad 11: AGND -> GND_CNV
- U4 pad 12: AGND -> GND_CNV
- U4 pad 13: +5V_ISO -> +5V_CNV
- U4 pad 14: +5V_ISO -> +5V_CNV
- U4 pad 15: AGND -> GND_CNV
- U4 pad 16: AGND -> GND_CNV
- U4 pad 2: GND -> GND_MCU
- U4 pad 3: +5V -> +5V_MCU
- U4 pad 4: GND -> GND_MCU
- U4 pad 5: GND -> GND_MCU
- U4 pad 6: GND -> GND_MCU
- U4 pad 7: GND -> GND_MCU
- U4 pad 8: GND -> GND_MCU
- U4 pad 9: AGND -> GND_CNV
Routing:
- net +5V_CNV: track 0.00 -> 145.9 mm, vias 0 -> 2
- net AVDD: track 109.8 -> 0.00 mm, vias 2 -> 0
- net +5V_ISO: track 93.2 -> 0.00 mm
- net +5V_CNV_FLT: track 0.00 -> 92.7 mm
- net /SENSE-: track 0.00 -> 82.0 mm
- net /EXC-: track 0.00 -> 81.6 mm
- net /SENSE+: track 0.00 -> 75.5 mm
- net /SCK_ISO: track 58.9 -> 0.00 mm, vias 2 -> 0
- net AGND: track 58.7 -> 0.00 mm, vias 37 -> 0
- net /LED1: track 56.9 -> 0.00 mm, vias 2 -> 0
- net /LED0: track 53.6 -> 0.00 mm, vias 2 -> 0
- net /CS1_ISO: track 48.7 -> 0.00 mm
- net /CS_CNV: track 0.00 -> 48.7 mm, vias 0 -> 2
- net /MOSI_ISO: track 48.5 -> 0.00 mm, vias 2 -> 0
- net /MISO_ISO: track 48.3 -> 0.00 mm, vias 3 -> 0
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- added copper zone on B.Cu, net GND_CNV
- added copper zone on F.Cu, net GND_CNV
- added copper zone on B.Cu, net GND_MCU
- added copper zone on F.Cu, net GND_MCU
- removed copper zone on B.Cu, net AGND
- removed copper zone on B.Cu, net GND
- removed copper zone on F.Cu, net GND
Other:
- board size 79.8 x 99.8 mm -> 80 x 100 mm
- board text added: "GND CNV"
- board text added: "GND MCU"
- board text added: "Shield"
- board text removed: "GND"

Commit message: nextpcb order
Routing:
- net +5V_MCU: track 33.8 -> 29.7 mm, vias 6 -> 4
- net +3.3V_MCU: track 45.6 -> 41.5 mm, vias 6 -> 4
- net /MOSI_CNV: track 27.9 -> 29.1 mm
- net GND_CNV: vias 29 -> 44
- added copper zone on B.Cu, net +3.3V_MCU
- added copper zone on F.Cu, net +3.3V_MCU
- added copper zone on B.Cu, net +5V_MCU
- added copper zone on F.Cu, net +5V_MCU
Changed lines of the file:
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@@
 			(outputformat 1)
 			(mirror no)
-			(drillshape 1)
+			(drillshape 0)
 			(scaleselection 1)
-			(outputdirectory "")
+			(outputdirectory "./test_gerber")
 		)
 	)
@@
 	)
 	(segment
-		(start 96.52 90.79)
-		(end 97.871 92.141)
+		(start 87.93 98.33)
+		(end 87.755 98.33)
 		(width 0.3)
 		(layer "F.Cu")
@@
 	)
 	(segment
-		(start 87.93 98.33)
-		(end 87.755 98.33)
+		(start 97.871 94.849603)
+		(end 96.390603 96.33)
 		(width 0.3)
 		(layer "F.Cu")
@@
 	)
 	(segment
-		(start 97.871 94.849603)
-		(end 96.281603 96.439)
+		(start 96.52 90.79)
+		(end 97.871 92.141)
 		(width 0.3)
 		(layer "F.Cu")
@@
 	)
 	(segment
-		(start 96.281603 96.439)
-		(end 89.821 96.439)
+		(start 96.390603 96.33)
+		(end 89.93 96.33)
 		(width 0.3)
 		(layer "F.Cu")
@@
 	)
 	(segment
-		(start 89.821 96.439)
+		(start 89.93 96.33)
 		(end 87.93 98.33)
 		(width 0.3)
@@
 	)
 	(via
-		(at 34.43 66.830004)
-		(size 0.8)
-		(drill 0.4)
-		(layers "F.Cu" "B.Cu")
-		(net 26)
-	)
-	(via
-		(at 33.43 66.830004)
-		(size 0.8)
-		(drill 0.4)
-		(layers "F.Cu" "B.Cu")
-		(net 26)
-	)
-	(via
-		(at 35.43 66.830004)
+		(at 28.43 66.830004)
 		(size 0.8)
 		(drill 0.4)
@@
 	)
 	(via
-		(at 28.43 66.830004)
+		(at 27.43 67.83)
 		(size 0.8)
 		(drill 0.4)
@@
 	)
 	(segment
-		(start 31.374 66.830004)
-		(end 33.43 66.830004)
-		(width 0.6)
-		(layer "B.Cu")
-		(net 26)
-	)
-	(segment
 		(start 31.373996 66.83)
 		(end 31.374 66.830004)
@@
 	)
 	(segment
-		(start 33.43 66.830004)
-		(end 34.43 66.830004)
-		(width 0.6)
-		(layer "B.Cu")
-		(net 26)
-	)
-	(segment
-		(start 34.43 66.830004)
-		(end 35.43 66.830004)
-		(width 0.6)
-		(layer "B.Cu")
-		(net 26)
-	)
-	(segment
 		(start 31.373994 74.83)
 		(end 31.374 74.829994)
@@
 	)
 	(segment
-		(start 66.88 97.5106)
-		(end 66.039778 97.5106)
+		(start 60.73 77.33)
+		(end 58.825 75.425)
 		(width 0.3)
 		(layer "F.Cu")
@@
 	)
 	(segment
-		(start 58.825 75.425)
-		(end 56.8068 75.425)
+		(start 66.88 97.5106)
+		(end 64.1106 97.5106)
 		(width 0.3)
 		(layer "F.Cu")
@@
 	)
 	(segment
-		(start 60.73 92.200822)
+		(start 60.73 94.13)
 		(end 60.73 77.33)
 		(width 0.3)
@@
 	)
 	(segment
-		(start 66.039778 97.5106)
-		(end 60.73 92.200822)
+		(start 64.1106 97.5106)
+		(end 60.73 94.13)
 		(width 0.3)
 		(layer "F.Cu")
@@
 	)
 	(segment
-		(start 60.73 77.33)
-		(end 58.825 75.425)
+		(start 58.825 75.425)
+		(end 56.8068 75.425)
 		(width 0.3)
 		(layer "F.Cu")
@@
 	)
 	(via
-		(at 35.43 65.830006)
-		(size 0.8)
-		(drill 0.4)
-		(layers "F.Cu" "B.Cu")
-		(net 40)
-	)
-	(via
-		(at 34.43 65.830006)
-		(size 0.8)
-		(drill 0.4)
-		(layers "F.Cu" "B.Cu")
-		(net 40)
-	)
-	(via
 		(at 27.43 65.83)
 		(size 0.8)
@@
 	)
 	(via
-		(at 29.43 65.83)
+		(at 27.43 64.83)
 		(size 0.8)
 		(drill 0.4)
@@
 	)
 	(via
-		(at 33.43 65.830006)
+		(at 29.43 65.83)
 		(size 0.8)
 		(drill 0.4)
@@
 		(net 40)
 	)
-	(segment
-		(start 33.43 65.830006)
-		(end 34.43 65.830006)
-		(width 0.6)
-		(layer "B.Cu")
-		(net 40)
+	(via
+		(at 60.93 68.83)
+		(size 0.8)
+		(drill 0.4)
+		(layers "F.Cu" "B.Cu")
+		(free yes)
+		(net 41)
 	)
-	(segment
-		(start 31.374 65.830006)
-		(end 33.43 65.830006)
-		(width 0.6)
-		(layer "B.Cu")
-		(net 40)
+	(via
+		(at 58.93 70.83)
+		(size 0.8)
+		(drill 0.4)
+		(layers "F.Cu" "B.Cu")
+		(free yes)
+		(net 41)
 	)
-	(segment
-		(start 34.43 65.830006)
-		(end 35.43 65.830006)
-		(width 0.6)
-		(layer "B.Cu")
-		(net 40)
+	(via
+		(at 94.93 129.83)
+		(size 0.8)
+		(drill 0.4)
+		(layers "F.Cu" "B.Cu")
+		(free yes)
+		(net 41)
+	)
+	(via
+		(at 59.93 69.83)
+		(size 0.8)
+		(drill 0.4)
+		(layers "F.Cu" "B.Cu")
+		(free yes)
+		(net 41)
 	)
 	(via
@@
 	)
 	(via
+		(at 92.93 129.83)
+		(size 0.8)
+		(drill 0.4)
+		(layers "F.Cu" "B.Cu")
+		(free yes)
+		(net 41)
+	)
+	(via
 		(at 61.93 88.83)
 		(size 0.8)
@@
 	)
 	(via
+		(at 60.93 70.83)
+		(size 0.8)
+		(drill 0.4)
+		(layers "F.Cu" "B.Cu")
+		(free yes)
+		(net 41)
+	)
+	(via
 		(at 57.93 85.33)
 		(size 0.8)
@@
 	)
 	(via
+		(at 92.93 72.83)
+		(size 0.8)
+		(drill 0.4)
+		(layers "F.Cu" "B.Cu")
+		(free yes)
+		(net 41)
+	)
+	(via
+		(at 94.93 70.83)
+		(size 0.8)
+		(drill 0.4)
+		(layers "F.Cu" "B.Cu")
+		(free yes)
+		(net 41)
+	)
+	(via
 		(at 68.93 87.83)
 		(size 0.8)
@@
 	)
 	(via
+		(at 58.93 68.83)
+		(size 0.8)
+		(drill 0.4)
+		(layers "F.Cu" "B.Cu")
+		(free yes)
+		(net 41)
+	)
+	(via
 		(at 55.93 85.33)
 		(size 0.8)
@@
 	)
 	(via
+		(at 93.93 128.83)
+		(size 0.8)
+		(drill 0.4)
+		(layers "F.Cu" "B.Cu")
+		(free yes)
+		(net 41)
+	)
+	(via
+		(at 93.93 71.83)
+		(size 0.8)
+		(drill 0.4)
+		(layers "F.Cu" "B.Cu")
+		(free yes)
+		(net 41)
+	)
+	(via
 		(at 61.43 75.83)
 		(size 0.8)
@@
 	)
 	(via
+		(at 92.93 127.83)
+		(size 0.8)
+		(drill 0.4)
+		(layers "F.Cu" "B.Cu")
+		(free yes)
+		(net 41)
+	)
+	(via
 		(at 72.93 86.83)
 		(size 0.8)
@@
 	)
 	(via
+		(at 92.93 70.83)
+		(size 0.8)
+		(drill 0.4)
+		(layers "F.Cu" "B.Cu")
+		(free yes)
+		(net 41)
+	)
+	(via
 		(at 59.93 58.83)
 		(size 0.8)
@@
 	)
 	(via
+		(at 94.93 127.83)
+		(size 0.8)
+		(drill 0.4)
+		(layers "F.Cu" "B.Cu")
+		(free yes)
+		(net 41)
+	)
+	(via
 		(at 71.93 87.83)
 		(size 0.8)
@@
 	)
 	(via
+		(at 94.93 72.83)
+		(size 0.8)
+		(drill 0.4)
+		(layers "F.Cu" "B.Cu")
+		(free yes)
+		(net 41)
+	)
+	(via
 		(at 60.93 59.83)
 		(size 0.8)
@@
 	)
 	(zone
+		(net 40)
+		(net_name "+5V_MCU")
+		(layers "F.Cu" "B.Cu")
+		(hatch edge 0.5)
+		(priority 3)
+		(connect_pads yes
+			(clearance 0.3)
+		)
+		(min_thickness 0.25)
+		(filled_areas_thickness no)
+		(fill yes
+			(thermal_gap 0.5)
+			(thermal_bridge_width 0.5)
+		)
+		(polygon
+			(pts
+				(xy 26.93 64.33) (xy 27.93 64.33) (xy 28.93 65.33) (xy 32.43 65.33) (xy 32.43 66.33) (xy 26.93 66.33)
+			)
+		)
+	)
+	(zone
+		(net 26)
+		(net_name "+3.3V_MCU")
+		(layers "F.Cu" "B.Cu")
+		(hatch edge 0.5)
+		(priority 2)
+		(connect_pads yes
+			(clearance 0.3)
+		)
+		(min_thickness 0.25)
+		(filled_areas_thickness no)
+		(fill yes
+			(thermal_gap 0.5)
+			(thermal_bridge_width 0.5)
+		)
+		(polygon
+			(pts
+				(xy 26.93 66.33) (xy 32.43 66.33) (xy 32.43 67.33) (xy 28.93 67.33) (xy 27.93 68.33) (xy 26.93 68.33)
+			)
+		)
+	)
+	(zone
 		(net 39)
 		(net_name "GND_MCU")
 		(layers "F.Cu" "B.Cu")
 		(hatch edge 0.5)
-		(priority 2)
+		(priority 1)
 		(connect_pads
 			(clearance 0.4)
@@
 		(polygon
 			(pts
-				(xy 23.93 49.33) (xy 23.93 93.33) (xy 49.93 93.33) (xy 49.93 49.33)
+				(xy 49.93 93.33) (xy 23.93 93.33) (xy 23.93 49.33) (xy 49.93 49.33)
+			)
+		)
+		(polygon
+			(pts
+				(xy 26.93 64.33) (xy 26.93 68.33) (xy 27.93 68.33) (xy 28.93 67.33) (xy 32.43 67.33) (xy 32.43 65.33)
+				(xy 28.93 65.33) (xy 27.93 64.33)
 			)
 		)
@@
 		(fill yes
 			(thermal_gap 0.4)
-			(thermal_bridge_width 0.5)
+			(thermal_bridge_width 0.6)
 		)
 		(polygon

Commit message: update docs
Parts:
- renumbered C12 to C1, C9 to C10, C39 to C11, C7 to C12, C20 to C13, C17 to C15, C26 to C16, C29 to C17, C21 to C18, C11 to C2, C15 to C20, C13 to C21, C18 to C22, C16 to C23, C27 to C24, C30 to C26, C28 to C27, C5 to C3, C38 to C4, C6 to C5, C37 to C6, C1 to C7, C3 to C8, C40 to C9, H2 to H1, H3 to H2, H4 to H3, H1 to H4, J2 to J1, J6 to J2, J4 to J3, J5 to J4, J7 to J5, R11 to R1, R7 to R10, R9 to R2, R2 to R3, R1 to R4, R4 to R5, R3 to R6, R6 to R7, R5 to R8, R8 to R9, U6 to U1, U1 to U3, U8 to U5, U5 to U6
Other:
- board text added: "CS0"
- board text added: "CS1"
- board text added: "CS2"
- board text added: "CS3"
- board text added: "LED"
- board text added: "SPI"

Commit message: update
Parts:
- removed C4: 100nF, Capacitor_SMD:C_0603_1608Metric
- removed C6: 10uF, Capacitor_SMD:C_0805_2012Metric
- removed U4: CA-IS3105W, kicad_inventree_lib:SOIC16-WBW_CLG-M
- added PS1: 5V/5V, kicad_inventree_lib:B2405LS-1WR3, F.Cu at (32.1, 97.4)
- C1: value 10uF -> 4.7uF
- C2: value 100nF -> 10uF; footprint Capacitor_SMD:C_0603_1608Metric -> Capacitor_SMD:C_0805_2012Metric
- JP1, JP2, JP3, JP4: footprint Jumper:SolderJumper-2_P1.3mm_Open_RoundedPad1.0x1.5mm -> kicad_inventree_lib:SolderJumper-2_P1.3mm_Open_RoundedPad1.0x1.5mm
- moved C2 38.5 mm to (35.4, 99.8)
- moved C1 29.2 mm to (35.4, 90.8), turned to -90 degrees
- moved J2 8.00 mm to (42.9, 110.3)
- moved J3 1.91 mm to (95.9, 90.8)
- moved J4 1.91 mm to (95.9, 116.9)
Connections:
- C2 pad 1: +5V_MCU -> +5V_CNV
- C2 pad 2: GND_MCU -> GND_CNV
Routing:
- net +5V_MCU: track 29.7 -> 38.9 mm
- net /P3: track 40.2 -> 32.2 mm
- net /P2: track 41.3 -> 33.3 mm
- net /P1: track 42.4 -> 34.4 mm
- net /P0: track 43.5 -> 35.5 mm
- net /CS_LED: track 37.1 -> 29.1 mm
- net /MISO_LED: track 39.8 -> 31.9 mm
- net /SENSE-: track 82.0 -> 88.5 mm
- net +5V_CNV: track 145.9 -> 140.3 mm
- net /SENSE+: track 75.5 -> 80.3 mm
- net /EXC-: track 81.6 -> 86.4 mm
- net /1.SIG+: track 16.2 -> 18.2 mm
- net /2.SIG-: track 21.3 -> 23.2 mm
- net /2.SIG+: track 13.1 -> 15.0 mm
- net /0.SIG-: track 13.3 -> 15.2 mm
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Other:
- outline, holes or cut-outs redrawn
