File: current/PMCPU-LLP-v0.0.1/PMCPU-LLP.kicad_sch (KiCad schematic)
At the start: 62 parts, among them J10 15EDGKNH-3.5-10P, J11 PinHeader_01x03_P2.00_THT_str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, J12 AFA07-S10FCC-00, J13 15EDGRC-3.5-07P, J14 15EDGRC-3.5-05P, J2 AFA07-S10FCC-00, J3 15EDGRHC-THR-3.5-10P, J4 K7805-2000R3, J5 K7803-2000R3, J6 FFC_12P_P1.0_100mm_straight, J7 AFA07-S10FCC-00, J8 AFA07-S10FCC-00, J9 AFA07-S10FCC-00, U1 64900001039, U2 5117, U4 CA-IS3098W, U5 CA-IS3062VW, U6 DS3231, U7 SN74LVC2G14DBVR, U8 CA-IS3098W

Commit message: update
Parts:
- removed J12, J2, J8, J9: AFA07-S10FCC-00, kicad_inventree_lib:CONN10_AFA07-S12_JUS, symbol kicad_inventree_lib:AFA07-S12FCC-00
- added JM1, JM2: AFA07-S20FCC-00, kicad_inventree_lib:AFA07S20FCA00, symbol kicad_inventree_lib:AFA07-S20FCC-00
Connections:
- net +3.3V_CPU: now also JM1.15 (Pin_11), JM1.16 (Pin_11), JM2.5 (Pin_5), JM2.6 (Pin_6)
- net +5V_CPU: now also JM1.17 (Pin_11), JM1.18 (Pin_11), JM2.3 (Pin_3), JM2.4 (Pin_4)
- net GND_BUS: now also JM1.1 (Pin_1), JM1.14 (Pin_11), JM1.19 (Pin_11), JM1.2 (Pin_2), JM1.20 (Pin_11), JM1.5 (Pin_5), JM1.6 (Pin_6), JM1.MP1 (Pin_11), JM1.MP2 (Pin_11), JM2.1 (Pin_1), JM2.15 (Pin_11), JM2.16 (Pin_11), JM2.19 (Pin_11), JM2.2 (Pin_2), JM2.20 (Pin_11), JM2.7 (Pin_7), JM2.MP1 (Pin_11), JM2.MP2 (Pin_11)
- net I2C0_SCL: now also JM1.3 (Pin_3), JM2.18 (Pin_11)
- net I2C0_SDA: now also JM1.4 (Pin_4), JM2.17 (Pin_11)
- net RTS_EXT: now also U3.24 (RM_IO29)
- net SPI_CS0: now also JM1.10 (Pin_10), JM2.11 (Pin_11)
- net SPI_CS1: now also JM1.9 (Pin_9), JM2.12 (Pin_11)
- net SPI_CS2: now also JM1.8 (Pin_8), JM2.13 (Pin_11)
- net SPI_CS3: now also JM1.7 (Pin_7), JM2.14 (Pin_11)
- net SPI_MISO: now also JM1.12 (Pin_11), JM2.9 (Pin_9)
- net SPI_MOSI: now also JM1.13 (Pin_11), JM2.8 (Pin_8)
- net SPI_SCK: now also JM1.11 (Pin_11), JM2.10 (Pin_10)
- no-connect marks 27 -> 31
Other:
- note added: "Коннектор MCU"
- note removed: "Коннектор I2C"
- note removed: "Коннектор SPI"
