File: current/PMMCU-ESP32C3-v0.0.7/PMMCU-ESP32C3.kicad_pcb (KiCad board)
At the start: 2 copper layers, 34 x 96 mm, 35 parts, among them J1 U254-051T-4BH83-S1S, J4 AFA07-S12FCC-00, J6 15EDGRHC-THR-3.5-10P, J7 PinHeader_01x03_P2.00_THT_str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, SW1 Button, SW2 Button, SW4 DIP 3 pos, U1 ESP32-C3-WROOM-02U-N4, U2 CJA1117B-3.3, U3 5117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

Commit message: update
Parts:
- removed C3, C6: 10uF, Capacitor_SMD:C_0805_2012Metric
- removed C8, C9: 100nF, Capacitor_SMD:C_0603_1608Metric
- removed J7: PinHeader_01x03_P2.00_THT_straight, Connector_PinHeader_2.00mm:PinHeader_1x03_P2.00mm_Vertical
- removed SW4: DIP 3 pos, kicad_inventree_lib:DA03BLP
- removed U6: CA-IS3098W, kicad_inventree_lib:SOIC16-WBW_CLG
- added C11: 100nF, Capacitor_SMD:C_0603_1608Metric, F.Cu at (53.5, 125.5)
- added C12: 1uF, Capacitor_SMD:C_0603_1608Metric, F.Cu at (49.0, 125.5)
- added C13: 10uF, Capacitor_SMD:C_0805_2012Metric, F.Cu at (56.0, 125.5)
- added C14: 10uF, Capacitor_SMD:C_0805_2012Metric, F.Cu at (56.0, 109.0)
- added C15: 1uF, Capacitor_SMD:C_0603_1608Metric, F.Cu at (48.0, 109.0)
- added C16: 100nF, Capacitor_SMD:C_0603_1608Metric, F.Cu at (56.0, 106.5)
- added CR1: STWD100NYWY3F, kicad_inventree_lib:SOT23-5L_STM, F.Cu at (63.5, 69.0)
- added JP1: SolderJumper_2_Open, kicad_inventree_lib:SolderJumper-2_P1.3mm_Open_RoundedPad1.0x1.5mm, F.Cu at (54.0, 61.0)
- added JP2: SolderJumper_2_Open, kicad_inventree_lib:SolderJumper-2_P1.3mm_Open_RoundedPad1.0x1.5mm, F.Cu at (57.0, 61.0)
- added JP3: SolderJumper_2_Open, kicad_inventree_lib:SolderJumper-2_P1.3mm_Open_RoundedPad1.0x1.5mm, F.Cu at (60.0, 61.0)
- added U7: CA-IS3062VW, kicad_inventree_lib:SOIC16-WBW_CLG-M, F.Cu at (52.0, 117.0)
- moved J1 4.25 mm to (67.2, 57.7)
- moved C7 1.93 mm to (49.8, 130.5), turned to -90 degrees
Connections:
- net /A renamed /CANL_BUS
- net /B renamed /CANH_BUS
- JM1 pad 5: GND_MCU -> unconnected-(JM1-Pin_5-Pad5)
- JM1 pad 6: GND_MCU -> /RST
- RN1 pad 6: unconnected-(RN1C-R3.2-Pad6) -> /CS0_MCU
- RN1 pad 7: /CS0_MCU -> /CS1_MCU
- RN1 pad 8: /CS1_MCU -> /RST
- U1 pad 11: /UART_RX -> /WDT
- U1 pad 12: /UART_TX -> /LED2
- U1 pad 3: /UART_RTS -> /CAN_TX
- U1 pad 4: /LED2 -> /CAN_RX
- U5 pad 1: /UART_RX -> /CAN_RX
- U5 pad 3: /UART_TX -> /CAN_TX
Routing:
- net /UART_RX: track 64.9 -> 0.00 mm
- net /UART_TX: track 63.1 -> 0.00 mm, vias 1 -> 0
- net /CAN_RX: track 0.00 -> 46.3 mm, vias 0 -> 2
- net /CAN_TX: track 0.00 -> 43.9 mm
- net /UART_RTS: track 35.7 -> 0.00 mm
- net /RST: track 0.00 -> 30.1 mm, vias 0 -> 3
- net GND_MCU: track 75.3 -> 100.1 mm, vias 22 -> 20
- net +5V_MCU: track 87.2 -> 106.9 mm, vias 0 -> 2
- net /LED2: track 52.0 -> 67.4 mm, vias 3 -> 2
- net +5V_BUS: track 0.00 -> 15.1 mm, vias 0 -> 2
- net +3.3V_MCU: track 165.5 -> 178.7 mm, vias 4 -> 6
- net GND_BUS: track 58.4 -> 68.7 mm
- net +3.3V_BUS: track 9.19 -> 0.00 mm
- net /WDT: track 0.00 -> 4.22 mm
- net +24V_BUS: track 15.6 -> 18.3 mm
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Other:
- board text added: "-"
- board text added: "IO21"
- board text added: "RST"
- board text removed: "IO5"
