File: current/PMMCU-ESP32C3-v0.0.7/PMMCU-ESP32C3.kicad_sch (KiCad schematic)
At the start: 49 parts, among them J1 U254-051T-4BH83-S1S, J4 AFA07-S12FCC-00, J5 15EDGKNH-3.5-10P, J6 15EDGRHC-THR-3.5-10P, J7 PinHeader_01x03_P2.00_THT_str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, SW1 Button, SW2 Button, SW4 DIP 3 pos, U1 ESP32-C3-WROOM-02U-N4, U2 CJA1117B-3.3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

Commit message: update
Parts:
- removed C3, C6: 10uF, Capacitor_SMD:C_0805_2012Metric, symbol kicad_inventree_lib:C_10uF_16V_0805_MLCC-X7R
- removed C8, C9: 100nF, Capacitor_SMD:C_0603_1608Metric, symbol kicad_inventree_lib:C_100nF_16V_0603_MLCC-X7R
- removed J7: PinHeader_01x03_P2.00_THT_straight, Connector_PinHeader_2.00mm:PinHeader_1x03_P2.00mm_Vertical, symbol kicad_inventree_lib:PinHeader_01x03_P2.00_THT_straight
- removed SW4: DIP 3 pos, kicad_inventree_lib:DA03BLP, symbol kicad_inventree_lib:DA-03BLP
- removed U6: CA-IS3098W, kicad_inventree_lib:SOIC16-WBW_CLG, symbol kicad_inventree_lib:CA-IS3098W
- added C11, C16: 100nF, Capacitor_SMD:C_0603_1608Metric, symbol kicad_inventree_lib:C_100nF_16V_0603_MLCC-X7R
- added C12, C15: 1uF, Capacitor_SMD:C_0603_1608Metric, symbol kicad_inventree_lib:C_1uF_50V_0603_MLCC-X7R
- added C13, C14: 10uF, Capacitor_SMD:C_0805_2012Metric, symbol kicad_inventree_lib:C_10uF_16V_0805_MLCC-X7R
- added CR1: STWD100NYWY3F, kicad_inventree_lib:SOT23-5L_STM, symbol kicad_inventree_lib:STWD100NYWY3F
- added JP1, JP2, JP3: SolderJumper_2_Open, kicad_inventree_lib:SolderJumper-2_P1.3mm_Open_RoundedPad1.0x1.5mm, symbol kicad_inventree_lib:SolderJumper_2_Open
- added U7: CA-IS3062VW, kicad_inventree_lib:SOIC16-WBW_CLG-M, symbol kicad_inventree_lib:CA-IS3062VW
Connections:
- net +3.3V_MCU: now also C15.1, CR1.5 (VCC), U7.7 (Vccl)
- net +5V_MCU: now also C14.1, C16.1, U7.1 (Vcc)
- net CS0_MCU: now also RN1.6 (R3.2); no longer RN1.7 (R2.2)
- net CS1_MCU: now also RN1.7 (R2.2); no longer RN1.8 (R1.2)
- net GND_BUS: now also C11.2, C12.2, C13.2, U7.10 (GND2), U7.15 (GND2), U7.9 (GND2)
- net GND_MCU: now also C14.2, C15.2, C16.2, CR1.2 (GND), JP1.2 (B), JP2.2 (B), JP3.2 (B), U7.2 (GND1), U7.8 (GND1); no longer JM1.5 (Pin_5), JM1.6 (Pin_6)
- net LED2: now also U1.12 (TXD_(IO21)); no longer U1.4 (IO5)
- net at RN3.2 (R2.1): now also JP3.1 (A)
- net at RN3.3 (R3.1): now also JP2.1 (A)
- net at RN3.4 (R4.1): now also JP1.1 (A)
- net A renamed CANL_BUS
- net CANL_BUS: now also U7.12 (CANL)
- net B renamed CANH_BUS
- net CANH_BUS: now also U7.13 (CANH)
- net UART_RTS renamed CAN_TX
- net CAN_TX: now also U5.3 (2A), U7.3 (TXD)
- net UART_RX renamed CAN_RX
- net CAN_RX: now also U1.4 (IO5), U7.5 (RXD); no longer U1.11 (RXD_(IO20))
- removed net UART_TX: U1.12 (TXD_(IO21)), U5.3 (2A)
- new net: U7.14 (NC), U7.4 (NC), U7.6 (NC)
- new net +5V_BUS: C11.1, C12.1, C13.1, U7.11 (Visoin), U7.16 (Viso)
- new net RST: CR1.1 (*WDO), JM1.6 (Pin_6), RN1.8 (R1.2)
- new net WDT: CR1.4 (WDI), U1.11 (RXD_(IO20))
- no-connect marks 25 -> 23
Other:
- note added: "Watchdog"
- note added: "Плата светодиодов"
- note added: "Шина между модулями CAN"
- note removed: "RS-485"
- note removed: "Тестовый коннектор"
- moved on the sheet: C1, C10, C2, C4, C5, C7, J1, J4, J5, J6, JM1, PS1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
