File: current/PMCNV-RQx8-v0.0.8/PMCNV-RQx8.kicad_pcb (KiCad board)
At the start: 2 copper layers, 80 x 100 mm, 33 parts, among them J2 15EDGRC-3.5-08P, J3 AFA07-S12FCC-00, J4 15EDGRC-3.5-08P, J6 15EDGRC-3.5-05P, K1 G5NB-1A-E-DC5, K2 G5NB-1A-E-DC5, K3 G5NB-1A-E-DC5, K4 G5NB-1A-E-DC5, K5 G5NB-1A-E-DC5, K6 G5NB-1A-E-DC5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

Commit message: update
Parts:
- moved C7 0.51 mm to (86.4, 125.3)
- moved C10 0.50 mm to (86.4, 134.3)
Routing:
- net /A1: track 10.7 -> 10.0 mm
- net +5V_EXT: track 56.8 -> 57.3 mm
