File: current/PMCPU-LLU-v0.0.2/PMCPU-LLU.kicad_pcb (KiCad board)
At the start: 2 copper layers, 80 x 100 mm, 32 parts, among them J11 PinHeader_01x03_P2.00_THT_str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, J12 AFA07-S10FCC-00, J2 AFA07-S10FCC-00, J3 15EDGRHC-THR-3.5-10P, J4 K7805-2000R3, J5 K7803-2000R3, J7 AFA07-S10FCC-00, J8 AFA07-S10FCC-00, J9 AFA07-S10FCC-00, U1 64900001039, U2 5117, U4 CA-IS3098W, U6 DS3231, U7 SN74LVC2G14DBVR

Commit message: update
Parts:
- removed J11: PinHeader_01x03_P2.00_THT_straight, Connector_PinHeader_2.00mm:PinHeader_1x03_P2.00mm_Vertical
- removed J12, J2, J8, J9: AFA07-S10FCC-00, kicad_inventree_lib:CONN10_AFA07-S12_JUS
- removed the J3 at (52.9, 137.3)
- removed J4: K7805-2000R3, kicad_inventree_lib:K7805-2000R3
- removed the J5 at (51.5, 122.3)
- removed PE1: PE, kicad_inventree_lib:PE
- removed the U2 at (37.9, 80.3)
- removed the U4 at (68.6, 137.2)
- added C1: 100nF, Capacitor_SMD:C_0603_1608Metric, F.Cu at (60.9, 132.3)
- added C13: 100nF, Capacitor_SMD:C_0603_1608Metric, F.Cu at (101.9, 120.3)
- added C14: 10uF, Capacitor_SMD:C_0805_2012Metric, F.Cu at (101.9, 130.3)
- added C15: 1uF, Capacitor_SMD:C_0603_1608Metric, F.Cu at (101.9, 137.3)
- added C16: 10uF, Capacitor_SMD:C_0805_2012Metric, F.Cu at (101.9, 117.3)
- added C17: 100nF, Capacitor_SMD:C_0603_1608Metric, F.Cu at (101.9, 133.3)
- added C4: 10uF, Capacitor_SMD:C_0805_2012Metric, F.Cu at (78.9, 135.3)
- added C8: 100nF, Capacitor_SMD:C_0603_1608Metric, F.Cu at (83.9, 120.3)
- added CR1: STWD100NYWY3F, kicad_inventree_lib:SOT23-5L_STM, F.Cu at (58.8, 71.8)
- added D9: B5819W, Diode_SMD:D_SOD-123, F.Cu at (61.3, 109.3)
- added H4: M4, MountingHole:MountingHole_4.3mm_M4_Pad_Via, F.Cu at (96.9, 145.3)
- added J1: 15EDGRC-3.5-05P, kicad_inventree_lib:15EDGRC-3.5-05P, F.Cu at (61.9, 140.3)
- added J6: 15EDGRC-3.5-05P, kicad_inventree_lib:15EDGRC-3.5-05P, F.Cu at (106.9, 140.3)
- added JM1: AFA07-S20FCC-00, kicad_inventree_lib:AFA07S20FCA00, B.Cu at (41.9, 80.3)
- added JM2: AFA07-S20FCC-00, kicad_inventree_lib:AFA07S20FCA00, F.Cu at (41.9, 80.3)
- added R9: 10k, Resistor_SMD:R_0603_1608Metric, F.Cu at (58.1, 75.3)
- added RN1: 3k3, Resistor_SMD:R_Array_Convex_4x0603, F.Cu at (59.0, 92.1)
- added U5: CA-IS3098W, kicad_inventree_lib:SOIC16-WBW_CLG, F.Cu at (92.9, 121.3)
- added U6: CA-IS3062VW, kicad_inventree_lib:SOIC16-WBW_CLG-M, F.Cu at (92.9, 134.3)
- C10: value 10uF -> 1uF; footprint Capacitor_SMD:C_0805_2012Metric -> Capacitor_SMD:C_0603_1608Metric
- C11: value 100nF -> 10uF; footprint Capacitor_SMD:C_0603_1608Metric -> Capacitor_SMD:C_0805_2012Metric
- C2, C5: value 22uF -> 1uF; footprint Capacitor_SMD:C_2220_5750Metric -> Capacitor_SMD:C_0603_1608Metric
- C3: value 22uF -> 10uF; footprint Capacitor_SMD:C_2220_5750Metric -> Capacitor_SMD:C_0805_2012Metric
- C6: value 22uF -> 100nF; footprint Capacitor_SMD:C_2220_5750Metric -> Capacitor_SMD:C_0603_1608Metric
- H1, H2, H3: value MountingHole_M3 -> M4; footprint kicad_inventree_lib:MountingHole_M3 -> MountingHole:MountingHole_4.3mm_M4_Pad_Via
- SP1: footprint kicad_inventree_lib:PM_LED-xx-v0.0.1 -> kicad_inventree_lib:PMLED-xx-v0.0.2
- U1: value 64900001039 -> CA-IS3062VW; footprint kicad_inventree_lib:649-Series-Holder -> kicad_inventree_lib:SOIC16-WBW_CLG-M
- moved H3 107.4 mm to (39.9, 145.3)
- moved H1 91.0 mm to (39.9, 55.3)
- moved U4 66.8 mm to (40.9, 127.3)
- moved H2 58.0 mm to (96.9, 55.3)
- moved J5 49.6 mm to (50.9, 132.6), turned to 0 degrees
- moved C6 41.5 mm to (78.9, 132.3), turned to 0 degrees
- moved C3 34.1 mm to (60.9, 135.3), turned to 180 degrees
- moved J3 26.2 mm to (41.9, 110.3)
- moved U1 23.0 mm to (69.9, 131.3), turned to 180 degrees
- moved C5 21.2 mm to (78.9, 128.3), turned to 0 degrees
- moved C2 18.1 mm to (60.9, 128.3), turned to 180 degrees
- moved C11 16.8 mm to (83.9, 117.3)
- moved C9 16.3 mm to (83.9, 133.3)
- moved C10 14.9 mm to (83.9, 137.3)
- moved C12 11.9 mm to (83.9, 130.3)
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- renumbered C1 to C7, J7 to J3, J1 to J5, U5 to U2, U7 to U3, U6 to U4
Connections:
- C10 pad 1: +3.3V_BUS -> +3.3V_CPU
- C10 pad 2: GND_BUS -> GND_CPU
- C11 pad 2: GND_BUS -> GND_CPU
- C12 pad 1: +3.3V_CPU -> +5V_CPU
- C12 pad 2: GND_BUS -> GND_CPU
- C2 pad 1: +24V_fuse -> +5V_BUS
- C2 pad 2: GND_BUS -> GND_EB
- C3 pad 1: +5V_CPU -> +5V_BUS
- C3 pad 2: GND_BUS -> GND_EB
- C5 pad 1: +24V_fuse -> +3.3V_CPU
- C5 pad 2: GND_BUS -> GND_CPU
- C6 pad 1: +3.3V_CPU -> +5V_CPU
- C6 pad 2: GND_BUS -> GND_CPU
- C7 pad 2: GND_BUS -> GND_CPU
- C9 pad 1: +3.3V_BUS -> +5V_CPU
- C9 pad 2: GND_BUS -> GND_CPU
- J3 pad 1: GND_BUS -> GND_CPU
- J3 pad 12: GND_BUS -> GND_CPU
- J3 pad 13: GND_BUS -> GND_CPU
- J5 pad 2: GND_BUS -> GND_CPU
- U1 pad 1: +24V_BUS -> +5V_CPU
- U1 pad 2: +24V_fuse -> GND_CPU
- U2 pad 03: /SPI_CS3 -> /SPI0_CS3
- U2 pad 04: GND_BUS -> GND_CPU
- U2 pad 05: /SPI_CS2 -> /SPI0_CS2
- U2 pad 06: /SPI_CS1 -> /SPI0_CS1
- U2 pad 07: /SPI_CS0 -> /SPI0_CS0
- U2 pad 09: /SPI_SCK -> /SPI0_SCK
- U2 pad 0A: /SPI_MISO -> /SPI0_MISO
- U2 pad 0B: /SPI_MOSI -> /SPI0_MOSI
- U2 pad 0C: GND_BUS -> GND_CPU
- U2 pad 12: GND_BUS -> GND_CPU
- U2 pad 16: GND_BUS -> GND_CPU
- U2 pad 19: GND_BUS -> GND_CPU
- U2 pad 21: GND_BUS -> GND_CPU
- U2 pad 22: unconnected-(U5-3V3-Pad22) -> Net-(D9-A)
- U2 pad 23: GND_BUS -> GND_CPU
- U2 pad 2C: GND_BUS -> GND_CPU
- U2 pad 31: GND_BUS -> GND_CPU
- U2 pad 34: GND_BUS -> GND_CPU
- U2 pad 38: GND_BUS -> GND_CPU
- U2 pad 3C: GND_BUS -> GND_CPU
- U3 pad 2: GND_BUS -> GND_CPU
- U4 pad 10: GND_BUS -> GND_CPU
- U4 pad 11: GND_BUS -> GND_CPU
- U4 pad 12: GND_BUS -> GND_CPU
- U4 pad 13: GND_BUS -> GND_CPU
- U4 pad 5: GND_BUS -> GND_CPU
- U4 pad 6: GND_BUS -> GND_CPU
- U4 pad 7: GND_BUS -> GND_CPU
- U4 pad 8: GND_BUS -> GND_CPU
- U4 pad 9: GND_BUS -> GND_CPU
Routing:
- net +3.3V_CPU: track 193.5 -> 0.00 mm, vias 4 -> 0
- net +5V_CPU: track 136.7 -> 0.00 mm, vias 3 -> 0
- net GND_BUS: track 84.4 -> 0.00 mm, vias 29 -> 0
- net /SPI_MOSI: track 65.9 -> 0.00 mm, vias 1 -> 0
- net /SPI_MISO: track 63.4 -> 0.00 mm, vias 1 -> 0
- net +24V_fuse: track 62.4 -> 0.00 mm, vias 2 -> 0
- net /SPI_SCK: track 60.8 -> 0.00 mm, vias 1 -> 0
- net /SPI_CS0: track 55.8 -> 0.00 mm, vias 1 -> 0
- net /SPI_CS1: track 53.2 -> 0.00 mm, vias 1 -> 0
- net /SPI_CS2: track 50.7 -> 0.00 mm, vias 1 -> 0
- net /I2C0_SDA: track 50.1 -> 0.00 mm, vias 1 -> 0
- net /LED_0: track 48.9 -> 0.00 mm
- net /B: track 48.2 -> 0.00 mm
- net /I2C0_SCL: track 47.1 -> 0.00 mm, vias 1 -> 0
- net /LED_1: track 45.9 -> 0.00 mm
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- added copper zone on B.Cu, net GND_CPU
- added copper zone on F.Cu, net GND_CPU
- added copper zone on B.Cu, net GND_EXT_CAN
- added copper zone on F.Cu, net GND_EXT_CAN
- added copper zone on B.Cu, net GND_EXT_RS
- added copper zone on F.Cu, net GND_EXT_RS
- removed copper zone on B.Cu, net GND_BUS
- removed copper zone on F.Cu, net GND_BUS
Other:
- outline, holes or cut-outs redrawn
- board text removed: "GND"

Commit message: update
Parts:
- removed U3: SN74LVC2G14DBVR, kicad_inventree_lib:DBV6-M
- moved D9 48.0 mm to (61.9, 61.3)
- moved kicad_logo 28.7 mm to (61.4, 118.3)
- moved oshw_logo 28.5 mm to (72.9, 118.3)
- moved RN1 13.1 mm to (58.8, 105.2), turned to 180 degrees
- moved CR1 12.8 mm to (53.4, 83.3)
- moved R9 6.85 mm to (53.4, 80.3), turned to 180 degrees
- moved U4 1.58 mm to (42.4, 126.8)
- moved C11 1.00 mm to (83.9, 118.3)
- moved C13 1.00 mm to (101.9, 121.3)
- moved C16 1.00 mm to (101.9, 118.3)
- moved C7 1.00 mm to (81.9, 142.3)
- moved C8 1.00 mm to (83.9, 121.3)
- moved U5 1.00 mm to (92.9, 122.3)
Connections:
- RN1 pad 1: /I2C0_SCL -> /I2C1_SDA
- RN1 pad 2: /I2C0_SDA -> /I2C1_SCL
- RN1 pad 3: /I2C1_SCL -> /I2C0_SCL
- RN1 pad 4: /I2C1_SDA -> /I2C0_SDA
- U2 pad 00: unconnected-(U2-3V3-Pad00) -> Net-(D9-A)
- U2 pad 13: unconnected-(U2-RM_IO22-Pad13) -> /WDT
- U2 pad 22: Net-(D9-A) -> unconnected-(U2-3V3-Pad22)
- U2 pad 24: /I2C0_SCL -> /CAN0_RXD
- U2 pad 25: /I2C0_SDA -> /CAN0_TXD
- U2 pad 26: unconnected-(U2-RM_IO26-Pad26) -> /I2C1_SDA
- U2 pad 27: unconnected-(U2-RM_IO27-Pad27) -> /I2C1_SCL
- U2 pad 28: /LED_2 -> /LED_1
- U2 pad 29: /LED_1 -> /LED_0
- U2 pad 2A: /LED_0 -> /I2C0_SCL
- U2 pad 2B: unconnected-(U2-RM_IO31-Pad2B) -> /I2C0_SDA
- U2 pad 35: /UART_TX -> /UART1_RX
- U2 pad 36: /UART_RTS -> /LED_2
- U2 pad 37: unconnected-(U2-Pad37) -> /UART1_RTS
- U2 pad 39: /UART_RX -> /UART1_TX
- U2 pad 3A: /I2C1_SCL -> /CAN1_TXD
- U2 pad 3B: /I2C1_SDA -> /CAN1_RXD
Routing:
- net +3.3V_CPU: track 0.00 -> 255.3 mm, vias 0 -> 13
- net +5V_CPU: track 0.00 -> 182.6 mm, vias 0 -> 6
- net /I2C0_SDA: track 0.00 -> 74.4 mm, vias 0 -> 1
- net /SPI0_MOSI: track 0.00 -> 72.4 mm, vias 0 -> 1
- net /I2C0_SCL: track 0.00 -> 71.8 mm, vias 0 -> 1
- net /SPI0_MISO: track 0.00 -> 69.8 mm, vias 0 -> 1
- net /SPI0_SCK: track 0.00 -> 67.2 mm, vias 0 -> 1
- net /SPI0_CS0: track 0.00 -> 62.0 mm, vias 0 -> 1
- net /I2C1_SCL: track 0.00 -> 61.4 mm
- net /SPI0_CS1: track 0.00 -> 59.4 mm, vias 0 -> 1
- net /LED_0: track 0.00 -> 58.8 mm, vias 0 -> 1
- net /SPI0_CS2: track 0.00 -> 56.8 mm, vias 0 -> 1
- net /I2C1_SDA: track 0.00 -> 56.7 mm
- net /LED_1: track 0.00 -> 56.1 mm, vias 0 -> 1
- net /LED_2: track 0.00 -> 53.1 mm, vias 0 -> 1
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Other:
- board text added: "${article} v${version} SN: _______________"
- board text removed: "${article} v${version}"
- board text removed: "I2C"
- board text removed: "SPI"
