File: current/PMPS-20W-v0.0.5/PMPS-20W.kicad_pcb (KiCad board)
At the start: 2 copper layers, 80 x 100 mm, 32 parts, among them J10 15EDGRC-3.5-03P, J11 AFA07-S12FCC-00, J2 K7805-2000R3, J3 K7803-2000R3, J4 K7805-2000R3, J6 15EDGRC-3.5-05P, J7 15EDGRC-3.5-05P, U1 IRM-20-24, U2 64900001039, U4 64900001039

Commit message: update
Parts:
- H1, H2, H3, H4: footprint MountingHole:MountingHole_4.3mm_M4_Pad_Via -> kicad_inventree_lib:MountingHole_4.3mm_M4_Pad_Via
- J2, J4: value K7805-2000R3 -> K78052000R3
- moved J11 5.00 mm to (87.9, 70.3)
- moved kicad_logo 2.00 mm to (99.9, 123.3)
- moved oshw_logo 2.00 mm to (110.9, 123.3)
Routing:
- net +3V3: track 151.9 -> 157.7 mm
- net +24V: track 214.7 -> 219.7 mm
- net +5V: track 126.1 -> 131.1 mm
- net +5V(2): track 88.2 -> 89.8 mm
