File: current/PMLED-18-v0.0.2/PMLED-18.kicad_sch (KiCad schematic)
At the start: 44 parts, among them J1 AFA07-S12FCC-00, J2 AFA07-S12FCC-00, J3 AFA07-S12FCC-00, J4 AFA07-S12FCC-00

Commit message: update
Parts:
- H1, H2, H3, H5: footprint MountingHole:MountingHole_2.2mm_M2_Pad_Via -> MountingHole:MountingHole_2.2mm_M2_Pad
Changed lines of the file:
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@@
 			)
 		)
-		(property "Footprint" "MountingHole:MountingHole_2.2mm_M2_Pad_Via"
+		(property "Footprint" "MountingHole:MountingHole_2.2mm_M2_Pad"
 			(at 160.02 167.64 0)
 			(effects
@@
 			)
 		)
-		(property "Footprint" "MountingHole:MountingHole_2.2mm_M2_Pad_Via"
+		(property "Footprint" "MountingHole:MountingHole_2.2mm_M2_Pad"
 			(at 160.02 152.4 0)
 			(effects
@@
 			)
 		)
-		(property "Footprint" "MountingHole:MountingHole_2.2mm_M2_Pad_Via"
+		(property "Footprint" "MountingHole:MountingHole_2.2mm_M2_Pad"
 			(at 160.02 160.02 0)
 			(effects
@@
 			)
 		)
-		(property "Footprint" "MountingHole:MountingHole_2.2mm_M2_Pad_Via"
+		(property "Footprint" "MountingHole:MountingHole_2.2mm_M2_Pad"
 			(at 160.02 175.26 0)
 			(effects

Commit message: update
Parts:
- R1, R10, R11, R12, R13, R14, R15, R16, R17, R18, R2, R3, R4, R5, R6, R7, R8, R9: footprint Resistor_SMD:R_0603_1608Metric -> kicad_inventree_lib:R_0603_1608Metric
Changed lines of the file:
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@@
 			)
 		)
-		(property "Footprint" "Resistor_SMD:R_0603_1608Metric"
+		(property "Footprint" "kicad_inventree_lib:R_0603_1608Metric"
 			(at 102.87 77.978 90)
 			(effects
@@
 			)
 		)
-		(property "Footprint" "Resistor_SMD:R_0603_1608Metric"
+		(property "Footprint" "kicad_inventree_lib:R_0603_1608Metric"
 			(at 214.63 37.338 90)
 			(effects
@@
 			)
 		)
-		(property "Footprint" "Resistor_SMD:R_0603_1608Metric"
+		(property "Footprint" "kicad_inventree_lib:R_0603_1608Metric"
 			(at 102.87 37.338 90)
 			(effects
@@
 			)
 		)
-		(property "Footprint" "Resistor_SMD:R_0603_1608Metric"
+		(property "Footprint" "kicad_inventree_lib:R_0603_1608Metric"
 			(at 158.75 77.978 90)
 			(effects
@@
 			)
 		)
-		(property "Footprint" "Resistor_SMD:R_0603_1608Metric"
+		(property "Footprint" "kicad_inventree_lib:R_0603_1608Metric"
 			(at 102.87 88.138 90)
 			(effects
@@
 			)
 		)
-		(property "Footprint" "Resistor_SMD:R_0603_1608Metric"
+		(property "Footprint" "kicad_inventree_lib:R_0603_1608Metric"
 			(at 102.87 57.658 90)
 			(effects
@@
 			)
 		)
-		(property "Footprint" "Resistor_SMD:R_0603_1608Metric"
+		(property "Footprint" "kicad_inventree_lib:R_0603_1608Metric"
 			(at 158.75 98.298 90)
 			(effects
@@
 			)
 		)
-		(property "Footprint" "Resistor_SMD:R_0603_1608Metric"
+		(property "Footprint" "kicad_inventree_lib:R_0603_1608Metric"
 			(at 102.87 47.498 90)
 			(effects
@@
 			)
 		)
-		(property "Footprint" "Resistor_SMD:R_0603_1608Metric"
+		(property "Footprint" "kicad_inventree_lib:R_0603_1608Metric"
 			(at 102.87 67.818 90)
 			(effects
@@
 			)
 		)
-		(property "Footprint" "Resistor_SMD:R_0603_1608Metric"
+		(property "Footprint" "kicad_inventree_lib:R_0603_1608Metric"
 			(at 158.75 27.178 90)
 			(effects
@@
 			)
 		)
-		(property "Footprint" "Resistor_SMD:R_0603_1608Metric"
+		(property "Footprint" "kicad_inventree_lib:R_0603_1608Metric"
 			(at 158.75 37.338 90)
 			(effects
@@
 			)
 		)
-		(property "Footprint" "Resistor_SMD:R_0603_1608Metric"
+		(property "Footprint" "kicad_inventree_lib:R_0603_1608Metric"
 			(at 102.87 98.298 90)
 			(effects
@@
 			)
 		)
-		(property "Footprint" "Resistor_SMD:R_0603_1608Metric"
+		(property "Footprint" "kicad_inventree_lib:R_0603_1608Metric"
 			(at 158.75 67.818 90)
 			(effects
@@
 			)
 		)
-		(property "Footprint" "Resistor_SMD:R_0603_1608Metric"
+		(property "Footprint" "kicad_inventree_lib:R_0603_1608Metric"
 			(at 214.63 27.178 90)
 			(effects
@@
 			)
 		)
-		(property "Footprint" "Resistor_SMD:R_0603_1608Metric"
+		(property "Footprint" "kicad_inventree_lib:R_0603_1608Metric"
 			(at 102.87 27.178 90)
 			(effects
@@
 			)
 		)
-		(property "Footprint" "Resistor_SMD:R_0603_1608Metric"
+		(property "Footprint" "kicad_inventree_lib:R_0603_1608Metric"
 			(at 158.75 88.138 90)
 			(effects
@@
 			)
 		)
-		(property "Footprint" "Resistor_SMD:R_0603_1608Metric"
+		(property "Footprint" "kicad_inventree_lib:R_0603_1608Metric"
 			(at 158.75 47.498 90)
 			(effects
@@
 			)
 		)
-		(property "Footprint" "Resistor_SMD:R_0603_1608Metric"
+		(property "Footprint" "kicad_inventree_lib:R_0603_1608Metric"
 			(at 158.75 57.658 90)
 			(effects
