File: pcb/PMPS-20W-v0.1.0/PMPS-20W.kicad_sch (KiCad schematic)
At the start: 56 parts, among them J1 15EDGK-3.5-05P, J10 15EDGRC-3.5-03P, J11 AFA11-S12GLA-00, J12 AFA11-S20GLA-00, J13 FFC_12P_P1.0_100mm_straight, J14 AFA07-S12FCC-00, J15 FFC_20P_P1.0_50mm_straight, J2 K7805-2000R3, J3 K7803-2000R3, J4 K7805-2000R3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

Commit message: PMPS-20W
Parts:
- added J16, J18: K7805-500R3, kicad_inventree_lib:K7805500R3, symbol kicad_inventree_lib:K7805-500R3
- added J17, J19: K7805-1000R3, kicad_inventree_lib:K7805-2000R3, symbol kicad_inventree_lib:K7805-1000R3
- added J20: K7803-500R3, kicad_inventree_lib:K7805-2000R3, symbol kicad_inventree_lib:K7803-500R3
- added J21: K7803-1000R3, kicad_inventree_lib:K7805-2000R3, symbol kicad_inventree_lib:K7803-1000R3
- added U3: IRM-05-24, kicad_inventree_lib:IRM-XX-24, symbol kicad_inventree_lib:IRM-05-24
- added U5: IRM-10-24, kicad_inventree_lib:IRM-XX-24, symbol kicad_inventree_lib:IRM-10-24
- added U6: IRM-15-24, kicad_inventree_lib:IRM-XX-24, symbol kicad_inventree_lib:IRM-15-24
- C2, C4: option (none) -> 2:500,2:1000,2:2000
- C3, C6: option (none) -> 4:500,4:1000,4:2000
- C5, C7: option (none) -> 3:500,3:1000,3:2000
- J12: option (none) -> 5:T,5:TB
- J2: option (none) -> 3:2000
- J3: option (none) -> 4:2000
- J4: option (none) -> 2:2000
- J8: option (none) -> 5:B,5:TB
- U1: footprint kicad_inventree_lib:IRM-20-24_MWU -> kicad_inventree_lib:IRM-XX-24; option (none) -> 1:20; optional 1 -> (none); optional_note При установке БП IRM-20-24 -> (none)
Connections:
- no-connect marks 43 -> 73
Other:
- note added: "Посадочное место IRM-XX-24"
- moved on the sheet: C2, C3, C4, C5, C6, C7, C8, F1, F2, J2, J3, J4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
